File: hw/sch_pcb/LION5CELL01.kicad_pcb (KiCad board)
At the start: 2 copper layers, 141.7 x 80.8 mm, 62 parts, among them IC1 FT260Q-T, IC2 PCA9541ABS/01, J1 SM08B-GHS-TB, J2 SD_Card-FPS009-4200-0, J3 SM06B-GHS-TB, J4 HEADER_2x03, J5 HEADER_1x01, J6 HEADER_1x01, U1 ATMEGA1284P-AU, U2 FT231XQ, U3 USBLC6-2SC6, U4 AT24CS64-SSHM, U5 PCF85263A, Y1 8 MHz, Y2 ABS07-120-32.768KHZ-T

Commit message: wip: add new components, try to prepare layout outlines
Parts:
- removed BT6: KEYS2998, Battery:BatteryHolder_Keystone_2998_1x6.8mm
- removed J1: SM08B-GHS-TB, Connector_JST:JST_GH_SM08B-GHS-TB_1x08-1MP_P1.25mm_Horizontal
- removed the J3 at (132.9, 115.8)
- removed R11: 100R, Resistor_SMD:R_0603_1608Metric
- removed the R2 at (168.4, 80.8)
- removed the R3 at (185.9, 95.7)
- added BT8: 3xBATT, Mlab_Batery:BAT_BK-18650-PC6, F.Cu at (119.2, 104.1)
- added BT9: 3xBATT, Mlab_Batery:BAT_BK-18650-PC6, F.Cu at (179.5, 104.1)
- added C1: 100nF, Capacitor_SMD:C_0805_2012Metric, B.Cu at (108.3, 39.0)
- added C10: 1uF, Capacitor_SMD:C_0805_2012Metric, B.Cu at (121.4, 39.0)
- added C13: 1nF, Capacitor_SMD:C_0805_2012Metric, B.Cu at (124.4, 39.0)
- added C2: 100nF, Capacitor_SMD:C_0805_2012Metric, B.Cu at (111.3, 39.0)
- added C28: 100nF, Capacitor_SMD:C_0805_2012Metric, B.Cu at (121.3, 18.0)
- added C29: 1uF, Capacitor_SMD:C_0805_2012Metric, B.Cu at (124.3, 18.0)
- added C30: 100nF, Capacitor_SMD:C_0805_2012Metric, B.Cu at (103.2, 22.5)
- added C31: 100nF, Capacitor_SMD:C_0805_2012Metric, B.Cu at (106.2, 22.5)
- added C32: 3n3, Capacitor_SMD:C_0805_2012Metric, B.Cu at (109.2, 22.5)
- added C33: 100nF, Capacitor_SMD:C_0805_2012Metric, B.Cu at (112.2, 22.5)
- added C34: 100nF, Capacitor_SMD:C_0805_2012Metric, B.Cu at (115.2, 22.5)
- added C35: 47n, Capacitor_SMD:C_0805_2012Metric, B.Cu at (118.2, 22.5)
- added C36: 10uF, Capacitor_SMD:C_0805_2012Metric, B.Cu at (260.8, 85.2)
- added C37: 10uF, Capacitor_SMD:C_0805_2012Metric, B.Cu at (260.8, 88.2)
- added C38: 10uF, Capacitor_SMD:C_0805_2012Metric, B.Cu at (260.8, 91.2)
- added C39: 10u, Capacitor_SMD:C_0805_2012Metric, B.Cu at (106.2, 26.9)
- added C40: 1u, Capacitor_SMD:C_0805_2012Metric, B.Cu at (286.5, 19.1)
- added C41: 1u, Capacitor_SMD:C_0805_2012Metric, B.Cu at (286.5, 22.1)
- added C42: 1u, Capacitor_SMD:C_0805_2012Metric, B.Cu at (286.5, 25.1)
- added C43: 4u7, Capacitor_SMD:C_0805_2012Metric, B.Cu at (118.2, 26.9)
- added C44: 1u, Capacitor_SMD:C_0805_2012Metric, B.Cu at (286.5, 28.1)
- added C45: 100n, Capacitor_SMD:C_0805_2012Metric, B.Cu at (286.5, 31.1)
- added C47: 20u, Capacitor_SMD:C_0805_2012Metric, B.Cu at (106.2, 31.4)
- added C48: 10u, Capacitor_SMD:C_0805_2012Metric, B.Cu at (109.2, 31.4)
- added C49: 0u1, Capacitor_SMD:C_0805_2012Metric, B.Cu at (112.2, 31.4)
- added C5: 22uF, Capacitor_SMD:C_0805_2012Metric, B.Cu at (269.7, 91.2)
- added C50: 10u, Capacitor_SMD:C_0805_2012Metric, B.Cu at (115.2, 31.4)
- added C6: 47uF, Capacitor_SMD:C_0805_2012Metric, B.Cu at (265.2, 85.2)
- added C7: 47uF, Capacitor_SMD:C_0805_2012Metric, B.Cu at (265.2, 88.2)
- added C8: 47uF, Capacitor_SMD:C_0805_2012Metric, B.Cu at (265.2, 91.2)
- added D10: ORAGE, Mlab_D:LED_1206, B.Cu at (242.7, 145.9)
- added D11: GREEN, Mlab_D:LED_1206_mill, B.Cu at (291.8, 19.3)
- added D13: RED, Mlab_D:LED_1206_mill, B.Cu at (291.8, 22.9)
- added D14: YELLOW, Mlab_D:LED_1206_mill, B.Cu at (291.8, 26.4)
- added D15: BLUE, Mlab_D:LED_1206_mill, B.Cu at (291.8, 30.0)
- added D16: RED, Mlab_D:LED_1206_mill, B.Cu at (291.8, 33.5)
- added D3: ORAGE, Mlab_D:LED_1206, B.Cu at (246.0, 146.5)
- added D4: ORAGE, Mlab_D:LED_1206, B.Cu at (250.0, 146.5)
- added D5: ORAGE, Mlab_D:LED_1206, B.Cu at (254.0, 146.5)
- added D6: ORAGE, Mlab_D:LED_1206, B.Cu at (258.0, 146.5)
- added D7: ORAGE, Mlab_D:LED_1206, B.Cu at (262.0, 146.5)
- added D8: ORAGE, Mlab_D:LED_1206, B.Cu at (265.5, 146.6)
- added D9: ORAGE, Mlab_D:LED_1206, B.Cu at (238.7, 145.9)
- added F1: Fuse, Mlab_F:Drzak_2410, B.Cu at (194.3, 137.8)
- added F2: Fuse, Mlab_F:Drzak_2410, B.Cu at (184.0, 137.7)
- added F3: Fuse, Mlab_F:Drzak_2410, B.Cu at (164.6, 137.8)
- added F4: Fuse, Mlab_F:Drzak_2410, B.Cu at (142.9, 137.7)
- added F5: Fuse, Mlab_F:Drzak_2410, B.Cu at (123.6, 137.7)
- added F6: Fuse, Mlab_F:Drzak_2410, B.Cu at (104.3, 137.8)
- added J10: HEADER_2x04_PARALLEL, Connector_PinHeader_2.54mm:PinHeader_2x04_P2.54mm_Vertical, B.Cu at (250.3, 20.5)
- added J7: USBC_USB4105-GF-A, Mlab_CON:USBC GCT_USB4105-GF-A, B.Cu at (216.6, 80.0)
- added JP10: Jumper_3_Bridged12, Jumper:SolderJumper-3_P1.3mm_Bridged12_RoundedPad1.0x1.5mm, B.Cu at (248.5, 47.2)
- added JP11: Jumper_3_Bridged12, Connector_PinHeader_2.54mm:PinHeader_1x03_P2.54mm_Vertical, B.Cu at (260.9, 38.3)
- added JP3: Jumper_2_Open, Connector_PinHeader_2.54mm:PinHeader_1x02_P2.54mm_Vertical, B.Cu at (165.1, 43.4)
- added JP4: Jumper_2_Open, Connector_PinHeader_2.54mm:PinHeader_1x02_P2.54mm_Vertical, B.Cu at (264.7, 78.8)
- added JP5: Jumper_2_Open, Connector_PinHeader_2.54mm:PinHeader_1x02_P2.54mm_Vertical, B.Cu at (160.4, 43.4)
- added JP7: Jumper_2_Open, Connector_PinHeader_2.54mm:PinHeader_1x02_P2.54mm_Vertical, B.Cu at (255.4, 78.8)
- added JP9: Jumper_2_Open, Connector_PinHeader_2.54mm:PinHeader_2x01_P2.54mm_Vertical, B.Cu at (256.2, 47.8)
- added L1: 1uH - DFE252012P-1R0M=P2, Inductor_SMD:L_1008_2520Metric, B.Cu at (269.4, 94.6)
- added L2: 1uH - DFE252012P-1R0M=P2, Inductor_SMD:L_1008_2520Metric, B.Cu at (269.4, 98.3)
- added L5: DE1205-10, Mlab_L:DE1205-10, B.Cu at (193.3, 22.9)
- added L6: 1uH - DFE252012P-1R0M=P2, Inductor_SMD:L_1008_2520Metric, B.Cu at (269.4, 102.1)
- added Q1: IRF9317TRPBF, Package_SO:SOIC-8_3.9x4.9mm_P1.27mm, B.Cu at (189.0, 88.0)
- added R10: 1k, Resistor_SMD:R_0603_1608Metric, B.Cu at (265.0, 94.0)
- added R23: 47k, Resistor_SMD:R_0805_2012Metric, B.Cu at (145.3, 31.4)
- added R24: 47k, Resistor_SMD:R_0805_2012Metric, B.Cu at (148.2, 31.4)
- added R25: 47k, Resistor_SMD:R_0805_2012Metric, B.Cu at (151.2, 31.4)
- added R26: 10K NTC, Resistor_SMD:R_0805_2012Metric_Pad1.20x1.40mm_HandSolder, B.Cu at (213.4, 35.6)
- added R27: 1k, Resistor_SMD:R_0805_2012Metric, B.Cu at (154.2, 31.4)
- added R28: 100R, Resistor_SMD:R_0805_2012Metric, B.Cu at (139.4, 35.8)
- added R29: 100R, Resistor_SMD:R_0805_2012Metric, B.Cu at (142.3, 35.8)
- added R30: 0R01 75PPM, Resistor_SMD:R_2512_6332Metric_Pad1.40x3.35mm_HandSolder, B.Cu at (186.2, 75.0)
- added R31: 270R, Resistor_SMD:R_0805_2012Metric, B.Cu at (255.2, 134.6)
- added R32: 270R, Resistor_SMD:R_0805_2012Metric, B.Cu at (258.2, 134.6)
- added R33: 270R, Resistor_SMD:R_0805_2012Metric, B.Cu at (261.1, 134.6)
- added R34: 270R, Resistor_SMD:R_0805_2012Metric, B.Cu at (264.1, 134.6)
- added R35: 270R, Resistor_SMD:R_0805_2012Metric, B.Cu at (249.3, 139.0)
- added R36: 270R, Resistor_SMD:R_0805_2012Metric, B.Cu at (252.3, 139.0)
- added R37: 270R, Resistor_SMD:R_0805_2012Metric, B.Cu at (255.2, 139.0)
- added R38: 270R, Resistor_SMD:R_0805_2012Metric, B.Cu at (258.2, 139.0)
- added R39: R_Small, Resistor_SMD:R_0603_1608Metric, B.Cu at (168.7, 17.8)
- added R40: 511k, Resistor_SMD:R_0805_2012Metric, B.Cu at (274.1, 96.9)
- added R41: 91k, Resistor_SMD:R_0805_2012Metric, B.Cu at (274.1, 99.9)
- added R42: 806k, Resistor_SMD:R_0805_2012Metric, B.Cu at (274.1, 102.8)
- added R43: 91k, Resistor_SMD:R_0805_2012Metric, B.Cu at (274.1, 105.8)
- added R44: 100k, Resistor_SMD:R_0805_2012Metric, B.Cu at (274.2, 19.7)
- added R45: R_Small, Resistor_SMD:R_0603_1608Metric, B.Cu at (171.2, 21.8)
- added R46: 4k7, Resistor_SMD:R_0805_2012Metric, B.Cu at (274.2, 22.6)
- added R47: 4k7, Resistor_SMD:R_0805_2012Metric, B.Cu at (274.2, 25.6)
- added R48: 4k7, Resistor_SMD:R_0805_2012Metric, B.Cu at (274.2, 28.5)
- added R49: 4k7, Resistor_SMD:R_0805_2012Metric, B.Cu at (274.2, 31.5)
- added R5: 10k, Resistor_SMD:R_0603_1608Metric, B.Cu at (116.7, 43.2)
- added R50: 4k7, Resistor_SMD:R_0805_2012Metric, B.Cu at (274.2, 34.4)
- added R51: 4k7, Resistor_SMD:R_0805_2012Metric, B.Cu at (274.2, 37.4)
- added R52: 4k7, Resistor_SMD:R_0805_2012Metric, B.Cu at (269.8, 19.7)
- added R53: 100k, Resistor_SMD:R_0805_2012Metric, B.Cu at (269.8, 22.6)
- added R54: 62R, Resistor_SMD:R_0805_2012Metric, B.Cu at (269.8, 25.6)
- added R55: R, Resistor_SMD:R_0603_1608Metric, B.Cu at (171.2, 29.8)
- added R56: R, Resistor_SMD:R_0603_1608Metric, B.Cu at (173.7, 29.8)
- added R57: R, Resistor_SMD:R_0603_1608Metric, B.Cu at (176.2, 29.8)
- added R58: R, Resistor_SMD:R_0603_1608Metric, B.Cu at (178.7, 29.8)
- added R59: 62R, Resistor_SMD:R_0805_2012Metric, B.Cu at (269.8, 28.5)
- added R6: 1k, Resistor_SMD:R_0805_2012Metric, B.Cu at (274.1, 85.1)
- added R60: 62R, Resistor_SMD:R_0805_2012Metric, B.Cu at (269.8, 31.5)
- added R61: 10R, Resistor_SMD:R_0805_2012Metric, B.Cu at (269.8, 34.4)
- added R62: 1k, Resistor_SMD:R_0805_2012Metric, B.Cu at (269.8, 37.4)
- added R63: 62R, Resistor_SMD:R_0805_2012Metric, B.Cu at (265.4, 19.7)
- added R64: 100k, Resistor_SMD:R_0805_2012Metric, B.Cu at (265.4, 22.6)
- added R65: 20k, Resistor_SMD:R_0805_2012Metric, B.Cu at (265.4, 25.6)
- added R66: 100R, Resistor_SMD:R_0805_2012Metric, B.Cu at (265.4, 28.5)
- added R67: 1k, Resistor_SMD:R_0805_2012Metric, B.Cu at (265.4, 31.5)
- added R68: 1k, Resistor_SMD:R_0805_2012Metric, B.Cu at (165.2, 49.7)
- added R8: 1k, Resistor_SMD:R_0805_2012Metric, B.Cu at (274.1, 91.0)
- added R9: 1k, Resistor_SMD:R_0805_2012Metric, B.Cu at (274.1, 94.0)
- added U10: SN74HC164D, Package_SO:SO-14_3.9x8.65mm_P1.27mm, B.Cu at (208.5, 125.8)
- added U13: STUSB4500QTR, Package_DFN_QFN:QFN-24-1EP_4x4mm_P0.5mm_EP2.7x2.7mm, B.Cu at (205.6, 79.7)
- added U5: TPS22965-Q1, Package_SON:WSON-8-1EP_2x2mm_P0.5mm_EP0.9x1.6mm_ThermalVias, B.Cu at (121.7, 43.3)
- added U9: BQ34Z100, Mlab_IO:TSSOP-14_4.4x5mm_Pitch0.65mm, B.Cu at (172.4, 80.8)
- C11: renamed from C2; moved to B.Cu
- C12: renamed from C5; moved to B.Cu
- C14: renamed from C7; moved to B.Cu
- C15: renamed from C12; moved to B.Cu
- C16: renamed from C6; moved to B.Cu
- C17: renamed from C9; moved to B.Cu
- C18: renamed from C15; moved to B.Cu
- C19: renamed from C10; moved to B.Cu
- C20: renamed from C8; moved to B.Cu
- C21: renamed from C11; moved to B.Cu
- C22: renamed from C13; moved to B.Cu
- C23: renamed from C14; moved to B.Cu
- C24: renamed from C16; moved to B.Cu
- C25: renamed from C19; moved to B.Cu
- C26: renamed from C18; moved to B.Cu
- C27: renamed from C17; moved to B.Cu
- C3, C4: value 100nF -> 22uF; footprint Mlab_C:SMD-0805 -> Capacitor_SMD:C_0805_2012Metric; moved to B.Cu
- C9: renamed from C1; moved to B.Cu
- FID1, FID2, FID3, FID4, IC1, IC2, JP1, Y1, Y2: moved to B.Cu
- J3: renamed from J2; moved to B.Cu
- J4: renamed from J5; moved to B.Cu
- J5: renamed from J6; moved to B.Cu
- J6: renamed from J4; moved to B.Cu
- JP2: value SolderJumper_2_Bridged -> Jumper_2_Open; footprint Jumper:SolderJumper-2_P1.3mm_Bridged_RoundedPad1.0x1.5mm -> Connector_PinHeader_2.54mm:PinHeader_1x02_P2.54mm_Vertical; moved to B.Cu
- L3: renamed from L1; moved to B.Cu
- L4: renamed from L2; moved to B.Cu
- R1: value 10k -> 100R; moved to B.Cu
- R12: value 100R -> 511k; moved to B.Cu
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Connections:
- net /mcu/PB4 renamed /mcu/CS_SD
- net /mcu/PB5 renamed /mcu/MOSI
- net /mcu/PB6 renamed /mcu/MISO
- net /mcu/PB7 renamed /mcu/SCK
- C27 pad 1: +3.3V -> unconnected-(C27-Pad1)
- C27 pad 2: GND -> unconnected-(C27-Pad2)
- C3 pad 1: +3V3 -> +VSW
- C4 pad 1: GND -> +VSW
- C4 pad 2: /VCCIO -> GND
- IC1 pad 24: Net-(IC1-AGND) -> GND
- IC1 pad 29: Net-(IC1-AGND) -> GND
- IC2 pad 11: /SCL_INT -> SCL_I2C
- IC2 pad 12: /SDA_INT -> SDA_I2C
- JP1 pad 2: Net-(JP1-B) -> /DTR
- JP2 pad 1: /VCCIO -> GND
- JP2 pad 2: +3V3 -> /sw_source/5v_mod
- R1 pad 1: /mcu/SDA -> RST#
- R1 pad 2: +3.3V -> Net-(JP1-A)
- R12 pad 1: RX0 -> +3.3V
- R12 pad 2: Net-(J3-Pad2) -> /sw_source/3v3i_FB
- R13 pad 1: TX0 -> /sw_source/3v3i_FB
- R13 pad 2: Net-(J3-Pad3) -> GND
- R4 pad 1: Net-(U2-~{RESET}) -> SCL_I2C
- R4 pad 2: GND -> +3.3V
- U1 pad 5: /VBUS -> VBUS
- U2 pad 1: /RXD -> SDA_I2C
- U2 pad 2: /#RI -> GND
- U2 pad 3: GND -> unconnected-(U2-ALERT-Pad3)
- U2 pad 4: /#DSR -> SCL_I2C
- U2 pad 5: /#DCD -> +3.3V
- U2 pad 6: /#CTS -> unconnected-(U2-~{RESET}-Pad6)
- U2 pad 7: /TXLED/CBUS2 -> GND
- U2 pad 8: /DP -> GND
- U2 pad 9: /DN -> GND
- U6 pad 13: /mcu/TIMEPULSE -> unconnected-(U6-(PCINT28/XCK1/OC1B)PD4-Pad13)
- U6 pad 14: /mcu/EXTINT -> unconnected-(U6-(PCINT294/OC1A)PD5-Pad14)
- U6 pad 15: /mcu/GEO_STAT -> unconnected-(U6-(PCINT30/OC2B/ICP)PD6-Pad15)
- U6 pad 37: PA0 -> unconnected-(U6-(PCINT0/ADC0)PA0-Pad37)
- U6 pad 40: PB0 -> unconnected-(U6-(PCINT8/T0/XCK)PB0-Pad40)
Routing:
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Other:
- board size 141.7 x 80.8 mm -> 141.7 x 85.9 mm
- board text added: "MLAB pattern"
- board text added: "adapter_module"
- board text added: "module dimensions"

Commit message: wip, update schematics, board outlines
Parts:
- removed the F4 at (142.9, 137.7)
- removed JP10: Jumper_3_Bridged12, Jumper:SolderJumper-3_P1.3mm_Bridged12_RoundedPad1.0x1.5mm
- removed JP11: Jumper_3_Bridged12, Connector_PinHeader_2.54mm:PinHeader_1x03_P2.54mm_Vertical
- removed JP9: Jumper_2_Open, Connector_PinHeader_2.54mm:PinHeader_2x01_P2.54mm_Vertical
- removed the R25 at (151.2, 31.4)
- removed the R44 at (274.2, 19.7)
- removed the R53 at (269.8, 22.6)
- added C11: 100nF, Capacitor_SMD:C_0805_2012Metric, B.Cu at (325.4, 71.5)
- added C6: 4u7, Capacitor_SMD:C_0805_2012Metric, B.Cu at (325.4, 59.5)
- added C7: 4u7, Capacitor_SMD:C_0805_2012Metric, B.Cu at (325.4, 62.5)
- added C8: 0u1, Capacitor_SMD:C_0805_2012Metric, B.Cu at (325.4, 65.5)
- added C9: 4u7, Capacitor_SMD:C_0805_2012Metric, B.Cu at (325.4, 68.5)
- added R18: 10k, Resistor_SMD:R_0805_2012Metric, B.Cu at (321.0, 59.4)
- added R19: 10k, Resistor_SMD:R_0805_2012Metric, B.Cu at (321.0, 62.4)
- added R20: 10k, Resistor_SMD:R_0805_2012Metric, B.Cu at (321.0, 65.3)
- added R21: 10k, Resistor_SMD:R_0805_2012Metric, B.Cu at (321.0, 68.3)
- added R22: 10k, Resistor_SMD:R_0805_2012Metric, B.Cu at (321.0, 71.2)
- added R24: 33R, Resistor_SMD:R_0805_2012Metric, B.Cu at (316.5, 62.4)
- added R28: 1k, Resistor_SMD:R_0805_2012Metric, B.Cu at (316.5, 65.3)
- added R68: 10k, Resistor_SMD:R_0805_2012Metric, B.Cu at (316.5, 68.3)
- added R69: 10k, Resistor_SMD:R_0805_2012Metric, B.Cu at (316.5, 71.2)
- added R70: 10k, Resistor_SMD:R_0805_2012Metric, B.Cu at (312.1, 59.4)
- added R71: 10k, Resistor_SMD:R_0805_2012Metric, B.Cu at (312.1, 62.4)
- added R72: 10k, Resistor_SMD:R_0805_2012Metric, B.Cu at (312.1, 65.3)
- added TH1: Thermistor_NTC, Resistor_SMD:R_0805_2012Metric, B.Cu at (298.6, 59.4)
- added TP1: FTDI FS, TestPoint:TestPoint_Pad_D1.5mm, B.Cu at (308.2, 59.7)
- added TP2: MUX_RST, TestPoint:TestPoint_Pad_D1.5mm, B.Cu at (308.2, 63.3)
- added TP3: CH_PG, TestPoint:TestPoint_Pad_D1.5mm, B.Cu at (302.6, 59.7)
- added TP4: CH_STAT, TestPoint:TestPoint_Pad_D1.5mm, B.Cu at (302.6, 63.3)
- added TP5: CH_INT, TestPoint:TestPoint_Pad_D1.5mm, B.Cu at (302.6, 66.8)
- added U16: TCA4307, Package_SO:VSSOP-8_3.0x3.0mm_P0.65mm, B.Cu at (319.2, 75.0)
- added U7: BQ25628E, Package_DFN_QFN:Texas_S-PWQFN-N20, F.Cu at (168.4, 103.5)
- BT1: renamed from BT8; footprint Mlab_Batery:BAT_BK-18650-PC6 -> Mlab_Batery:BAT_BK-18650-PC4
- C27: renamed from C9; footprint Capacitor_SMD:C_0603_1608Metric -> Capacitor_SMD:C_0805_2012Metric
- C28: renamed from C11; footprint Capacitor_SMD:C_0603_1608Metric -> Capacitor_SMD:C_0805_2012Metric
- C30: renamed from C12; footprint Capacitor_SMD:C_0603_1608Metric -> Capacitor_SMD:C_0805_2012Metric
- C31: renamed from C14; footprint Capacitor_SMD:C_0603_1608Metric -> Capacitor_SMD:C_0805_2012Metric
- C34: renamed from C17; footprint Capacitor_SMD:C_0603_1608Metric -> Capacitor_SMD:C_0805_2012Metric
- C35: renamed from C16; footprint Capacitor_SMD:C_0603_1608Metric -> Capacitor_SMD:C_0805_2012Metric
- C36: renamed from C18; footprint Capacitor_SMD:C_0603_1608Metric -> Capacitor_SMD:C_0805_2012Metric
- C37: renamed from C19; footprint Capacitor_SMD:C_0603_1608Metric -> Capacitor_SMD:C_0805_2012Metric
- C38: renamed from C20; footprint Capacitor_SMD:C_0603_1608Metric -> Capacitor_SMD:C_0805_2012Metric
- C39: renamed from C21; footprint Capacitor_SMD:C_0603_1608Metric -> Capacitor_SMD:C_0805_2012Metric
- C40: renamed from C22; footprint Capacitor_SMD:C_0603_1608Metric -> Capacitor_SMD:C_0805_2012Metric
- C41: renamed from C23; footprint Capacitor_SMD:C_0603_1608Metric -> Capacitor_SMD:C_0805_2012Metric
- C42: renamed from C24; footprint Capacitor_SMD:C_0603_1608Metric -> Capacitor_SMD:C_0805_2012Metric
- C43: renamed from C25; footprint Capacitor_SMD:C_0603_1608Metric -> Capacitor_SMD:C_0805_2012Metric
- C44: renamed from C26; footprint Capacitor_SMD:C_0603_1608Metric -> Capacitor_SMD:C_0805_2012Metric
- C45: renamed from C27; footprint Capacitor_SMD:C_0603_1608Metric -> Capacitor_SMD:C_0805_2012Metric
- R23: value 47k -> 33R
- R25: renamed from R1; footprint Resistor_SMD:R_0603_1608Metric -> Resistor_SMD:R_0805_2012Metric
- R26: renamed from R2; footprint Resistor_SMD:R_0603_1608Metric -> Resistor_SMD:R_0805_2012Metric
- R27: renamed from R3; footprint Resistor_SMD:R_0603_1608Metric -> Resistor_SMD:R_0805_2012Metric
- R29: renamed from R4; footprint Resistor_SMD:R_0603_1608Metric -> Resistor_SMD:R_0805_2012Metric
- R30: renamed from R5; footprint Resistor_SMD:R_0603_1608Metric -> Resistor_SMD:R_0805_2012Metric
- R32: renamed from R55; footprint Resistor_SMD:R_0603_1608Metric -> Resistor_SMD:R_0805_2012Metric
- R33: renamed from R56; footprint Resistor_SMD:R_0603_1608Metric -> Resistor_SMD:R_0805_2012Metric
- R34: renamed from R26; footprint Resistor_SMD:R_0805_2012Metric_Pad1.20x1.40mm_HandSolder -> Resistor_SMD:R_0805_2012Metric
- R36: renamed from R39; footprint Resistor_SMD:R_0603_1608Metric -> Resistor_SMD:R_0805_2012Metric
- R37: renamed from R45; footprint Resistor_SMD:R_0603_1608Metric -> Resistor_SMD:R_0805_2012Metric
- R40: renamed from R30; footprint Resistor_SMD:R_2512_6332Metric_Pad1.40x3.35mm_HandSolder -> Resistor_SMD:R_0805_2012Metric
- R49: renamed from R57; footprint Resistor_SMD:R_0603_1608Metric -> Resistor_SMD:R_0805_2012Metric
- R50: renamed from R58; footprint Resistor_SMD:R_0603_1608Metric -> Resistor_SMD:R_0805_2012Metric
- R51: renamed from R17; footprint Resistor_SMD:R_0603_1608Metric -> Resistor_SMD:R_0805_2012Metric
- R52: renamed from R18; footprint Resistor_SMD:R_0603_1608Metric -> Resistor_SMD:R_0805_2012Metric
- R53: renamed from R19; footprint Resistor_SMD:R_0603_1608Metric -> Resistor_SMD:R_0805_2012Metric
- R54: renamed from R20; footprint Resistor_SMD:R_0603_1608Metric -> Resistor_SMD:R_0805_2012Metric
- R55: renamed from R21; footprint Resistor_SMD:R_0603_1608Metric -> Resistor_SMD:R_0805_2012Metric
- R56: renamed from R22; footprint Resistor_SMD:R_0603_1608Metric -> Resistor_SMD:R_0805_2012Metric
- R61: renamed from R10; footprint Resistor_SMD:R_0603_1608Metric -> Resistor_SMD:R_0805_2012Metric
- R62: renamed from R12; footprint Resistor_SMD:R_0603_1608Metric -> Resistor_SMD:R_0805_2012Metric
- R63: renamed from R13; footprint Resistor_SMD:R_0603_1608Metric -> Resistor_SMD:R_0805_2012Metric
- Y1: footprint Mlab_XTAL:Crystal_HC49-4H_Vertical -> Crystal:Crystal_SMD_3225-4Pin_3.2x2.5mm
- moved R23 173.5 mm to (316.5, 59.4), turned to 180 degrees
- moved FID4 92.1 mm to (205.9, 138.0)
- moved J3 88.7 mm to (34.2, 118.0), turned to -90 degrees
- moved FID1 74.3 mm to (193.3, 71.9)
- moved Y1 53.9 mm to (111.7, 109.7), turned to -45 degrees
- moved C38 47.8 mm to (109.3, 112.1), turned to -90 degrees
- moved C35 47.7 mm to (109.3, 106.8), turned to 90 degrees
- moved FID2 46.8 mm to (112.1, 140.2)
- moved F1 38.6 mm to (142.9, 137.8)
- moved R40 20.4 mm to (165.9, 73.5)
- moved BT1 9.65 mm to (128.8, 104.1)
- moved J1 7.40 mm to (216.6, 87.4)
- moved U1 0.29 mm to (205.4, 79.4)
- renumbered BT9 to BT2, C40 to C1, C1 to C10, C2 to C12, C48 to C13, C49 to C14, C50 to C15, C28 to C16, C29 to C17, C30 to C18, C31 to C19, C41 to C2, C35 to C20, C32 to C21, C39 to C22, C33 to C23, C47 to C24, C43 to C25, C34 to C26, C10 to C29, C42 to C3, C13 to C32, C15 to C33, C44 to C4, C3 to C46, C4 to C47, C5 to C48, C6 to C49, C45 to C5, C7 to C50, C8 to C51, C36 to C52, C37 to C53, C38 to C54, D11 to D1, D5 to D10, D6 to D11, D7 to D12, D8 to D13, D9 to D14, D10 to D15, D13 to D2, D14 to D3, D15 to D4, D16 to D5, D3 to D8, D4 to D9, F6 to F1, F5 to F2, F2 to F4, F1 to F5, J7 to J1, J10 to J2, JP3 to JP2, JP5 to JP3, JP2 to JP4, JP4 to JP5, JP7 to JP6, L5 to L1, L3 to L2, L4 to L3, L1 to L4, L2 to L5, R46 to R1, R60 to R10, R61 to R11, R62 to R12, R64 to R13, R63 to R14, R65 to R15, R66 to R16, R67 to R17, R47 to R2, R48 to R3, R24 to R31, R27 to R35, R28 to R38, R29 to R39, R49 to R4, R31 to R41, R32 to R42, R33 to R43, R34 to R44, R35 to R45, R36 to R46, R37 to R47, R38 to R48, R50 to R5, R9 to R57, R68 to R58, R6 to R59, R51 to R6, R8 to R60, R40 to R64, R41 to R65, R42 to R66, R43 to R67, R52 to R7, R54 to R8, R59 to R9, U13 to U1, U6 to U10, U7 to U11, U8 to U12, U1 to U2, U2 to U3, IC2 to U4, U9 to U6, U5 to U9
Connections:
- net GAUGE_BTN_A renamed /liion/GAUGE_BTN_A
- net GAUGE_BTN_B renamed /liion/GAUGE_BTN_B
- C18 pad 1: Net-(U9-SRP) -> Net-(U6-SRN)
- C18 pad 2: Net-(U9-SRN) -> Net-(U6-SRN)
- C19 pad 1: Net-(U9-SRN) -> Net-(U6-SRN)
- C2 pad 1: VCC -> +3.3V
- C23 pad 1: Net-(U9-SRP) -> Net-(U6-SRN)
- C38 pad 1: Net-(U6-XTAL1) -> Net-(U10-XTAL1)
- C45 pad 1: unconnected-(C27-Pad1) -> +3.3V
- C45 pad 2: unconnected-(C27-Pad2) -> GND
- C46 pad 1: +VSW -> unconnected-(C46-Pad1)
- C46 pad 2: GND -> unconnected-(C46-Pad2)
- C47 pad 1: +VSW -> unconnected-(C47-Pad1)
- C47 pad 2: GND -> unconnected-(C47-Pad2)
- C48 pad 1: +VSW -> unconnected-(C48-Pad1)
- C48 pad 2: GND -> unconnected-(C48-Pad2)
- C49 pad 1: +3.3V -> unconnected-(C49-Pad1)
- C49 pad 2: GND -> unconnected-(C49-Pad2)
- C50 pad 1: 3v3_EXT -> unconnected-(C50-Pad1)
- C50 pad 2: GND -> unconnected-(C50-Pad2)
- C51 pad 1: 5v_EXT -> unconnected-(C51-Pad1)
- C51 pad 2: GND -> unconnected-(C51-Pad2)
- C52 pad 1: +3.3V -> unconnected-(C52-Pad1)
- C52 pad 2: GND -> unconnected-(C52-Pad2)
- C53 pad 1: 3v3_EXT -> unconnected-(C53-Pad1)
- C53 pad 2: GND -> unconnected-(C53-Pad2)
- C54 pad 1: 5v_EXT -> unconnected-(C54-Pad1)
- C54 pad 2: GND -> unconnected-(C54-Pad2)
- IC1 pad 1: unconnected-(IC1-DEBUGGER-Pad1) -> Net-(IC1-DEBUGGER)
- IC1 pad 19: unconnected-(IC1-GND-Pad19) -> GND
- IC1 pad 2: unconnected-(IC1-STEST_RSTN-Pad2) -> Net-(IC1-STEST_RSTN)
- IC1 pad 20: unconnected-(IC1-DM-Pad20) -> Net-(IC1-DM)
- IC1 pad 21: unconnected-(IC1-DP-Pad21) -> Net-(IC1-DP)
- IC1 pad 22: unconnected-(IC1-VOUT3V3-Pad22) -> +3.3V
- IC1 pad 23: unconnected-(IC1-VCCIN-Pad23) -> +3.3V
- IC1 pad 25: unconnected-(IC1-FSOURCE-Pad25) -> Net-(IC1-FSOURCE)
- IC1 pad 3: GND -> Net-(IC1-RESETN)
- IC1 pad 4: GND -> Net-(IC1-DCNF0)
- IC1 pad 5: GND -> Net-(IC1-DCNF1)
- IC1 pad 6: unconnected-(IC1-VCCIO-Pad6) -> +3.3V
- R23 pad 1: /liion/I2C_SDA -> Net-(IC1-DP)
- R23 pad 2: +3V3 -> /DP
- R26 pad 2: unconnected-(R2-Pad2) -> GND
- R27 pad 2: unconnected-(R3-Pad2) -> GND
- R38 pad 1: unconnected-(R28-Pad1) -> /liion/GAUGE_SRP
- R38 pad 2: Net-(U9-SRP) -> Net-(U6-SRN)
- R39 pad 2: Net-(U9-SRN) -> Net-(U6-SRN)
- R62 pad 1: +3.3V -> unconnected-(R62-Pad1)
- R62 pad 2: /sw_source/3v3i_FB -> unconnected-(R62-Pad2)
- R63 pad 1: /sw_source/3v3i_FB -> unconnected-(R63-Pad1)
- R63 pad 2: GND -> unconnected-(R63-Pad2)
- R64 pad 1: 3v3_EXT -> unconnected-(R64-Pad1)
- R64 pad 2: /sw_source/3v3_FB -> unconnected-(R64-Pad2)
- R65 pad 1: /sw_source/3v3_FB -> unconnected-(R65-Pad1)
- R65 pad 2: GND -> unconnected-(R65-Pad2)
- R66 pad 1: 5v_EXT -> unconnected-(R66-Pad1)
- R66 pad 2: /sw_source/5v_FB -> unconnected-(R66-Pad2)
- R67 pad 1: /sw_source/5v_FB -> unconnected-(R67-Pad1)
- R67 pad 2: GND -> unconnected-(R67-Pad2)
- U1 pad 12: /ADDR0 -> GND
- U1 pad 13: /ADDR1 -> GND
- U1 pad 22: VCC -> +3.3V
- U10 pad 8: Net-(U6-XTAL1) -> Net-(U10-XTAL1)
- U11 pad 5: /mcu/PC1 -> /mcu/SDA
- U11 pad 6: /mcu/PC0 -> /mcu/SCL
- U12 pad 6: /mcu/PC1 -> /mcu/SDA
- U12 pad 7: /mcu/PC0 -> /mcu/SCL
- U4 pad 14: unconnected-(IC2-VDD-Pad14) -> +3.3V
- U4 pad 17: unconnected-(IC2-EP-Pad17) -> (no net)
- U4 pad 2: unconnected-(IC2-~{RESET}-Pad2) -> Net-(U4-~{RESET})
- U6 pad 10: Net-(U9-SRN) -> Net-(U6-SRN)
- U6 pad 13: /liion/I2C_SCL -> SCL_I2C
- U6 pad 14: /liion/I2C_SDA -> SDA_I2C
- U6 pad 9: Net-(U9-SRP) -> Net-(U6-SRN)
- Y1 pad 2: Net-(U6-XTAL1) -> GND
Routing:
- net +BATT: track 90.0 -> 69.6 mm
- net /liion/GAUGE_SRP: track 98.9 -> 79.6 mm
- net (no net): track 0.00 -> 8.28 mm
- net Net-(U10-XTAL2): track 0.00 -> 7.81 mm
- net Net-(U10-XTAL1): track 0.00 -> 7.75 mm
- net Net-(BT1A-+): track 4.54 -> 0.00 mm
- net Net-(BT8C-+): track 4.14 -> 0.00 mm
- net Net-(BT1B-+): track 4.14 -> 0.00 mm
- net GND: vias 0 -> 1

Commit message: WIP: schematics and layout improvements
Parts:
- removed D13, D14, D15: ORAGE, Mlab_D:LED_1206
- removed J5: HEADER_1x01, Mlab_Pin_Headers:Straight_1x01
- removed the R46 at (252.3, 139.0)
- removed the R47 at (255.2, 139.0)
- removed the R48 at (258.2, 139.0)
- removed the R50 at (178.7, 29.8)
- removed R51, R52, R53: 100R, Resistor_SMD:R_0805_2012Metric
- removed the R54 at (142.8, 90.9)
- removed the U9 at (121.7, 43.3)
- added C55: 100n, Capacitor_SMD:C_0805_2012Metric, B.Cu at (337.9, 122.9)
- added C56: 100nF, Capacitor_SMD:C_0805_2012Metric, B.Cu at (327.1, 131.9)
- added C57: 100n, Capacitor_SMD:C_0805_2012Metric, B.Cu at (337.9, 125.9)
- added C58: C_Small, Capacitor_SMD:C_0805_2012Metric, B.Cu at (337.9, 128.9)
- added C59: C_Small, Capacitor_SMD:C_0805_2012Metric, B.Cu at (337.9, 131.9)
- added C60: 100nF, Capacitor_SMD:C_0805_2012Metric, B.Cu at (337.9, 134.9)
- added C61: 1u, Capacitor_SMD:C_0805_2012Metric, B.Cu at (337.9, 137.9)
- added C62: 100nF, Capacitor_SMD:C_0805_2012Metric, B.Cu at (337.9, 140.9)
- added D16: ORANGE, LED_SMD:LED_1206_3216Metric, F.Cu at (217.7, 80.4)
- added D17: ORANGE, LED_SMD:LED_1206_3216Metric, B.Cu at (217.7, 89.4)
- added D18: ORANGE, LED_SMD:LED_1206_3216Metric, B.Cu at (217.7, 94.0)
- added D19: ORANGE, LED_SMD:LED_1206_3216Metric, B.Cu at (217.7, 98.7)
- added D6: RED, LED_SMD:LED_1206_3216Metric, F.Cu at (217.8, 87.7)
- added D7: GREEN, LED_SMD:LED_1206_3216Metric, F.Cu at (217.8, 92.3)
- added IC1: MAX14502AETL+, Mlab_IO:QFN40P500X500X80-41N, B.Cu at (172.7, 95.3)
- added J11: SD_Card-FPS009-4200-0, Mlab_CON:FPS009-4200-0, B.Cu at (216.1, 115.1)
- added L7: 100uH, Inductor_SMD:L_0805_2012Metric_Pad1.15x1.40mm_HandSolder, B.Cu at (322.5, 131.0)
- added NT1: NetTie_2, NetTie:NetTie-2_SMD_Pad0.5mm, B.Cu at (189.1, 56.9)
- added Q2: BC817-25, Package_TO_SOT_SMD:SOT-23-3, B.Cu at (319.6, 137.6)
- added Q3: BC817-25, Package_TO_SOT_SMD:SOT-23-3, F.Cu at (247.9, 115.6)
- added Q4: BC817-25, Package_TO_SOT_SMD:SOT-23-3, B.Cu at (326.7, 137.6)
- added Q5: BC817-25, Package_TO_SOT_SMD:SOT-23-3, F.Cu at (247.9, 120.1)
- added Q6: BC817-25, Package_TO_SOT_SMD:SOT-23-3, F.Cu at (247.9, 124.5)
- added R55: 10k, Resistor_SMD:R_0805_2012Metric, F.Cu at (246.3, 106.0)
- added R57: 100R, Resistor_SMD:R_0603_1608Metric, B.Cu at (345.6, 162.6)
- added R58: 1k, Resistor_SMD:R_0805_2012Metric, F.Cu at (246.3, 109.0)
- added R59: R, Resistor_SMD:R_0805_2012Metric, F.Cu at (246.3, 111.9)
- added R60: 10k, Resistor_SMD:R_0805_2012Metric, F.Cu at (250.7, 106.0)
- added R61: 1k, Resistor_SMD:R_0805_2012Metric, F.Cu at (250.7, 109.0)
- added R63: R, Resistor_SMD:R_0805_2012Metric, F.Cu at (250.7, 111.9)
- added R75: 1k, Resistor_SMD:R_0805_2012Metric, B.Cu at (327.1, 141.3)
- added R76: 6.19k, Resistor_SMD:R_0805_2012Metric, B.Cu at (177.2, 95.0)
- added R79: 100R, Resistor_SMD:R_0805_2012Metric, B.Cu at (177.2, 102.4)
- added R80: 100R, Resistor_SMD:R_0805_2012Metric, B.Cu at (177.2, 119.2)
- added R91: 100R, Resistor_SMD:R_0805_2012Metric, B.Cu at (177.2, 121.2)
- added R92: 100R, Resistor_SMD:R_0805_2012Metric, B.Cu at (177.2, 116.6)
- added R93: 100R, Resistor_SMD:R_0805_2012Metric, B.Cu at (177.2, 104.4)
- added R94: 100R, Resistor_SMD:R_0805_2012Metric, B.Cu at (177.2, 109.0)
- added U11: TPS22965-Q1, Package_SON:WSON-8-1EP_2x2mm_P0.5mm_EP0.9x1.6mm_ThermalVias, B.Cu at (318.0, 131.3)
- added U18: TS5A4594, Package_TO_SOT_SMD:SOT-23-5, B.Cu at (322.3, 123.6)
- added U19: ISL21080DIH309, Package_TO_SOT_SMD:SOT-23, B.Cu at (337.7, 144.7)
- C1: value 1u -> 1n
- C32: value 1nF -> 10uF
- C33: value 10uF -> 1nF; footprint Capacitor_SMD:C_0603_1608Metric -> Capacitor_SMD:C_0805_2012Metric
- C36: value 100nF -> 10uF; footprint Capacitor_SMD:C_0805_2012Metric -> Capacitor_SMD:C_0603_1608Metric
- D1, D2, D3, D4, D5: footprint Mlab_D:LED_1206_mill -> LED_SMD:LED_1206_3216Metric
- D10, D11, D12, D8, D9: footprint Mlab_D:LED_1206 -> LED_SMD:LED_1206_3216Metric; moved to F.Cu
- J2: value HEADER_2x04_PARALLEL -> 46436-9327; footprint Connector_PinHeader_2.54mm:PinHeader_2x04_P2.54mm_Vertical -> Mlab_CON:MOLEX_46436-9327; moved to F.Cu
- J3: value SD_Card-FPS009-4200-0 -> SM06B-GHS-TB; footprint Mlab_CON:FPS009-4200-0 -> Connector_JST:JST_GH_SM06B-GHS-TB_1x06-1MP_P1.25mm_Horizontal
- J4: value HEADER_1x01 -> SM04B-GHS-TB; footprint Mlab_Pin_Headers:Straight_1x01 -> Connector_JST:JST_GH_SM04B-GHS-TB_1x04-1MP_P1.25mm_Horizontal
- JP2, JP3: footprint Connector_PinHeader_2.54mm:PinHeader_1x02_P2.54mm_Vertical -> Jumper:SolderJumper-2_P1.3mm_Open_RoundedPad1.0x1.5mm
- JP4: renamed from JP6; footprint Connector_PinHeader_2.54mm:PinHeader_1x02_P2.54mm_Vertical -> Jumper:SolderJumper-2_P1.3mm_Open_RoundedPad1.0x1.5mm
- JP5: renamed from JP4; footprint Connector_PinHeader_2.54mm:PinHeader_1x02_P2.54mm_Vertical -> Jumper:SolderJumper-2_P1.3mm_Open_RoundedPad1.0x1.5mm
- JP6: renamed from JP5; footprint Connector_PinHeader_2.54mm:PinHeader_1x02_P2.54mm_Vertical -> Jumper:SolderJumper-2_P1.3mm_Open_RoundedPad1.0x1.5mm
- L3: value 100uH -> 1uH; footprint Inductor_SMD:L_0805_2012Metric_Pad1.15x1.40mm_HandSolder -> Inductor_SMD:L_1008_2520Metric
- R1, R4: value 4k7 -> 1k
- R2, R3: value 4k7 -> 10k
- R26, R27: value 270R -> R
- R41: renamed from R36; value R_Small -> R
- R42: renamed from R37; value R_Small -> R
- R46: renamed from R41; moved to F.Cu
- R47: renamed from R42; moved to F.Cu
- R48: renamed from R43; moved to F.Cu
- R49: renamed from R44; moved to F.Cu
- R5: value 4k7 -> 10k; moved to F.Cu
- R50: renamed from R45; moved to F.Cu
- R56: value 10R -> 100R; footprint Resistor_SMD:R_0805_2012Metric -> Resistor_SMD:R_0603_1608Metric
- R6: value 4k7 -> 1k; moved to F.Cu
- R7: value 4k7 -> R; moved to F.Cu
- TH1: value Thermistor_NTC -> 10k NTC
- U10: footprint Package_SO:SO-14_3.9x8.65mm_P1.27mm -> Package_SO:TSSOP-14_4.4x5mm_P0.65mm
- U9: renamed from U7; moved to B.Cu
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- renumbered C18 to C17, C17 to C18, C20 to C19, C21 to C20, C23 to C21, C19 to C22, C22 to C23, R14 to R12, R12 to R13, R13 to R14, R71 to R28, R72 to R29, R69 to R30, R70 to R31, R68 to R32, R28 to R33, R29 to R34, R30 to R35, R31 to R36, R32 to R37, R33 to R38, R34 to R39, R35 to R40, R38 to R43, R39 to R44, R40 to R45, R49 to R54, R55 to R62, R57 to R64, R58 to R65, R59 to R66, R60 to R67, R61 to R68, R62 to R69, R63 to R70, R64 to R71, R65 to R72, R66 to R73, R67 to R74, U10 to U12, U11 to U13, U12 to U14, IC1 to U3, U3 to U4, U4 to U5, U16 to U7, U6 to U8
Connections:
- C17 pad 1: Net-(U6-SRN) -> Net-(U8-SRP)
- C17 pad 2: Net-(U6-SRN) -> Net-(U8-SRN)
- C21 pad 1: Net-(U6-SRN) -> Net-(U8-SRP)
- C22 pad 1: Net-(U6-SRN) -> Net-(U8-SRN)
- C32 pad 1: Net-(U9-CT) -> 3v3_SD
- C33 pad 1: /mcu/SD_VDD -> Net-(U11-CT)
- C36 pad 1: /mcu/SD_VDD -> 3v3_SD
- C46 pad 1: unconnected-(C46-Pad1) -> +VSW
- C46 pad 2: unconnected-(C46-Pad2) -> GND
- C47 pad 1: unconnected-(C47-Pad1) -> +VSW
- C47 pad 2: unconnected-(C47-Pad2) -> GND
- C48 pad 1: unconnected-(C48-Pad1) -> +VSW
- C48 pad 2: unconnected-(C48-Pad2) -> GND
- C49 pad 1: unconnected-(C49-Pad1) -> +3.3V
- C49 pad 2: unconnected-(C49-Pad2) -> GND
- C5 pad 1: Net-(C5-Pad1) -> USB_POWER
- C50 pad 1: unconnected-(C50-Pad1) -> 3v3_EXT
- C50 pad 2: unconnected-(C50-Pad2) -> GND
- C51 pad 1: unconnected-(C51-Pad1) -> 5v_EXT
- C51 pad 2: unconnected-(C51-Pad2) -> GND
- C52 pad 1: unconnected-(C52-Pad1) -> +3.3V
- C52 pad 2: unconnected-(C52-Pad2) -> GND
- C53 pad 1: unconnected-(C53-Pad1) -> 3v3_EXT
- C53 pad 2: unconnected-(C53-Pad2) -> GND
- C54 pad 1: unconnected-(C54-Pad1) -> 5v_EXT
- C54 pad 2: unconnected-(C54-Pad2) -> GND
- J3 pad 1: Net-(J3-CD/DAT3) -> 5v_EXT
- J3 pad 2: Net-(J3-CMD) -> Net-(J3-Pad2)
- J3 pad 3: GND -> Net-(J3-Pad3)
- J3 pad 4: Net-(J3-VDD) -> unconnected-(J3-Pad4)
- J3 pad 5: Net-(J3-CLK) -> unconnected-(J3-Pad5)
- J4 pad 1: /mcu/PC3 -> 5v_EXT
- L3 pad 1: /mcu/SD_VDD -> 3v3_SD
- L3 pad 2: Net-(J3-VDD) -> Net-(U18-COM)
- Q1 pad 5: Net-(C5-Pad1) -> USB_POWER
- Q1 pad 6: Net-(C5-Pad1) -> USB_POWER
- Q1 pad 7: Net-(C5-Pad1) -> USB_POWER
- Q1 pad 8: Net-(C5-Pad1) -> USB_POWER
- R1 pad 1: VCC -> /ATTACH
- R1 pad 2: /ALERT -> Net-(Q4-B)
- R17 pad 1: Net-(C5-Pad1) -> USB_POWER
- R2 pad 1: VCC -> USB_CONNECTED
- R2 pad 2: /SIDE -> +3.3V
- R23 pad 2: /DP -> USB_FTDI_D+
- R24 pad 2: /DN -> USB_FTDI_D-
- R26 pad 2: GND -> /UART_TX_LED
- R27 pad 2: GND -> /UART_RX_LED
- R28 pad 1: /SCL_MCU -> SCL_MCU
- R29 pad 1: /SDA_MCU -> SDA_MCU
- R3 pad 1: VCC -> /liion/CH_STAT
- R3 pad 2: /ATTACH -> +3.3V
- R4 pad 1: VCC -> /liion/CH_STAT
- R4 pad 2: /GPIO -> Net-(Q2-B)
- R43 pad 2: Net-(U6-SRN) -> Net-(U8-SRP)
- R44 pad 2: Net-(U6-SRN) -> Net-(U8-SRN)
- R5 pad 1: VCC -> /mcu/LED_U1
- R5 pad 2: /PWR_OK2 -> +3.3V
- R56 pad 1: Net-(U10-(PCINT31/OC2A)PD7) -> EXT_TX
- R56 pad 2: POWER_ANALOG_3V3 -> Net-(J3-Pad2)
- R6 pad 1: VCC -> /mcu/LED_U1
- R6 pad 2: /PWR_OK3 -> Net-(Q3-B)
- R69 pad 1: unconnected-(R62-Pad1) -> +3.3V
- R69 pad 2: unconnected-(R62-Pad2) -> /sw_source/3v3i_FB
- R7 pad 1: VCC -> +3.3V
- R7 pad 2: /RESET -> Net-(D17-A)
- R70 pad 1: unconnected-(R63-Pad1) -> /sw_source/3v3i_FB
- R70 pad 2: unconnected-(R63-Pad2) -> GND
- R71 pad 1: unconnected-(R64-Pad1) -> 3v3_EXT
- R71 pad 2: unconnected-(R64-Pad2) -> /sw_source/3v3_FB
- R72 pad 1: unconnected-(R65-Pad1) -> /sw_source/3v3_FB
- R72 pad 2: unconnected-(R65-Pad2) -> GND
- R73 pad 1: unconnected-(R66-Pad1) -> 5v_EXT
- R73 pad 2: unconnected-(R66-Pad2) -> /sw_source/5v_FB
- R74 pad 1: unconnected-(R67-Pad1) -> /sw_source/5v_FB
- R74 pad 2: unconnected-(R67-Pad2) -> GND
- U10 pad 11: /liion/F -> unconnected-(U10-QF-Pad11)
- U10 pad 12: /liion/G -> unconnected-(U10-QG-Pad12)
- U10 pad 13: /liion/H -> unconnected-(U10-QH-Pad13)
- U12 pad 1: /mcu/MOSI -> /mcu/MOSI_MCU
- U12 pad 10: TX0 -> /MCU_TXD
- U12 pad 11: /mcu/RX1 -> EXT_RX
- U12 pad 12: /mcu/TX1 -> EXT_TX
- U12 pad 16: Net-(U10-(PCINT31/OC2A)PD7) -> unconnected-(U12-(PCINT31/OC2A)PD7-Pad16)
- U12 pad 19: /mcu/SCL -> SCL_MCU
- U12 pad 2: /mcu/MISO -> /mcu/MISO_MCU
- U12 pad 20: /mcu/SDA -> SDA_MCU
- U12 pad 21: unconnected-(U10-(PCINT18/TCK)PC2-Pad21) -> /mcu/SPI_MUX_EN
- U12 pad 22: /mcu/PC3 -> /mcu/SPI_MUX_SEL
- U12 pad 23: /mcu/PC4 -> unconnected-(U12-(PCINT20/TDO)PC4-Pad23)
- U12 pad 24: /mcu/PC5_D1 -> unconnected-(U12-(PCINT21/TDI)PC5-Pad24)
- U12 pad 25: /mcu/PC6_D2 -> EXT_C0
- U12 pad 26: /mcu/PC7_D3 -> EXT_C1
- U12 pad 3: /mcu/SCK -> /mcu/SCK_MCU
- U12 pad 35: unconnected-(U10-(PCINT2/ADC2)PA2-Pad35) -> EXT_A1
- U12 pad 36: /mcu/Voltage_Reference -> EXT_A0
- U12 pad 37: unconnected-(U10-(PCINT0/ADC0)PA0-Pad37) -> Net-(U12-(PCINT0/ADC0)PA0)
- U12 pad 40: unconnected-(U10-(PCINT8/T0/XCK)PB0-Pad40) -> EXT_B0
- U12 pad 41: unconnected-(U10-(PCINT9/CLKO/T1)PB1-Pad41) -> EXT_B1
- U12 pad 42: unconnected-(U10-(PCINT10/AIN0/INT2)PB2-Pad42) -> DET_I2C_EN
- U12 pad 43: /mcu/SD_PWR -> 3v3_SD_CTRL
- U12 pad 9: RX0 -> /MCU_RXD
- U13 pad 5: /mcu/SDA -> SDA_MCU
- U13 pad 6: /mcu/SCL -> SCL_MCU
- U14 pad 6: /mcu/SDA -> SDA_MCU
- U14 pad 7: /mcu/SCL -> SCL_MCU
- U2 pad 1: /DN -> USB_D-
- U2 pad 3: /DP -> USB_D+
- U2 pad 5: VBUS -> unconnected-(U2-VBUS-Pad5)
- U3 pad 10: /MCU_RXD -> /MCU_TXD
- U3 pad 11: /MCU_TXD -> /MCU_RXD
- U3 pad 26: unconnected-(IC1-VBUS_DET-Pad26) -> Net-(U3-VBUS_DET)
- U3 pad 27: unconnected-(IC1-DIO12-Pad27) -> /UART_RX_LED
- U3 pad 7: unconnected-(IC1-DIO0-Pad7) -> /UART_TX_LED
- U5 pad 1: /SCL_MCU -> SCL_MCU
- U5 pad 16: /SDA_MCU -> SDA_MCU
- U7 pad 2: OUT_SCL_I2C -> EXT_I2C_SCL
- U7 pad 7: OUT_SDA_I2C -> EXT_I2C_SDA
- U8 pad 10: Net-(U6-SRN) -> Net-(U8-SRN)
- U8 pad 9: Net-(U6-SRN) -> Net-(U8-SRP)
- U9 pad 18: CH_PWR -> USB_POWER
Routing:
- net SCL_MCU: track 0.00 -> 57.2 mm, vias 0 -> 2
- net SDA_MCU: track 0.00 -> 52.4 mm
- net /mcu/CDAT1_2: track 0.00 -> 35.2 mm, vias 0 -> 2
- net GND: track 0.00 -> 33.8 mm, vias 1 -> 2
- net /mcu/CDAT1_3: track 0.00 -> 30.5 mm, vias 0 -> 2
- net /mcu/CCMD1: track 0.00 -> 20.1 mm
- net /mcu/CDAT1_0: track 0.00 -> 17.3 mm, vias 0 -> 2
- net /mcu/CDAT1_1: track 0.00 -> 14.8 mm, vias 0 -> 2
- net /mcu/CCLK1: track 0.00 -> 12.2 mm
- net /SDA_USB: track 0.00 -> 10.5 mm, vias 0 -> 2
- net /SCL_USB: track 0.00 -> 10.4 mm
- net Net-(U5-~{RESET}): track 0.00 -> 5.75 mm
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- added copper zone on F.Cu, net +BATT
- added copper zone on B.Cu, net GND
- added copper zone on F.Cu, net GND
Other:
- board size 141.7 x 85.9 mm -> 162.1 x 85.9 mm

Commit message: wip layout, add datasheets
Parts:
- removed C30, C43: 100nF, Capacitor_SMD:C_0805_2012Metric
- removed J3: SM06B-GHS-TB, Connector_JST:JST_GH_SM06B-GHS-TB_1x06-1MP_P1.25mm_Horizontal
- removed J4: SM04B-GHS-TB, Connector_JST:JST_GH_SM04B-GHS-TB_1x04-1MP_P1.25mm_Horizontal
- removed R40: 1k, Resistor_SMD:R_0805_2012Metric
- removed R56, R57: 100R, Resistor_SMD:R_0603_1608Metric
- added R51: 1k, Resistor_SMD:R_0805_2012Metric, B.Cu at (258.6, 115.0)
- added R52: 500R, Resistor_SMD:R_0805_2012Metric, B.Cu at (258.6, 118.0)
- added R53: 250R, Resistor_SMD:R_0805_2012Metric, B.Cu at (258.6, 120.9)
- added R77: 1k, Resistor_SMD:R_0805_2012Metric, B.Cu at (258.6, 123.9)
- added U15: TPS631000DRLR, Package_TO_SOT_SMD:SOT-583-8, B.Cu at (147.6, 76.8)
- added U16: TPS631000DRLR, Package_TO_SOT_SMD:SOT-583-8, B.Cu at (128.0, 77.0)
- added U17: TPS631000DRLR, Package_TO_SOT_SMD:SOT-583-8, B.Cu at (107.5, 77.0)
- C14: value 0u1 -> 100n
- Q3, Q5, Q6, R5, R55, R58, R59, R6, R60, R61, R63, R7: moved to B.Cu
- moved U19 255.8 mm to (84.0, 112.2)
- moved U7 217.5 mm to (105.3, 115.0), turned to 90 degrees
- moved R73 171.0 mm to (105.0, 77.3), turned to -90 degrees
- moved R74 171.0 mm to (105.0, 80.7), turned to -90 degrees
- moved JP5 166.3 mm to (107.7, 80.1), turned to 90 degrees
- moved L6 164.3 mm to (107.5, 74.3)
- moved R66 163.7 mm to (110.5, 78.5), turned to 90 degrees
- moved C51 161.7 mm to (104.5, 73.9), turned to 90 degrees
- moved R24 160.1 mm to (161.7, 103.0), turned to 90 degrees
- moved C48 159.9 mm to (110.5, 75.1), turned to 90 degrees
- moved R23 159.0 mm to (163.7, 103.0), turned to 90 degrees
- moved C54 158.4 mm to (103.0, 77.3), turned to -90 degrees
- moved U11 153.5 mm to (165.1, 117.5)
- moved U18 153.4 mm to (169.0, 117.3)
- moved L7 152.7 mm to (170.8, 112.9), turned to 0 degrees
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Connections:
- IC1 pad 2: SCL_MCU -> SCL_I2C
- IC1 pad 29: /mcu/SCK_SD -> 3v3_SD
- IC1 pad 3: SDA_MCU -> SDA_I2C
- J2 pad C1: unconnected-(J2-PadC1) -> EXT_I2C_SCL
- J2 pad C2: unconnected-(J2-PadC2) -> EXT_I2C_SDA
- J2 pad E1: EXT_C1 -> EXT_C0
- J2 pad E2: EXT_C0 -> EXT_C1
- J2 pad E5: EXT_B1 -> EXT_B0
- J2 pad E6: EXT_B0 -> EXT_B1
- J6 pad 1: /mcu/MISO -> /mcu/MISO_MCU
- J6 pad 3: /mcu/SCK -> /mcu/SCK_MCU
- J6 pad 4: /mcu/MOSI -> /mcu/MOSI_MCU
- R34 pad 1: SCL_I2C -> SDA_I2C
- R35 pad 1: SDA_I2C -> SCL_I2C
- U12 pad 13: unconnected-(U12-(PCINT28/XCK1/OC1B)PD4-Pad13) -> /mcu/LED_U1
- U12 pad 14: unconnected-(U12-(PCINT294/OC1A)PD5-Pad14) -> /mcu/LED_U2
- U12 pad 15: unconnected-(U12-(PCINT30/OC2B/ICP)PD6-Pad15) -> /mcu/LED_U3
- U12 pad 30: unconnected-(U12-(PCINT7/ADC7)PA7-Pad30) -> /mcu/BTN_USER_B
- U12 pad 31: unconnected-(U12-(PCINT6/ADC6)PA6-Pad31) -> /mcu/BTN_USER_A
- U13 pad 5: SDA_MCU -> SDA_I2C
- U13 pad 6: SCL_MCU -> SCL_I2C
- U14 pad 6: SDA_MCU -> SDA_I2C
- U14 pad 7: SCL_MCU -> SCL_I2C
- U18 pad 2: VCC -> +3.3V
- U18 pad 5: VCC -> +3.3V
- U8 pad 2: /liion/GAUGE_BTN_B -> /liion/GAUGE_BTN_IN
Routing:
- net +3.3V: track 0.00 -> 122.7 mm, vias 0 -> 4
- net SDA_I2C: track 0.00 -> 88.8 mm
- net SCL_I2C: track 0.00 -> 84.0 mm, vias 0 -> 2
- net 3v3_EXT: track 0.00 -> 82.0 mm
- net +VSW: track 0.00 -> 77.6 mm, vias 0 -> 6
- net 5v_EXT: track 0.00 -> 54.8 mm
- net +BATT: track 69.6 -> 118.9 mm
- net 3v3_SD_CTRL: track 0.00 -> 48.1 mm
- net /mcu/CS_SD: track 0.00 -> 45.9 mm
- net USB_D+: track 0.00 -> 41.7 mm
- net USB_D-: track 0.00 -> 38.4 mm
- net /MCU_TXD: track 0.00 -> 36.2 mm, vias 0 -> 2
- net /MCU_RXD: track 0.00 -> 35.5 mm, vias 0 -> 2
- net EXT_RX: track 0.00 -> 31.4 mm, vias 0 -> 2
- net GND: track 33.8 -> 64.7 mm, vias 2 -> 25
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- added copper zone on B.Cu, net +3.3V
- added copper zone on B.Cu, net +VSW
- added copper zone on B.Cu, net 3v3_EXT
- added copper zone on B.Cu, net 5v_EXT
