File: hw/sch_pcb/LION5CELL01.kicad_pcb (KiCad board)
At the start: 2 copper layers, 162.1 x 85.9 mm, 222 parts, among them IC1 MAX14502AETL+, J1 USBC_USB4105-GF-A, J11 SD_Card-FPS009-4200-0, J2 46436-9327, J6 HEADER_2x03, Q1 IRF9317TRPBF, Q2 BC817-25, Q3 BC817-25, Q4 BC817-25, Q5 BC817-25, Q6 BC817-25, U1 STUSB4500QTR, U10 SN74HC164D, U11 TPS22965-Q1, U12 ATMEGA1284P-AU, U13 AT24CS64-SSHM, U14 PCF85263A, U15 TPS631000DRLR, U16 TPS631000DRLR, U17 TPS631000DRLR, U18 TS5A4594, U19 ISL21080DIH309, U2 USBLC6-2SC6, U3 FT260Q-T, U4 SHT35-DIS, U5 PCA9541ABS/01, U7 TCA4307, U8 BQ34Z100, U9 BQ25628E, Y1 8 MHz, Y2 ABS07-120-32.768KHZ-T

Commit message: WIP
Parts:
- removed C2, C3, C4: 1u, Capacitor_SMD:C_0805_2012Metric
- removed C32: 10uF, Capacitor_SMD:C_0805_2012Metric
- removed L1: DE1205-10, Mlab_L:DE1205-10
- removed U1: STUSB4500QTR, Package_DFN_QFN:QFN-24-1EP_4x4mm_P0.5mm_EP2.7x2.7mm
- removed U18: TS5A4594, Package_TO_SOT_SMD:SOT-23-5
- added C29: 1uF, Capacitor_SMD:C_0805_2012Metric, B.Cu at (167.8, 118.7)
- added R40: R_Small, Resistor_SMD:R_0805_2012Metric, F.Cu at (159.2, 50.2)
- added R56: 1k, Resistor_SMD:R_0805_2012Metric, F.Cu at (159.2, 53.2)
- added R57: 1k, Resistor_SMD:R_0805_2012Metric, F.Cu at (159.2, 56.1)
- added R78: R_Small, Resistor_SMD:R_0805_2012Metric, F.Cu at (159.2, 59.1)
- L3: value 1uH -> 1uH - DFE252012P-1R0M=P2
- R75: value 1k -> 5k1 (cca)
- U9: footprint Package_DFN_QFN:Texas_S-PWQFN-N20 -> Mlab_IO:Texas_S-WQFN-HR-18
- moved C33 105.0 mm to (167.2, 112.9)
- moved L3 31.8 mm to (182.8, 84.3), turned to 90 degrees
- moved U11 3.65 mm to (168.3, 115.7), turned to 90 degrees
Connections:
- IC1 pad 28: USB_CONNECTED -> Net-(IC1-KVBUS)
- IC1 pad 29: 3v3_SD -> /mcu/SCK_SD
- J1 pad A5: Net-(J1-CC1) -> unconnected-(J1-CC1-PadA5)
- J1 pad B5: Net-(J1-CC2) -> unconnected-(J1-CC2-PadB5)
- L3 pad 1: 3v3_SD -> Net-(U9-SW)
- L3 pad 2: Net-(U18-COM) -> +VSW
- R75 pad 1: USB_CONNECTED -> VBUS
- U2 pad 5: unconnected-(U2-VBUS-Pad5) -> VBUS
Routing:
- net unconnected-(J1-CC2-PadB5): track 0.00 -> 17.5 mm, vias 0 -> 2
- net Net-(J1-CC2): track 17.5 -> 0.00 mm, vias 2 -> 0
- net unconnected-(J1-CC1-PadA5): track 0.00 -> 11.0 mm
- net Net-(J1-CC1): track 11.0 -> 0.00 mm
- net +3.3V: track 122.7 -> 128.6 mm
- net Net-(U9-SW): track 10.4 -> 5.21 mm
- net Net-(L7-Pad1): track 0.00 -> 2.80 mm
- net Net-(U11-CT): track 0.00 -> 1.89 mm
- net 3v3_SD_CTRL: track 48.1 -> 48.8 mm, vias 0 -> 1

Commit message: WIP, layout improvement
Parts:
- removed C5: 100n, Capacitor_SMD:C_0805_2012Metric
- removed C6: 4u7, Capacitor_SMD:C_0805_2012Metric
- removed D1: GREEN, LED_SMD:LED_1206_3216Metric
- removed D2, D5: RED, LED_SMD:LED_1206_3216Metric
- removed D3: YELLOW, LED_SMD:LED_1206_3216Metric
- removed D4: BLUE, LED_SMD:LED_1206_3216Metric
- removed Q4: BC817-25, Package_TO_SOT_SMD:SOT-23-3
- removed R1, R17: 1k, Resistor_SMD:R_0805_2012Metric
- removed R10, R12, R8, R9: 62R, Resistor_SMD:R_0805_2012Metric
- removed R11: 10R, Resistor_SMD:R_0805_2012Metric
- removed R16: 100R, Resistor_SMD:R_0805_2012Metric
- removed R2, R20, R21, R22: 10k, Resistor_SMD:R_0805_2012Metric
- removed R38: R, Resistor_SMD:R_0805_2012Metric
- added D13: GREEN, LED_SMD:LED_1206_3216Metric, B.Cu at (63.5, 80.3)
- added IC2: TMUX1574DYYR, Mlab_IO:SOT-23-16 THIN, B.Cu at (137.4, 100.7)
- Q1: value IRF9317TRPBF -> BC817-25; footprint Package_SO:SOIC-8_3.9x4.9mm_P1.27mm -> Package_TO_SOT_SMD:SOT-23-3
- R13: value 1k -> 10k
- R14: value 100k -> 1k
- R15: value 20k -> R
- R18, R19: value 10k -> 1K
- R28, R29, R30, R31, R34, R35: value 10k -> 1k
- moved R13 191.3 mm to (68.5, 80.1)
- moved Q1 135.1 mm to (63.7, 84.2)
- moved R14 126.1 mm to (68.5, 83.0)
- moved R15 125.5 mm to (68.5, 86.0)
- moved U10 3.29 mm to (206.0, 138.4), turned to 0 degrees
- moved JP1 0.30 mm to (139.4, 94.9)
- moved R25 0.30 mm to (137.1, 94.8)
Connections:
- J1 pad A5: unconnected-(J1-CC1-PadA5) -> Net-(J1-CC1)
- J1 pad B5: unconnected-(J1-CC2-PadB5) -> Net-(J1-CC2)
- Q1 pad 1: VBUS -> Net-(D13-K)
- Q1 pad 2: VBUS -> Net-(Q1-B)
- Q1 pad 3: VBUS -> GND
- R13 pad 1: VBUS -> /liion/CH_PG
- R13 pad 2: /VBUS_VS_DISCH -> +3.3V
- R14 pad 1: VBUS -> /liion/CH_PG
- R14 pad 2: Net-(Q1-G) -> Net-(Q1-B)
- R15 pad 1: Net-(Q1-G) -> +3.3V
- R15 pad 2: /VBUS_EN_SINK -> Net-(D13-A)
- R37 pad 2: /liion/ch_ilim -> GND
- TP3 pad 1: Net-(U9-~{PG}) -> /liion/CH_PG
- U12 pad 10: /MCU_TXD -> /mcu/MCU_TX0
- U12 pad 9: /MCU_RXD -> /mcu/MCU_RX0
- U3 pad 1: Net-(U3-DEBUGGER) -> +3.3V
- U3 pad 2: Net-(U3-STEST_RSTN) -> +3.3V
- U3 pad 3: Net-(U3-RESETN) -> +3.3V
- U9 pad 18: USB_POWER -> VBUS
- U9 pad 3: Net-(U9-~{PG}) -> /liion/CH_PG
Routing:
- net /mcu/SCK_SD: track 0.00 -> 53.9 mm, vias 0 -> 2
- net /mcu/MOSI_SD: track 0.00 -> 48.7 mm, vias 0 -> 2
- net 3v3_SD_CTRL: track 48.8 -> 0.65 mm
- net /mcu/MISO_SD: track 0.00 -> 40.9 mm, vias 0 -> 2
- net +BATT: track 118.9 -> 153.2 mm, vias 0 -> 3
- net +3.3V: track 128.6 -> 146.8 mm, vias 4 -> 5
- net unconnected-(J1-CC2-PadB5): track 17.5 -> 0.00 mm, vias 2 -> 0
- net Net-(J1-CC2): track 0.00 -> 17.5 mm, vias 0 -> 2
- net /mcu/MISO_MCU: track 6.56 -> 19.7 mm, vias 0 -> 2
- net /mcu/CS_SD: track 45.9 -> 59.0 mm, vias 0 -> 2
- net unconnected-(J1-CC1-PadA5): track 11.0 -> 0.00 mm
- net Net-(J1-CC1): track 0.00 -> 11.0 mm
- net /mcu/MOSI_MCU: track 10.7 -> 21.2 mm
- net /mcu/SCK_MCU: track 12.2 -> 20.2 mm, vias 2 -> 3
- net Net-(U9-~{PG}): track 7.20 -> 0.00 mm
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
Commit message: wip, layout progress
Parts:
- removed C62: 100nF, Capacitor_SMD:C_0805_2012Metric
- removed R36: 47k, Resistor_SMD:R_0805_2012Metric
- removed U19: ISL21080DIH309, Package_TO_SOT_SMD:SOT-23
- added D1: ORAGE, Mlab_D:SMD_LED_RIGHT_KINGBRIGHT_1605, F.Cu at (217.5, 100.8)
- added D2: ORAGE, Mlab_D:SMD_LED_RIGHT_KINGBRIGHT_1605, F.Cu at (217.5, 103.6)
- added D3: ORAGE, Mlab_D:SMD_LED_RIGHT_KINGBRIGHT_1605, F.Cu at (217.5, 106.3)
- added NT2: NetTie_2, NetTie:NetTie-2_SMD_Pad0.5mm, B.Cu at (164.3, 69.0)
- added R1: R_Small, Resistor_SMD:R_0805_2012Metric, B.Cu at (206.8, 74.9)
- added R10: 270R, Resistor_SMD:R_0805_2012Metric, F.Cu at (215.1, 107.1)
- added R2: R_Small, Resistor_SMD:R_0805_2012Metric, B.Cu at (212.1, 86.4)
- added R8: 270R, Resistor_SMD:R_0805_2012Metric, F.Cu at (215.2, 101.5)
- added R9: 270R, Resistor_SMD:R_0805_2012Metric, F.Cu at (215.1, 104.3)
- BT1, BT2: value 3xBATT -> BATT
- D10, D11, D12, D16, D6, D7, D8, D9: footprint LED_SMD:LED_1206_3216Metric -> Mlab_D:SMD_LED_RIGHT_KINGBRIGHT_1605
- D13, D17, D18, D19: footprint LED_SMD:LED_1206_3216Metric -> Mlab_D:SMD_LED_RIGHT_KINGBRIGHT_1605; moved to F.Cu
- R39, TH1: moved to F.Cu
- R40, R56, R57, R78: moved to B.Cu
- R45: footprint Resistor_SMD:R_0805_2012Metric -> Resistor_SMD:R_2512_6332Metric
- moved Q1 191.0 mm to (236.4, 165.8)
- moved R15 191.0 mm to (241.2, 167.6)
- moved R14 183.4 mm to (231.8, 166.6)
- moved R13 182.9 mm to (237.8, 149.4)
- moved D13 163.3 mm to (217.6, 134.2), turned to -90 degrees
- moved R32 161.6 mm to (108.2, 114.7), turned to 90 degrees
- moved R4 123.2 mm to (241.9, 157.6)
- moved R54 114.0 mm to (238.4, 161.2)
- moved C26 113.3 mm to (199.4, 98.3), turned to 180 degrees
- moved C11 112.4 mm to (165.0, 107.1), turned to -90 degrees
- moved C1 82.9 mm to (206.8, 77.0)
- moved R35 78.1 mm to (134.3, 119.3), turned to -45 degrees
- moved TH1 77.7 mm to (172.5, 89.0), turned to 0 degrees
- moved R34 76.6 mm to (134.8, 117.0), turned to -45 degrees
- moved D16 51.1 mm to (217.6, 131.5)
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Connections:
- BT1 pad 1-: /liion/GAUGE_SRP -> Net-(BT1A--)
- BT1 pad 2-: /liion/GAUGE_SRP -> Net-(BT1A--)
- BT2 pad 1-: /liion/GAUGE_SRP -> Net-(BT1A--)
- BT2 pad 2-: /liion/GAUGE_SRP -> Net-(BT1A--)
- BT2 pad 3-: /liion/GAUGE_SRP -> Net-(BT1A--)
- NT1 pad 1: GND -> /liion/GAUGE_SRN
- NT1 pad 2: GNDA -> GND
- R44 pad 1: GND -> /liion/GAUGE_SRN
- R45 pad 1: /liion/GAUGE_SRP -> Net-(BT1A--)
- U10 pad 11: unconnected-(U10-QF-Pad11) -> /liion/F
- U10 pad 12: unconnected-(U10-QG-Pad12) -> /liion/G
- U10 pad 13: unconnected-(U10-QH-Pad13) -> /liion/H
- U12 pad 21: /mcu/SPI_MUX_EN -> /mcu/SPI_MUX_SEL
- U12 pad 22: /mcu/SPI_MUX_SEL -> /mcu/SPI_MUX_EN
- U12 pad 35: EXT_A1 -> unconnected-(U12-(PCINT2/ADC2)PA2-Pad35)
- U12 pad 36: EXT_A0 -> EXT_A1
- U12 pad 37: Net-(U12-(PCINT0/ADC0)PA0) -> EXT_A0
- U8 pad 12: /liion/CHARGE_CTRL -> unconnected-(U8-P5/HDQ-Pad12)
Routing:
- net SDA_I2C: track 88.8 -> 172.4 mm, vias 0 -> 4
- net /liion/GAUGE_SRP: track 85.0 -> 1.98 mm
- net Net-(BT1A--): track 0.00 -> 83.0 mm
- net SCL_I2C: track 84.0 -> 163.3 mm, vias 2 -> 8
- net EXT_MISO: track 0.00 -> 44.8 mm, vias 0 -> 1
- net EXT_MOSI: track 0.00 -> 44.4 mm, vias 0 -> 1
- net EXT_SCK: track 0.00 -> 42.5 mm, vias 0 -> 1
- net +3.3V: track 146.8 -> 185.8 mm, vias 5 -> 9
- net VBUS: track 15.2 -> 52.3 mm, vias 3 -> 5
- net SDA_MCU: track 74.8 -> 41.3 mm, vias 2 -> 0
- net /mcu/SPI_MUX_EN: track 0.00 -> 32.5 mm, vias 0 -> 2
- net SCL_MCU: track 72.2 -> 43.0 mm, vias 2 -> 0
- net /mcu/SPI_MUX_SEL: track 0.00 -> 28.5 mm, vias 0 -> 2
- net +3V3: track 0.00 -> 28.4 mm
- net /liion/H: track 0.00 -> 15.9 mm, vias 0 -> 1
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
Commit message: wip, layout improvements
Parts:
- added R11: 10k, Resistor_SMD:R_0805_2012Metric, B.Cu at (141.7, 94.9)
- added REF**: MountingHole_2.2mm_M2, MountingHole:MountingHole_2.2mm_M2, F.Cu at (215.9, 116.0)
- added SW1: SW_Push, Mlab_SW:SKRT, F.Cu at (211.7, 119.8)
- added SW2: MCU_RST, Mlab_SW:KMT031 NGJ LHS C&K, B.Cu at (124.8, 93.2)
- added SW3: SW_Push, Mlab_SW:SKRT, F.Cu at (211.6, 112.4)
- added SW4: SW_Push, Mlab_SW:KMT031 NGJ LHS C&K, B.Cu at (117.6, 93.2)
- D1, D12, D2, D3: value ORAGE -> GREEN
- D13, D16: moved to B.Cu
- D8, D9: value ORAGE -> RED
- moved R40 81.6 mm to (170.1, 129.9)
- moved R78 60.2 mm to (113.0, 97.6)
- moved D13 47.4 mm to (217.5, 86.9), turned to 90 degrees
- moved D16 39.0 mm to (217.5, 92.5), turned to 90 degrees
- moved D17 3.98 mm to (217.6, 124.5)
- moved D18 3.65 mm to (217.6, 127.3)
- moved D7 3.40 mm to (217.6, 77.9)
- moved D19 3.33 mm to (217.6, 130.1)
- moved D6 3.20 mm to (217.5, 81.8)
- moved J1 0.33 mm to (216.7, 79.7)
- moved U2 0.33 mm to (207.6, 79.7)
- moved C1 0.33 mm to (207.0, 76.8)
- moved R1 0.33 mm to (207.0, 74.7)
Connections:
- net /mcu/CCLK1 renamed /mcu/CCLK
- net /mcu/CCMD1 renamed /mcu/CCMD
- net /mcu/CDAT1_0 renamed /mcu/CDAT0
- net /mcu/CDAT1_1 renamed /mcu/CDAT1
- net /mcu/CDAT1_2 renamed /mcu/CDAT2
- net /mcu/CDAT1_3 renamed /mcu/CDAT3
- net /mcu/SCK_MCU renamed /mcu/SCLK_MCU
- net /mcu/SCK_SD renamed /mcu/SCLK_SD
- net EXT_SCK renamed EXT_SCLK
- IC2 pad 15: /mcu/SPI_MUX_EN -> GND
- U12 pad 22: /mcu/SPI_MUX_EN -> 3v3_SD_CTRL
- U12 pad 43: 3v3_SD_CTRL -> unconnected-(U12-(PCINT11/AIN1/OC0)PB3-Pad43)
Routing:
- net 3v3_SD_CTRL: track 0.65 -> 58.3 mm, vias 1 -> 4
- net +3.3V: track 185.8 -> 223.8 mm
- net /mcu/SPI_MUX_EN: track 32.5 -> 0.00 mm, vias 2 -> 0
- net /mcu/BTN_USER_B: track 0.00 -> 17.2 mm, vias 0 -> 2
- net /mcu/RST#_P: track 21.6 -> 30.8 mm, vias 2 -> 3
- net /mcu/SPI_MUX_SEL: track 28.5 -> 33.5 mm
- net /mcu/CDAT3: track 27.6 -> 25.6 mm
- net /mcu/CS_SD: track 58.7 -> 60.3 mm
- net GND: track 60.6 -> 62.1 mm, vias 30 -> 32
- net /mcu/MISO_MCU: track 21.9 -> 23.2 mm
- net /liion/A: track 14.0 -> 13.3 mm
- net /liion/B: track 13.8 -> 13.3 mm
Other:
- board size 162.1 x 85.9 mm -> 161.6 x 85.9 mm
