File: hw/sch_pcb/LION5CELL01.kicad_pcb (KiCad board)
At the start: 2 copper layers, 161.6 x 85.9 mm, 213 parts, among them IC1 MAX14502AETL+, IC2 TMUX1574DYYR, J1 USBC_USB4105-GF-A, J11 SD_Card-FPS009-4200-0, J2 46436-9327, J6 HEADER_2x03, Q1 BC817-25, Q2 BC817-25, Q3 BC817-25, Q5 BC817-25, Q6 BC817-25, SW1 SW_Push, SW2 MCU_RST, SW3 SW_Push, SW4 SW_Push, U10 SN74HC164D, U11 TPS22965-Q1, U12 ATMEGA1284P-AU, U13 AT24CS64-SSHM, U14 PCF85263A, U15 TPS631000DRLR, U16 TPS631000DRLR, U17 TPS631000DRLR, U2 USBLC6-2SC6, U3 FT260Q-T, U4 SHT35-DIS, U5 PCA9541ABS/01, U7 TCA4307, U8 BQ34Z100, U9 BQ25628E, Y1 8 MHz, Y2 ABS07-120-32.768KHZ-T

Commit message: wip: layout
Parts:
- moved R18 120.9 mm to (158.3, 115.7), turned to 90 degrees
- moved C8 118.2 mm to (163.0, 115.0), turned to 0 degrees
- moved R19 117.9 mm to (160.3, 115.7), turned to 90 degrees
- moved C9 116.6 mm to (163.0, 112.9), turned to 0 degrees
- moved C12 98.9 mm to (92.2, 136.0)
- moved C20 88.9 mm to (167.5, 89.5)
- moved C16 84.1 mm to (165.5, 89.5)
- moved C18 76.1 mm to (163.0, 83.5), turned to 90 degrees
- moved R40 64.6 mm to (113.0, 99.6)
- moved R58 55.4 mm to (204.5, 145.3)
- moved R6 55.4 mm to (208.9, 145.3)
- moved R61 55.4 mm to (200.1, 145.3)
- moved R5 55.4 mm to (208.9, 142.3)
- moved R55 55.4 mm to (204.5, 142.3)
- moved R7 49.8 mm to (206.1, 134.1), turned to -90 degrees
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Routing:
- net +3.3V: track 223.8 -> 308.5 mm, vias 9 -> 11
- net +BATT: track 153.2 -> 230.8 mm, vias 3 -> 7
- net /liion/CH_BTN: track 0.00 -> 49.9 mm, vias 0 -> 1
- net /liion/P2: track 0.00 -> 47.6 mm, vias 0 -> 2
- net /liion/P1: track 0.00 -> 45.4 mm, vias 0 -> 2
- net Net-(U8-P6/TS): track 0.00 -> 33.5 mm, vias 0 -> 1
- net +VSW: track 73.7 -> 106.7 mm, vias 6 -> 7
- net Net-(U8-REG25): track 0.00 -> 28.1 mm, vias 0 -> 1
- net Net-(U9-TS): track 0.00 -> 25.3 mm, vias 0 -> 2
- net EXT_A0: track 0.00 -> 24.7 mm, vias 0 -> 1
- net EXT_A1: track 0.00 -> 23.3 mm, vias 0 -> 1
- net Net-(IC1-KVBUS): track 7.15 -> 17.8 mm, vias 1 -> 2
- net +3V3: track 28.4 -> 37.2 mm
- net /liion/CH_STAT: track 0.00 -> 6.65 mm
- net Net-(U3-DCNF1): track 0.00 -> 5.18 mm
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
Commit message: Wip, layout
Parts:
- removed the C31 at (48.8, 108.2)
- removed the C34 at (51.8, 112.9)
- removed the C37 at (52.9, 103.6)
- removed the C39 at (44.8, 98.2)
- removed C58: C_Small, Capacitor_SMD:C_0805_2012Metric
- removed the C7 at (274.5, 72.8)
- removed the L2 at (39.4, 107.0)
- removed the R13 at (237.8, 149.4)
- removed the R27 at (165.4, 109.8)
- removed the R3 at (186.4, 87.1)
- removed the R5 at (208.9, 142.3)
- removed the R51 at (258.6, 115.0)
- removed the R55 at (204.5, 142.3)
- removed the R60 at (241.9, 106.0)
- removed REF**: MountingHole_2.2mm_M2, MountingHole:MountingHole_2.2mm_M2
- removed the TP1 at (257.3, 70.0)
- removed TP3: CH_PG, TestPoint:TestPoint_Pad_D1.5mm
- removed TP4: CH_STAT, TestPoint:TestPoint_Pad_D1.5mm
- removed TP5: CH_INT, TestPoint:TestPoint_Pad_D1.5mm
- added Q3: BC807-25, Package_TO_SOT_SMD:SOT-23-3, B.Cu at (162.3, 87.6)
- added Q7: BC817-25, Package_TO_SOT_SMD:SOT-23-3, B.Cu at (174.7, 125.9)
- added R11: R, Resistor_SMD:R_0805_2012Metric, F.Cu at (215.8, 78.0)
- added R47: 1k, Resistor_SMD:R_0805_2012Metric, B.Cu at (175.4, 129.8)
- C1: renamed from C8; value 0u1 -> 100n
- C10: renamed from C17; value 100nF -> 100n
- C13: renamed from C21; value 100nF -> 100n
- C14: renamed from C22; value 100nF -> 100n
- C15: renamed from C18; value 1uF -> 1u
- C20: renamed from C26; value 100nF -> 100n
- C21: renamed from C27; value 100nF -> 100n
- C22: renamed from C28; value 100nF -> 100n
- C25: renamed from C60; value 100nF -> 100n
- C31: renamed from C42; value 100nF -> 100n
- C32: renamed from C44; value 100nF -> 100n
- C33: renamed from C45; value 100nF -> 100n
- C4: renamed from C10; value 100nF -> 100n
- C44 (x2): renamed from C29; value 1uF -> 1u
- C46: renamed from C36; footprint Capacitor_SMD:C_0603_1608Metric -> Capacitor_SMD:C_0805_2012Metric
- C47: renamed from C56; value 100nF -> 100n
- C5: renamed from C11; value 100nF -> 100n
- C6: renamed from C12; value 100nF -> 100n
- C9: renamed from C16; value 100nF -> 100n
- R1: renamed from R18; value 1K -> 1k
- R10: renamed from R26; moved to F.Cu
- R2: renamed from R19; value 1K -> 1k
- R23: renamed from R39; value 10K NTC -> 10k NTC
- moved C25 117.6 mm to (166.4, 98.9), turned to 90 degrees
- moved C34 114.3 mm to (169.4, 104.3), turned to -90 degrees
- moved C26 111.6 mm to (171.4, 104.6), turned to -90 degrees
- moved R5 106.6 mm to (166.2, 108.3)
- moved R22 104.1 mm to (192.2, 75.7), turned to 90 degrees
- moved C44 103.7 mm to (169.7, 118.3), turned to 0 degrees
- moved Q2 103.5 mm to (193.0, 71.9), turned to 90 degrees
- moved C23 103.5 mm to (179.5, 100.2), turned to -90 degrees
- moved R21 99.1 mm to (188.3, 75.7), turned to 90 degrees
- moved R20 98.4 mm to (194.2, 75.7), turned to 90 degrees
- moved Q1 97.1 mm to (189.5, 71.8), turned to 90 degrees
- moved C24 96.9 mm to (186.2, 105.8)
- moved R19 96.9 mm to (190.2, 75.7), turned to 90 degrees
- moved R30 94.2 mm to (169.8, 89.6), turned to -90 degrees
- moved R29 92.8 mm to (171.8, 85.2), turned to 90 degrees
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- renumbered C15 to C11, C20 to C12, C19 to C16, C23 to C17, C24 to C18, C25 to C19, C9 to C2, C55 to C23, C59 to C24, C57 to C26, C40 to C27, C35 to C28, C41 to C29, C1 to C3, C38 to C30, C61 to C34, C46 to C35, C47 to C36, C48 to C37, C49 to C38, C50 to C39, C51 to C40, C52 to C41, C53 to C42, C54 to C43, C33 to C45, C13 to C7, C14 to C8, D6 to D1, D9 to D11, D8 to D12, D17 to D13, D19 to D14, D18 to D15, D7 to D2, D16 to D3, D13 to D4, D3 to D5, D2 to D6, D1 to D7, D12 to D8, D11 to D9, J11 to J3, J6 to J4, L3 to L1, L4 to L2, L5 to L3, L6 to L4, L7 to L5, NT2 to NT1, NT1 to NT2, Q2 to Q1, Q1 to Q2, Q3 to Q4, Q6 to Q5, Q5 to Q6, R28 to R12, R29 to R13, R30 to R14, R31 to R15, R33 to R16, R34 to R17, R35 to R18, R4 to R19, R14 to R20, R54 to R21, R15 to R22, R37 to R24, R43 to R25, R44 to R26, R41 to R27, R42 to R28, R52 to R29, R2 to R3, R53 to R30, R77 to R31, R45 to R32, R46 to R33, R47 to R34, R48 to R35, R49 to R36, R50 to R37, R8 to R38, R9 to R39, R1 to R4, R10 to R40, R6 to R41, R61 to R42, R7 to R43, R63 to R44, R76 to R45, R58 to R46, R79 to R48, R93 to R49, R75 to R5, R94 to R50, R92 to R51, R80 to R52, R91 to R53, R59 to R54, R56 to R55, R57 to R56, R62 to R57, R40 to R58, R78 to R59, R23 to R6, R11 to R60, R64 to R61, R65 to R62, R66 to R63, R67 to R64, R68 to R65, R69 to R66, R70 to R67, R71 to R68, R72 to R69, R24 to R7, R73 to R70, R74 to R71, R25 to R8, R32 to R9, SW3 to SW1, SW1 to SW2, SW4 to SW3, SW2 to SW4, TP2 to TP1, U3 to U1, U12 to U10, U13 to U11, U14 to U12, U15 to U13, U16 to U14, U17 to U15, U11 to U16, U7 to U3, U8 to U7, U9 to U8, U10 to U9
Connections:
- C20 pad 1: +3V3 -> +3.3V
- C9 pad 1: +3V3 -> +3.3V
- D10 pad 1: +3V3 -> Net-(D10-K)
- D10 pad 2: Net-(D10-K) -> +3.3V
- D11 pad 1: +3V3 -> Net-(D11-K)
- D11 pad 2: Net-(D9-K) -> +3.3V
- D12 pad 1: +3V3 -> Net-(D12-K)
- D12 pad 2: Net-(D8-K) -> +3.3V
- D13 pad 1: Net-(D17-K) -> Net-(D13-K)
- D13 pad 2: Net-(D17-A) -> +3.3V
- D14 pad 1: Net-(D19-K) -> Net-(D14-K)
- D14 pad 2: Net-(D19-A) -> +3.3V
- D15 pad 1: Net-(D18-K) -> Net-(D15-K)
- D15 pad 2: Net-(D18-A) -> +3.3V
- D3 pad 1: Net-(D16-K) -> Net-(D3-K)
- D3 pad 2: Net-(D16-A) -> +3.3V
- D4 pad 1: Net-(D13-K) -> Net-(D4-K)
- D4 pad 2: Net-(D13-A) -> +3.3V
- D5 pad 1: +3V3 -> Net-(D5-K)
- D5 pad 2: Net-(D3-K) -> +3.3V
- D6 pad 1: +3V3 -> Net-(D6-K)
- D6 pad 2: Net-(D2-K) (its old number) -> +3.3V
- D7 pad 1: +3V3 -> Net-(D7-K)
- D7 pad 2: Net-(D1-K) (its old number) -> +3.3V
- D8 pad 1: +3V3 -> Net-(D8-K)
- D8 pad 2: Net-(D12-K) -> +3.3V
- D9 pad 1: +3V3 -> Net-(D9-K)
- D9 pad 2: Net-(D11-K) -> +3.3V
- Q1 pad 1: Net-(D16-K) -> Net-(Q1-B)
- Q1 pad 2: Net-(Q2-B) -> GND
- Q1 pad 3: GND -> Net-(Q1-C)
- Q2 pad 1: Net-(D13-K) -> Net-(Q2-B)
- Q2 pad 2: Net-(Q1-B) -> GND
- Q2 pad 3: GND -> Net-(Q2-C)
- Q4 pad 1: Net-(D17-K) -> Net-(Q4-B)
- Q4 pad 2: Net-(Q3-B) (its old number) -> GND
- Q4 pad 3: GND -> Net-(Q4-C)
- Q5 pad 1: Net-(D19-K) -> Net-(Q5-B)
- Q5 pad 2: Net-(Q6-B) -> GND
- Q5 pad 3: GND -> Net-(Q5-C)
- Q6 pad 1: Net-(D18-K) -> Net-(Q6-B)
- Q6 pad 2: Net-(Q5-B) -> GND
- Q6 pad 3: GND -> Net-(Q6-C)
- R19 pad 2: Net-(Q2-B) -> Net-(Q1-B)
- R20 pad 2: Net-(Q1-B) -> Net-(Q2-B)
- R21 pad 1: +3.3V -> Net-(D3-K)
- R21 pad 2: Net-(D16-A) -> Net-(Q1-C)
- R22 pad 1: +3.3V -> Net-(D4-K)
- R22 pad 2: Net-(D13-A) -> Net-(Q2-C)
- R33 pad 1: Net-(D8-K) -> Net-(D5-K)
- R34 pad 1: Net-(D9-K) -> Net-(D6-K)
- R35 pad 1: Net-(D10-K) -> Net-(D7-K)
- R36 pad 1: Net-(D11-K) -> Net-(D8-K)
- R37 pad 1: Net-(D12-K) -> Net-(D9-K)
- R38 pad 1: Net-(D1-K) (its old number) -> Net-(D10-K)
- R39 pad 1: Net-(D2-K) (its old number) -> Net-(D11-K)
- R40 pad 1: Net-(D3-K) -> Net-(D12-K)
- R41 pad 2: Net-(Q3-B) (its old number) -> Net-(Q4-B)
- R42 pad 2: Net-(Q6-B) -> Net-(Q5-B)
- R43 pad 1: +3.3V -> Net-(D13-K)
- R43 pad 2: Net-(D17-A) -> Net-(Q4-C)
- R44 pad 1: +3.3V -> Net-(D14-K)
- R44 pad 2: Net-(D19-A) -> Net-(Q5-C)
- R46 pad 2: Net-(Q5-B) -> Net-(Q6-B)
- R54 pad 1: +3.3V -> Net-(D15-K)
- R54 pad 2: Net-(D18-A) -> Net-(Q6-C)
- U1 pad 25: Net-(U3-FSOURCE) -> unconnected-(U1-FSOURCE-Pad25)
- U10 pad 10: /mcu/MCU_TX0 -> /MCU_TXD
- U10 pad 16: unconnected-(U12-(PCINT31/OC2A)PD7-Pad16) -> /mcu/buzzer
- U10 pad 27: /mcu/AVCC -> +3.3V
- U10 pad 9: /mcu/MCU_RX0 -> /MCU_RXD
- U7 pad 5: +3V3 -> +3.3V
- U7 pad 6: +3V3 -> +3.3V
- U8 pad 11: Net-(U9-~{INT}) -> unconnected-(U8-~{INT}-Pad11)
- U9 pad 14: +3V3 -> +3.3V
- U9 pad 9: +3V3 -> +3.3V
Routing:
- net +3.3V: track 308.5 -> 512.6 mm, vias 11 -> 28
- net /mcu/BTN_USER_A: track 4.91 -> 116.8 mm, vias 0 -> 3
- net /UART_TX_LED: track 1.86 -> 82.8 mm, vias 0 -> 3
- net /UART_RX_LED: track 1.63 -> 77.1 mm, vias 0 -> 1
- net /mcu/buzzer: track 0.00 -> 69.1 mm, vias 0 -> 2
- net /mcu/LED_U3: track 0.00 -> 65.8 mm, vias 0 -> 2
- net /mcu/LED_U2: track 0.00 -> 60.7 mm, vias 0 -> 2
- net Net-(D13-K): track 0.00 -> 60.6 mm, vias 0 -> 1
- net /mcu/LED_U1: track 0.00 -> 55.9 mm, vias 0 -> 2
- net Net-(D15-K): track 0.00 -> 55.7 mm, vias 0 -> 1
- net Net-(D14-K): track 0.00 -> 53.2 mm, vias 0 -> 1
- net VBUS: track 52.2 -> 94.0 mm, vias 6 -> 9
- net Net-(D3-K): track 1.52 -> 38.9 mm, vias 0 -> 2
- net +3V3: track 37.2 -> 0.00 mm
- net Net-(D4-K): track 0.00 -> 31.5 mm, vias 0 -> 2
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
Commit message: WIP, routing
Parts:
- removed the C44 at (169.7, 118.3)
- added BZ1: LET9032ES-03L-2.7-16-R, MLAB_BUZZER:MagneticBuzzer_LET9032ES-03L-2.7-16-R, B.Cu at (151.8, 125.7)
- added U6: MS561101BA03-50, Mlab_IO:LGA-8_3x5mm_P1.25mm, B.Cu at (100.5, 141.8)
- SW1, SW2: value SW_Push -> SKRTLAE010
- SW3: value SW_Push -> KMT031
- SW4: value MCU_RST -> KMT031
- moved FID1 128.0 mm to (112.0, 86.0)
- moved FID3 57.8 mm to (196.0, 86.0)
- moved FID2 21.5 mm to (132.0, 132.0)
- moved F1 19.3 mm to (123.6, 137.7)
- moved F2 19.3 mm to (142.9, 137.8)
- moved C6 12.2 mm to (103.3, 141.1)
- moved FID4 6.44 mm to (205.0, 136.0)
- moved C21 3.69 mm to (130.0, 87.0), turned to -90 degrees
- moved C4 3.47 mm to (95.3, 142.6)
- moved C22 2.74 mm to (132.1, 87.0), turned to -90 degrees
- moved U4 2.67 mm to (92.8, 142.5)
- moved C20 1.60 mm to (204.4, 91.0), turned to 180 degrees
- moved C15 0.70 mm to (163.7, 83.5)
- moved R31 0.08 mm to (171.8, 89.5)
- moved R30 0.07 mm to (169.8, 89.5)
- renumbered IC1 to U10, U10 to U11, IC2 to U12, U11 to U13, U12 to U14, U13 to U15, U14 to U16, U15 to U17, U16 to U18, U1 to locked
Routing:
- net Net-(BZ1-+): track 0.00 -> 23.5 mm
- net SDA_I2C: track 174.5 -> 183.4 mm, vias 4 -> 6
- net (no net): track 8.28 -> 0.00 mm
- net SCL_I2C: track 163.5 -> 169.9 mm
- net +3.3V: track 512.6 -> 518.1 mm, vias 28 -> 30
- net Net-(BT1B-+): track 0.00 -> 4.14 mm
- net Net-(BT1A-+): track 0.00 -> 4.14 mm
- net GND: track 72.1 -> 76.0 mm, vias 61 -> 73
- net /mcu/CDAT2: track 28.9 -> 30.1 mm
- net /liion/P1: track 49.7 -> 50.8 mm
- net /mcu/CDAT3: track 27.7 -> 27.2 mm
Other:
- board text added: "BATTERY"
- board text added: "GND #RST MOSI SCLK 3v3 MISO"
- board text added: "MCU RST"
- board text added: "USER"
- board text added: "USER BTN"

Commit message: WIP
Parts:
- added J5: 46436-9327, Mlab_CON:MOLEX_46437-9327, F.Cu at (78.4, 86.4)
- added J6: HEADER_2x15, Connector_PinHeader_2.54mm:PinHeader_2x15_P2.54mm_Vertical, B.Cu at (63.6, 87.2)
- added JP7: Jumper_3_Bridged12, Jumper:SolderJumper-3_P1.3mm_Bridged12_RoundedPad1.0x1.5mm, F.Cu at (62.2, 83.5)
- moved H1 10.2 mm to (92.6, 69.4)
- moved H3 10.2 mm to (92.6, 140.6)
- moved C4 6.90 mm to (102.2, 142.8)
- moved C6 6.88 mm to (110.2, 141.3)
- moved U6 6.83 mm to (107.3, 142.1)
- moved U4 6.83 mm to (99.6, 142.8)
- moved U3 6.05 mm to (111.4, 115.0)
- moved R9 6.05 mm to (114.2, 114.8)
- moved J2 4.85 mm to (96.8, 123.8)
- moved C27 0.81 mm to (110.9, 103.0)
- moved C31 0.81 mm to (110.9, 105.1)
- moved SW3 0.12 mm to (117.6, 93.1)
- moved SW4 0.12 mm to (124.8, 93.1)
- renumbered R24 to R23, R25 to R24, R26 to R25, R27 to R26, R28 to R27, R29 to R28, R30 to R29, R31 to R30, R32 to R31, R33 to R32, R34 to R33, R35 to R34, R36 to R35, R37 to R36, R38 to R37, R39 to R38, R40 to R39, R41 to R40, R42 to R41, R43 to R42, R44 to R43, R45 to R44, R46 to R45, R47 to R46, R48 to R47, R49 to R48, R50 to R49, R51 to R50, R52 to R51, R53 to R52, R54 to R53, R55 to R54, R56 to R55, R57 to R56, R58 to R57, R59 to R58, R60 to R59, R61 to R60, R62 to R61, R63 to R62, R64 to R63, R65 to R64, R66 to R65, R67 to R66, R68 to R67, R69 to R68, R70 to R69, R71 to R70, R23 to TH1, TH1 to TH2
Connections:
- SW1 pad GND: (no net) -> GND
- SW2 pad GND: (no net) -> GND
- U5 pad 17: (no net) -> GND
Routing:
- net /External_connector/3v3: track 0.00 -> 47.4 mm
- net /External_connector/5v: track 0.00 -> 42.1 mm, vias 0 -> 1
- net /External_connector/I2C_PWR: track 0.00 -> 40.2 mm
- net /External_connector/SDA: track 0.00 -> 24.0 mm
- net /External_connector/A0: track 0.00 -> 18.2 mm
- net /External_connector/A1: track 0.00 -> 13.9 mm
- net /External_connector/C1: track 0.00 -> 13.6 mm
- net /External_connector/SCL: track 0.00 -> 13.2 mm
- net SDA_I2C: track 183.4 -> 171.1 mm
- net GND: track 76.0 -> 87.5 mm
- net /External_connector/B0: track 0.00 -> 10.9 mm
- net /External_connector/C0: track 0.00 -> 10.7 mm
- net /External_connector/B1: track 0.00 -> 10.7 mm
- net SCL_I2C: track 169.9 -> 159.3 mm
- net /External_connector/SCLK: track 0.00 -> 9.82 mm
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- added copper zone on B.Cu, net /External_connector/BATT
- added copper zone on F.Cu, net /External_connector/BATT
Other:
- outline, holes or cut-outs redrawn
- board text added: "3v3 P 5v"
- board text added: "GND 5V 3v3 x A0 A1 B1 B0 C1 C0 GND SCL P SDA GND"
- board text added: "GND 5V 3v3 x x RX TX MOS MIS SCL"
- board text added: "GND SCL P SDA GND"
