File: hw/sch_pcb/LION5CELL01.kicad_sch (KiCad schematic)
At the start: 23 parts, among them IC1 FT260Q-T, IC2 PCA9541ABS/01, U3 USBLC6-2SC6, U9 SHT35-DIS

Commit message: wip: add new components, try to prepare layout outlines
Parts:
- added C40, C41, C42, C44: 1u, Capacitor_SMD:C_0805_2012Metric, symbol Device:C_Small
- added C45: 100n, Capacitor_SMD:C_0805_2012Metric, symbol Device:C_Small
- added D11: GREEN, Mlab_D:LED_1206_mill, symbol Device:LED
- added D13, D16: RED, Mlab_D:LED_1206_mill, symbol Device:LED
- added D14: YELLOW, Mlab_D:LED_1206_mill, symbol Device:LED
- added D15: BLUE, Mlab_D:LED_1206_mill, symbol Device:LED
- added J10: HEADER_2x04_PARALLEL, Connector_PinHeader_2.54mm:PinHeader_2x04_P2.54mm_Vertical, symbol MLAB_HEADER:HEADER_2x04_PARALLEL
- added J7: USBC_USB4105-GF-A, Mlab_CON:USBC GCT_USB4105-GF-A, symbol MLAB_CONNECTORS:USBC_USB4105-GF-A
- added JP10: Jumper_3_Bridged12, Jumper:SolderJumper-3_P1.3mm_Bridged12_RoundedPad1.0x1.5mm, symbol Jumper:Jumper_3_Bridged12
- added JP11: Jumper_3_Bridged12, Connector_PinHeader_2.54mm:PinHeader_1x03_P2.54mm_Vertical, symbol Jumper:Jumper_3_Bridged12
- added JP9: Jumper_2_Open, Connector_PinHeader_2.54mm:PinHeader_2x01_P2.54mm_Vertical, symbol Jumper:Jumper_2_Open
- added Q1: IRF9317TRPBF, Package_SO:SOIC-8_3.9x4.9mm_P1.27mm, symbol MLAB_T:IRF7469PbF
- added R44, R53, R64: 100k, Resistor_SMD:R_0805_2012Metric, symbol Device:R_Small
- added R46, R47, R48, R49, R50, R51, R52: 4k7, Resistor_SMD:R_0805_2012Metric, symbol Device:R_Small
- added R54, R59, R60, R63: 62R, Resistor_SMD:R_0805_2012Metric, symbol Device:R_Small
- added R61: 10R, Resistor_SMD:R_0805_2012Metric, symbol Device:R_Small
- added R62, R67: 1k, Resistor_SMD:R_0805_2012Metric, symbol Device:R_Small
- added R65: 20k, Resistor_SMD:R_0805_2012Metric, symbol Device:R_Small
- added R66: 100R, Resistor_SMD:R_0805_2012Metric, symbol Device:R_Small
- added U13: STUSB4500QTR, Package_DFN_QFN:QFN-24-1EP_4x4mm_P0.5mm_EP2.7x2.7mm, symbol Interface_USB:STUSB4500QTR
- C? (x2): footprint (none) -> Capacitor_SMD:C_0805_2012Metric
- R2: renamed from R5; footprint Mlab_R:SMD-0805 -> Resistor_SMD:R_0603_1608Metric
- R3: renamed from R6; footprint Mlab_R:SMD-0805 -> Resistor_SMD:R_0603_1608Metric
- renumbered U3 to U1, U9 to U2
Connections:
- net D+: now also J7.A6 (D+), J7.B6 (D+)
- net D-: now also J7.A7 (D-), J7.B7 (D-)
- net GND: now also C40.2, C41.2, C42.2, C44.2, J10.1, J10.2, J10.7, J10.8, J7.A1/B12 (GND), J7.B1/A12 (GND), J7.G1 (SHIELD), J7.G2 (SHIELD), J7.G3 (SHIELD), J7.G4 (SHIELD), JP10.3 (B), JP9.2 (B), R53.1, U13.10 (GND), U13.25 (GND)
- net VBUS: now also C40.1, J7.A4/B9 (VBUS), J7.B4/A9 (VBUS), Q1.1 (S), Q1.2 (S), Q1.3 (S), R62.1, R64.1, U13.24 (VDD)
- new net: D14.2 (A), R60.2
- new net: Q1.4 (G), R64.2, R65.1, R66.2
- new net: C45.1, J10.3, J10.4, J10.5, J10.6, Q1.5 (D), Q1.6 (D), Q1.7 (D), Q1.8 (D), R67.1
- new net: C45.2, R66.1
- new net: D16.2 (A), R63.2
- new net: D11.2 (A), R54.2
- new net: J7.A5 (CC1), U13.1 (CC1DB), U13.2 (CC1)
- new net: C44.1, U13.21 (VREG_1V2)
- new net: C42.1, U13.23 (VREG_2V7)
- new net: J7.B5 (CC2), U13.4 (CC2), U13.5 (CC2DB)
- new net: D15.2 (A), R61.2
- new net: D13.2 (A), R59.2
- new net +3V3: JP11.1 (A), R54.1, R59.1, R60.1, R61.1, R63.1
- new net ADDR0: JP9.1 (A), R44.2, U13.12 (ADDR0)
- new net ADDR1: JP10.2 (C), U13.13 (ADDR1)
- new net ALERT: D13.1 (K), R46.2, U13.19 (ALERT)
- new net ATTACH: D11.1 (K), R48.2, U13.11 (ATTACH)
- new net DISCH: R67.2, U13.9 (DISCH)
- new net EXT_PWR: JP11.3 (B)
- new net GPIO: D14.1 (K), R49.2, U13.15 (GPIO)
- new net PWR_OK2: D15.1 (K), R50.2, U13.20 (POWER_OK2)
- new net PWR_OK3: D16.1 (K), R51.2, U13.14 (POWER_OK3)
- new net RESET: R52.2, U13.6 (RESET)
- new net SCL: U13.7 (SCL)
- new net SDA: U13.8 (SDA)
- new net SIDE: R47.2, U13.17 (A_B_SIDE)
- new net VBUS_EN_SINK: R65.2, U13.16 (VBUS_EN_SNK)
- new net VBUS_VS_DISCH: R62.2, U13.18 (VBUS_VS_DISCH)
- new net VCC: C41.1, JP10.1 (A), JP11.2 (C), R44.1, R46.1, R47.1, R48.1, R49.1, R50.1, R51.1, R52.1, R53.2, U13.22 (VSYS)
- no-connect marks 4 -> 6
Other:
- added sheet sw_source (sw_source.kicad_sch)
- note added: "Addr selector"
- note added: "LED indicators"
- note added: "Output disconnector"
- note added: "Power selector"
- note added: "Signal pull-ups"
- note added: "USB-C connector and PD-sink controller"
- note added: "Zkusit nahradit za 10k"

Commit message: wip, update schematics, board outlines
Parts:
- removed JP10: Jumper_3_Bridged12, Jumper:SolderJumper-3_P1.3mm_Bridged12_RoundedPad1.0x1.5mm, symbol Jumper:Jumper_3_Bridged12
- removed JP11: Jumper_3_Bridged12, Connector_PinHeader_2.54mm:PinHeader_1x03_P2.54mm_Vertical, symbol Jumper:Jumper_3_Bridged12
- removed JP9: Jumper_2_Open, Connector_PinHeader_2.54mm:PinHeader_2x01_P2.54mm_Vertical, symbol Jumper:Jumper_2_Open
- removed R44, R53: 100k, Resistor_SMD:R_0805_2012Metric, symbol Device:R_Small
- added C? (x3): 4u7, Capacitor_SMD:C_0805_2012Metric, symbol Device:C_Small
- added C?: 0u1, Capacitor_SMD:C_0805_2012Metric, symbol Device:C_Small
- added C?: 100nF, Capacitor_SMD:C_0805_2012Metric, symbol Device:C_Small
- added R18, R19, R20, R21, R22, R75: 10k, Resistor_SMD:R_0805_2012Metric, symbol Device:R_Small
- added R20 (x2), R21 (x3): 10k, Resistor_SMD:R_0805_2012Metric, symbol SPACEDOS01A_PCB01A-rescue:R-device-DATALOGGER01A-rescue-CCP2019V01A-rescue
- added R23, R24: 33R, Resistor_SMD:R_0805_2012Metric, symbol Device:R_Small
- added R33: 1k, Resistor_SMD:R_0805_2012Metric, symbol Device:R_Small
- added TP1: FTDI FS, TestPoint:TestPoint_Pad_D1.5mm, symbol Connector:TestPoint
- added TP1: MUX_RST, TestPoint:TestPoint_Pad_D1.5mm, symbol Connector:TestPoint
- added U7: TCA4307, Package_SO:VSSOP-8_3.0x3.0mm_P0.65mm, symbol MLAB_IO:TCA4307
- C1: renamed from C40; value 1u -> 1n
- C? (x2): symbol Device:C -> Device:C_Small
- IC?: Height (none) -> 1; I2C (none) -> 0x76
- JP1: footprint Jumper:SolderJumper-2_P1.3mm_Open_RoundedPad1.0x1.5mm -> (none); symbol Jumper:SolderJumper_2_Open -> Jumper:SolderJumper_2_Bridged
- R20, R21, R32: footprint Resistor_SMD:R_0603_1608Metric -> Resistor_SMD:R_0805_2012Metric
- R26: renamed from R2; footprint Resistor_SMD:R_0603_1608Metric -> Resistor_SMD:R_0805_2012Metric; symbol Device:R -> Device:R_Small; LCSC C228675 -> (none); UST_ID 5c70984512875079b91f8983 -> (none)
- R27: renamed from R3; footprint Resistor_SMD:R_0603_1608Metric -> Resistor_SMD:R_0805_2012Metric; symbol Device:R -> Device:R_Small; LCSC C228675 -> (none); UST_ID 5c70984512875079b91f8983 -> (none)
- U4: renamed from U2; Height (none) -> 0.9; I2C (none) -> 0x44
- U5: renamed from IC2; I2C (none) -> 0x70
- renumbered C41 to C2, C42 to C3, C44 to C4, C45 to C5, D11 to D1, D13 to D2, D14 to D3, D15 to D4, D16 to D5, D1 to D6, D2 to D7, J7 to J1, J10 to J2, R46 to R1, R60 to R10, R61 to R11, R63 to R12, R62 to R13, R64 to R14, R65 to R15, R66 to R16, R67 to R17, R47 to R2, R48 to R3, R49 to R4, R50 to R5, R51 to R6, R52 to R7, R54 to R8, R59 to R9, U13 to U1, U1 to U2, IC1 to U3
Connections:
- net ADDR0 is gone; now on net GND: U1.12 (ADDR0)
- net ADDR1 is gone; now on net GND: U1.13 (ADDR1)
- net +3.3V: now also C2.1, U1.22 (VSYS), U3.22 (VOUT3V3), U3.23 (VCCIN), U3.6 (VCCIO), U5.14 (VDD), C?.1, C?.1, C?.1, C?.1, R18.1, R19.1, R20.1, R20.2, R20.2, R21.1, R21.2, R21.2, R21.2, R22.1, R33.2, U7.8 (VCC)
- net DN: now also R24.2
- net DP: now also R23.2
- net GND: now also R26.2, R27.2, U3.19 (GND), C?.2, C?.2, C?.2, C?.2, C?.2, U7.4 (GND); no longer U3.3 (RESETN), U3.4 (DCNF0), U3.5 (DCNF1)
- net SCL_I2C: now also U7.3 (SCLin)
- net SCL_MCU: now also R20.1
- net SCL_USB: now also R20.1
- net SDA_I2C: now also U7.6 (SDAin)
- net SDA_MCU: now also R21.1
- net SDA_USB: now also R21.1
- net VCC: no longer C2.1, U1.22 (VSYS)
- net at U5.2 (~{RESET}): now also R33.1, TP1.1
- net at U3.1 (DEBUGGER): now also R22.2
- net at U3.2 (STEST_RSTN): now also R21.2
- net at U3.20 (DM): now also R24.1
- net at U3.21 (DP): now also R23.1
- net at U3.25 (FSOURCE): now also TP1.1
- net at U3.26 (VBUS_DET): now also R75.2
- new net: C?.1, R20.2, U3.3 (RESETN)
- new net: R19.2, U3.4 (DCNF0)
- new net: R18.2, U3.5 (DCNF1)
- new net DET_I2C_EN: R21.1, U7.1 (EN)
- new net OUT_SCL_I2C: U7.2 (SCLout)
- new net OUT_SDA_I2C: U7.7 (SDAout)
- no-connect marks 6 -> 10
Other:
- note added: "I2C: 0x44"
- note added: "I2C: 0x70"
- note added: "I2C: 0x76"
- note removed: "Addr selector"
- note removed: "Power selector"
- note removed: "Zkusit nahradit za 10k"
- moved on the sheet: C1, C2, C3, C4, C5, C?, D1, D2, D3, D4, D5, J1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

Commit message: WIP: schematics and layout improvements
Parts:
- removed J2: HEADER_2x04_PARALLEL, Connector_PinHeader_2.54mm:PinHeader_2x04_P2.54mm_Vertical, symbol MLAB_HEADER:HEADER_2x04_PARALLEL
- removed R3, R4, R5, R6, R7: 4k7, Resistor_SMD:R_0805_2012Metric, symbol Device:R_Small
- added Q4: BC817-25, Package_TO_SOT_SMD:SOT-23-3, symbol Simulation_SPICE:NPN
- D1, D2, D3, D4, D5: footprint Mlab_D:LED_1206_mill -> LED_SMD:LED_1206_3216Metric
- D6, D7: footprint Mlab_D:LED_1206_2 -> LED_SMD:LED_1206_3216Metric
- IC?: footprint MS561101BA03-50 -> (none)
- JP1: footprint (none) -> Jumper:SolderJumper-2_P1.3mm_Open_RoundedPad1.0x1.5mm
- R1: value 4k7 -> 1k; MFPN R0805 4k7 1% -> (none); MPN R0805 4k7 1% -> (none); UST_ID 5c70984612875079b91f8995 -> (none)
- R2: value 4k7 -> 10k; MFPN R0805 4k7 1% -> (none); MPN R0805 4k7 1% -> (none); UST_ID 5c70984612875079b91f8995 -> (none)
- R26, R27: value 270R -> R
- R75: value 10k -> 1k
Connections:
- net +5V is gone; now on net +3.3V: D6.2 (A), D7.2 (A)
- net +3.3V: now also R2.2
- net ALERT: no longer R1.2
- net ATTACH: now also R1.1
- net GND: now also Q4.3 (E); no longer R26.2, R27.2
- net MCU_RXD: now also U3.11 (DIO4); no longer U3.10 (DIO3)
- net MCU_TXD: now also U3.10 (DIO3); no longer U3.11 (DIO4)
- net SIDE: no longer R2.2
- net VBUS: no longer U2.5 (VBUS)
- net USB_POWER: now reaches C5.1, Q1.5 (D), Q1.6 (D), Q1.7 (D), Q1.8 (D), R17.1
- net USB_CONNECTED: now reaches R75.1
- net USB_CONNECTED: now also R2.1, Q4.1 (C)
- net UART_RX_LED: now reaches U3.27 (DIO12)
- net UART_RX_LED: now also R27.2
- net UART_TX_LED: now reaches U3.7 (DIO0)
- net UART_TX_LED: now also R26.2
- net DN renamed USB_D-
- net USB_D-: no longer R24.2
- net DP renamed USB_D+
- net USB_D+: no longer R23.2
- net OUT_SCL_I2C renamed EXT_I2C_SCL
- net OUT_SDA_I2C renamed EXT_I2C_SDA
- removed net VCC: R1.1, R2.1
- new net: Q4.2 (B), R1.2
- new net USB_FTDI_D+: R23.2
- new net USB_FTDI_D-: R24.2
- no-connect marks 10 -> 18
Other:
- added sheet External_connector (connector.kicad_sch)
- sheet mcu ports: added MCU_RX0, MCU_TX0; removed none
- note removed: "Signal pull-ups"
- moved on the sheet: C?, IC?, JP1, R32, U2, U4

Commit message: wip layout, add datasheets
Connections:
- net SCL_I2C: now also R21.1; no longer R20.1
- net SDA_I2C: now also R20.1; no longer R21.1
Other:
- moved on the sheet: R17, R20, R21

Commit message: WIP
Parts:
- removed C2, C3, C4: 1u, Capacitor_SMD:C_0805_2012Metric, symbol Device:C_Small
- removed Q4: BC817-25, Package_TO_SOT_SMD:SOT-23-3, symbol Simulation_SPICE:NPN
- removed U1: STUSB4500QTR, Package_DFN_QFN:QFN-24-1EP_4x4mm_P0.5mm_EP2.7x2.7mm, symbol Interface_USB:STUSB4500QTR
- R1: value 1k -> R_Small; footprint Resistor_SMD:R_0805_2012Metric -> (none)
- R2: value 10k -> R_Small; footprint Resistor_SMD:R_0805_2012Metric -> (none)
- R75: value 1k -> 5k1 (cca)
Connections:
- net +3.3V: no longer R2.2
- net ATTACH: no longer R1.1
- net GND: now also R1.1, R2.1
- net USB_CONNECTED: no longer R2.1, R75.1
- net VBUS: now also R75.1, U2.5 (VBUS)
- net at J1.A5 (CC1): now also R1.2
- net at J1.B5 (CC2): now also R2.2
- no-connect marks 18 -> 17
Other:
- note added: "Pridat spravne odpory"
- note added: "USB-C connector"
- note removed: "USB-C connector and PD-sink controller"
- moved on the sheet: C1, U2

Commit message: WIP, layout improvement
Parts:
- removed C5: 100n, Capacitor_SMD:C_0805_2012Metric, symbol Device:C_Small
- removed C?: 4u7, Capacitor_SMD:C_0805_2012Metric, symbol Device:C_Small
- removed D1: GREEN, LED_SMD:LED_1206_3216Metric, symbol Device:LED
- removed D2, D5: RED, LED_SMD:LED_1206_3216Metric, symbol Device:LED
- removed D3: YELLOW, LED_SMD:LED_1206_3216Metric, symbol Device:LED
- removed D4: BLUE, LED_SMD:LED_1206_3216Metric, symbol Device:LED
- removed Q1: IRF9317TRPBF, Package_SO:SOIC-8_3.9x4.9mm_P1.27mm, symbol MLAB_T:IRF7469PbF
- removed R10, R12, R8, R9: 62R, Resistor_SMD:R_0805_2012Metric, symbol Device:R_Small
- removed R11: 10R, Resistor_SMD:R_0805_2012Metric, symbol Device:R_Small
- removed R13, R17: 1k, Resistor_SMD:R_0805_2012Metric, symbol Device:R_Small
- removed R14: 100k, Resistor_SMD:R_0805_2012Metric, symbol Device:R_Small
- removed R15: 20k, Resistor_SMD:R_0805_2012Metric, symbol Device:R_Small
- removed R16: 100R, Resistor_SMD:R_0805_2012Metric, symbol Device:R_Small
- removed R20, R21, R22: 10k, Resistor_SMD:R_0805_2012Metric, symbol Device:R_Small
- added J2: 46436-9327, Mlab_CON:MOLEX_46436-9327, symbol MLAB_CONNECTORS:MOLEX_46436-9327
- R18, R19: value 10k -> 1K
- R20, R21: value 10k -> 1k
Connections:
- net +3.3V: now also U3.1 (DEBUGGER), U3.2 (STEST_RSTN), U3.3 (RESETN)
- net EXT_I2C_SCL: now also J2.C1
- net EXT_I2C_SDA: now also J2.C2
- net GND: now also J2.A2, J2.A5, J2.B2, J2.B5, J2.P2, J2.P3
- new net +BATT: J2.P1, J2.P4
- new net 3v3_EXT: J2.A3, J2.B3
- new net 5v_EXT: J2.A4, J2.B4
- new net EXT_A0: J2.D4
- new net EXT_A1: J2.D5
- new net EXT_B0: J2.E5
- new net EXT_B1: J2.E6
- new net EXT_C0: J2.E1
- new net EXT_C1: J2.E2
- new net EXT_MISO: J2.D2
- new net EXT_MOSI: J2.D3
- new net EXT_RX: J2.E4
- new net EXT_SCK: J2.D1
- new net EXT_TX: J2.E3
Other:
- note removed: "LED indicators"
- note removed: "Output disconnector"
- note removed: "Pridat spravne odpory"
- moved on the sheet: C1, C?, D6, D7, J1, JP1, R1, R18, R19, R2, R21, R23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

Commit message: wip, layout progress
Parts:
- D6, D7: footprint LED_SMD:LED_1206_3216Metric -> Mlab_D:SMD_LED_RIGHT_KINGBRIGHT_1605
- R1, R2: footprint (none) -> Resistor_SMD:R_0805_2012Metric
Changed lines of the file:
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@@
       (effects (font (size 1 1)) (justify right))
     )
-    (property "Footprint" "LED_SMD:LED_1206_3216Metric" (at 138.43 144.78 0)
+    (property "Footprint" "Mlab_D:SMD_LED_RIGHT_KINGBRIGHT_1605" (at 138.43 144.78 0)
       (effects (font (size 1 1)) hide)
     )
@@
       (effects (font (size 1.27 1.27)) (justify right))
     )
-    (property "Footprint" "" (at 52.07 64.77 0)
+    (property "Footprint" "Resistor_SMD:R_0805_2012Metric" (at 52.07 64.77 0)
       (effects (font (size 1.27 1.27)) hide)
     )
@@
       (effects (font (size 1.27 1.27)) (justify right))
     )
-    (property "Footprint" "" (at 59.69 64.77 0)
+    (property "Footprint" "Resistor_SMD:R_0805_2012Metric" (at 59.69 64.77 0)
       (effects (font (size 1.27 1.27)) hide)
     )
@@
       (effects (font (size 1 1)) (justify right))
     )
-    (property "Footprint" "LED_SMD:LED_1206_3216Metric" (at 129.54 144.78 0)
-      (effects (font (size 1 1)) hide)
-    )
+    (property "Footprint" "Mlab_D:SMD_LED_RIGHT_KINGBRIGHT_1605" (at 129.54 144.78 0)
+      (effects (font (size 1 1)) hide)
+    )

Commit message: wip, layout improvements
Connections:
- net EXT_SCK renamed EXT_SCLK
Changed lines of the file:
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@@
     )
   )
-  (global_label "EXT_SCK" (shape input) (at 212.09 132.08 0) (fields_autoplaced)
+  (global_label "EXT_SCLK" (shape input) (at 212.09 132.08 0) (fields_autoplaced)
     (effects (font (size 1.27 1.27)) (justify left))
-    (property "Intersheetrefs" "${INTERSHEET_REFS}" (at 223.1184 132.08 0)
+    (property "Intersheetrefs" "${INTERSHEET_REFS}" (at 224.1465 132.08 0)
       (effects (font (size 1.27 1.27)) (justify left) hide)
     )
