File: hw/sch_pcb/LION5CELL01.kicad_sch (KiCad schematic)
At the start: 46 parts, among them J1 USBC_USB4105-GF-A, J2 46436-9327, U2 USBLC6-2SC6, U3 FT260Q-T, U4 SHT35-DIS, U5 PCA9541ABS/01, U7 TCA4307

Commit message: Wip, layout
Parts:
- removed C?: 4u7, Capacitor_SMD:C_0805_2012Metric, symbol Device:C_Small
- removed TP1: FTDI FS, TestPoint:TestPoint_Pad_D1.5mm, symbol Connector:TestPoint
- C?: value 0u1 -> 100n
- C? (x3): value 100nF -> 100n
- R1: renamed from R18; value 1K -> 1k
- R2: renamed from R19; value 1K -> 1k
- renumbered C1 to C3, D6 to D1, D7 to D2, R26 to R10, R27 to R11, R33 to R16, R2 to R3, R1 to R4, R75 to R5, R23 to R6, R24 to R7, U3 to U1, U7 to U3
Other:
- moved on the sheet: C?

Commit message: WIP, routing
Parts:
- IC?: footprint (none) -> Mlab_IO:LGA-8_3x5mm_P1.25mm
Changed lines of the file:
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@@
       (effects (font (size 1 1)))
     )
-    (property "Footprint" "" (at 261.62 36.83 0)
+    (property "Footprint" "Mlab_IO:LGA-8_3x5mm_P1.25mm" (at 261.62 36.83 0)
       (effects (font (size 1 1)) (justify left) hide)
     )

Commit message: WIP
Parts:
- C3: UST_ID 5c70984712875079b91f8b50 -> (none)
- D1: UST_ID 5c70984412875079b91f8896 -> (none)
- D2: UST_ID 5c70984412875079b91f8895 -> (none)
- J1: UST_ID 5fa0f94612875025b397795e -> (none)
- R20, R21: UST_ID 5c70984512875079b91f8962 -> (none)
- R32: UST_ID 5c70984512875079b91f8956 -> (none)
- U2: UST_ID 5e82e0691287502a334a778c -> (none)
Connections:
- net GND: now also U5.17 (VSS_pad)
Changed lines of the file:
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@@
   (junction (at 261.62 81.28) (diameter 0) (color 0 0 0 0)
   )
-  (junction (at 236.22 106.68) (diameter 0) (color 0 0 0 0)
-  )
   (junction (at 168.91 119.38) (diameter 0) (color 0 0 0 0)
   )
@@
   (junction (at 232.41 46.99) (diameter 0) (color 0 0 0 0)
   )
+  (junction (at 233.68 106.68) (diameter 0) (color 0 0 0 0)
+  )
   (junction (at 83.82 127) (diameter 0) (color 0 0 0 0)
   )
@@
     (stroke (width 0) (type default))
   )
+  (wire (pts (xy 231.14 106.68) (xy 233.68 106.68))
+    (stroke (width 0) (type default))
+  )
   (wire (pts (xy 204.47 78.74) (xy 218.44 78.74))
     (stroke (width 0) (type default))
@@
     (stroke (width 0) (type default))
   )
-  (wire (pts (xy 236.22 106.68) (xy 238.76 106.68))
-    (stroke (width 0) (type default))
-  )
   (wire (pts (xy 199.39 106.68) (xy 199.39 109.22))
     (stroke (width 0) (type default))
@@
     (stroke (width 0) (type default))
   )
+  (wire (pts (xy 233.68 106.68) (xy 238.76 106.68))
+    (stroke (width 0) (type default))
+  )
   (wire (pts (xy 91.44 127) (xy 91.44 125.73))
     (stroke (width 0) (type default))
@@
       (effects (font (size 1 1)) hide)
     )
-    (property "UST_ID" "5c70984712875079b91f8b50" (at 102.87 63.5 0)
+    (property "UST_ID" "" (at 102.87 63.5 0)
       (effects (font (size 1 1)) hide)
     )
@@
       (effects (font (size 1 1)) hide)
     )
-    (property "UST_ID" "5c70984512875079b91f8962" (at 264.16 74.93 0)
+    (property "UST_ID" "" (at 264.16 74.93 0)
       (effects (font (size 1 1)) hide)
     )
@@
       (effects (font (size 1 1)) hide)
     )
-    (property "UST_ID" "5c70984412875079b91f8895" (at 138.43 144.78 0)
+    (property "UST_ID" "" (at 138.43 144.78 0)
       (effects (font (size 1 1)) hide)
     )
@@
       (effects (font (size 1 1)) hide)
     )
-    (property "UST_ID" "5c70984512875079b91f8962" (at 261.62 74.93 0)
+    (property "UST_ID" "" (at 261.62 74.93 0)
       (effects (font (size 1 1)) hide)
     )
@@
     (pin "15")
     (pin "16")
+    (pin "17")
     (pin "2")
     (pin "3")
@@
       (effects (font (size 1 1)) hide)
     )
-    (property "UST_ID" "5c70984512875079b91f8962" (at 209.55 71.12 0)
+    (property "UST_ID" "" (at 209.55 71.12 0)
       (effects (font (size 1 1)) hide)
     )
@@
     )
   )
-  (symbol (lib_name "GND_1") (lib_id "power:GND") (at 236.22 106.68 0) (unit 1)
+  (symbol (lib_name "GND_1") (lib_id "power:GND") (at 233.68 106.68 0) (unit 1)
     (in_bom yes) (on_board yes) (dnp no)
-    (property "Reference" "#PWR030" (at 236.22 113.03 0)
+    (property "Reference" "#PWR030" (at 233.68 113.03 0)
       (effects (font (size 1 1)) hide)
     )
-    (property "Value" "GND" (at 240.03 109.22 0)
+    (property "Value" "GND" (at 233.68 110.49 0)
       (effects (font (size 1 1)))
     )
-    (property "Footprint" "" (at 236.22 106.68 0)
+    (property "Footprint" "" (at 233.68 106.68 0)
       (effects (font (size 1 1)) hide)
     )
-    (property "Datasheet" "" (at 236.22 106.68 0)
+    (property "Datasheet" "" (at 233.68 106.68 0)
       (effects (font (size 1 1)) hide)
     )
@@
       (effects (font (size 1 1)) hide)
     )
-    (property "UST_ID" "5c70984412875079b91f8896" (at 129.54 144.78 0)
+    (property "UST_ID" "" (at 129.54 144.78 0)
       (effects (font (size 1 1)) hide)
     )
@@
       (effects (font (size 1 1)) hide)
     )
-    (property "UST_ID" "5fa0f94612875025b397795e" (at 34.29 69.85 0)
+    (property "UST_ID" "" (at 34.29 69.85 0)
       (effects (font (size 1 1)) hide)
     )
@@
       (effects (font (size 1 1)) hide)
     )
-    (property "UST_ID" "5c70984512875079b91f8962" (at 199.39 71.12 0)
+    (property "UST_ID" "" (at 199.39 71.12 0)
       (effects (font (size 1 1)) hide)
     )
@@
       (effects (font (size 1 1)) hide)
     )
-    (property "UST_ID" "5c70984512875079b91f8962" (at 214.63 71.12 0)
+    (property "UST_ID" "" (at 214.63 71.12 0)
       (effects (font (size 1 1)) hide)
     )
@@
       (effects (font (size 1 1)) hide)
     )
-    (property "UST_ID" "5c70984512875079b91f8956" (at 109.22 165.1 0)
+    (property "UST_ID" "" (at 109.22 165.1 0)
       (effects (font (size 1 1)) hide)
     )
@@
       (effects (font (size 1 1)) hide)
     )
-    (property "UST_ID" "5e82e0691287502a334a778c" (at 86.36 71.12 0)
+    (property "UST_ID" "" (at 86.36 71.12 0)
       (effects (font (size 1 1)) hide)
     )
@@
       (effects (font (size 1 1)) hide)
     )
-    (property "UST_ID" "5c70984512875079b91f8962" (at 204.47 71.12 0)
+    (property "UST_ID" "" (at 204.47 71.12 0)
       (effects (font (size 1 1)) hide)
     )
@@
       (effects (font (size 1 1)) hide)
     )
-    (property "UST_ID" "5c70984512875079b91f8962" (at 129.54 74.93 0)
+    (property "UST_ID" "" (at 129.54 74.93 0)
       (effects (font (size 1 1)) hide)
     )
