File: hw/sch_pcb/liion.kicad_sch (KiCad schematic)
At the start: 60 parts, among them U1 BQ34Z100, U12 BQ25628E, U2 SN74HC164D

Commit message: wip, update schematics, board outlines
Parts:
- removed unit 3 of BT8
- removed F4: Fuse, Mlab_F:Drzak_2410, symbol Device:Fuse
- removed R1, R3: 47k, Resistor_SMD:R_0805_2012Metric, symbol LION2CELL01D-rescue:R-RESCUE-LION2CELL01C
- added SW1: SW_Push_Dual, symbol Switch:SW_Push_Dual
- added TP5: CH_INT, TestPoint:TestPoint_Pad_D1.5mm, symbol Connector:TestPoint
- BT1: renamed from BT8; footprint Mlab_Batery:BAT_BK-18650-PC6 -> Mlab_Batery:BAT_BK-18650-PC4; symbol MLAB_BATERY:3xBATT -> MLAB_BATERY:2xBATT
- C1, C3, C4, C6, C7: symbol LION2CELL01D-rescue:C-RESCUE-LION2CELL01C -> Device:C_Small; UST_ID 5c70984712875079b91f8b4c -> (none)
- C2: symbol LION2CELL01D-rescue:C-RESCUE-LION2CELL01C -> Device:C_Small; UST_ID 5c70984712875079b91f8b50 -> (none)
- C5: symbol LION2CELL01D-rescue:C-RESCUE-LION2CELL01C -> Device:C_Small; UST_ID 5c70984712875079b91f8b47 -> (none)
- D16: renamed from D12; value LED_Dual_AAKK -> KPBA-2006SURKCGKC
- R10, R11, R12, R13, R14, R15, R16, R9: symbol LION2CELL01D-rescue:R-RESCUE-LION2CELL01C -> Device:R_Small; UST_ID 5c70984512875079b91f8983 -> (none)
- R2: symbol LION2CELL01D-rescue:R-RESCUE-LION2CELL01C -> Device:R_Small; UST_ID 5e3ffaff1287502a33bad825 -> (none)
- R37: renamed from R55; footprint Resistor_SMD:R_0603_1608Metric -> Resistor_SMD:R_0805_2012Metric
- R38: renamed from R56; footprint Resistor_SMD:R_0603_1608Metric -> Resistor_SMD:R_0805_2012Metric
- R4: footprint Resistor_SMD:R_0805_2012Metric_Pad1.20x1.40mm_HandSolder -> Resistor_SMD:R_0805_2012Metric
- R41: renamed from R39; value R_Small -> R; footprint Resistor_SMD:R_0603_1608Metric -> Resistor_SMD:R_0805_2012Metric
- R42: renamed from R45; value R_Small -> R; footprint Resistor_SMD:R_0603_1608Metric -> Resistor_SMD:R_0805_2012Metric
- R5: symbol LION2CELL01D-rescue:R-RESCUE-LION2CELL01C -> Device:R_Small; UST_ID 5c70984512875079b91f898c -> (none)
- R54: renamed from R57; footprint Resistor_SMD:R_0603_1608Metric -> Resistor_SMD:R_0805_2012Metric
- R55: renamed from R58; footprint Resistor_SMD:R_0603_1608Metric -> Resistor_SMD:R_0805_2012Metric
- R6, R7: symbol LION2CELL01D-rescue:R-RESCUE-LION2CELL01C -> Device:R_Small; UST_ID 5c70984512875079b91f8977 -> (none)
- R8: footprint Resistor_SMD:R_2512_6332Metric_Pad1.40x3.35mm_HandSolder -> Resistor_SMD:R_0805_2012Metric; symbol LION2CELL01D-rescue:R-RESCUE-LION2CELL01C -> Device:R_Small; UST_ID 5c70984712875079b91f8abf -> (none)
- TH1: renamed from TH2; value Thermistor_NTC -> 10k NTC; footprint (none) -> Resistor_SMD:R_0805_2012Metric
- TP3: renamed from TP2; footprint (none) -> TestPoint:TestPoint_Pad_D1.5mm
- TP4: renamed from TP1; footprint (none) -> TestPoint:TestPoint_Pad_D1.5mm
- U1: Height (none) -> 1,2; I2C (none) -> 0xAA
- U2: footprint Package_SO:SO-14_3.9x8.65mm_P1.27mm -> (none); symbol LION2CELL01D-rescue:SN74HC164D -> MLAB_IO:SN74HC164D; UST_ID 5c70984612875079b91f89ed -> (none)
- U9: renamed from U12; footprint (none) -> Package_DFN_QFN:Texas_S-PWQFN-N20; I2C (none) -> 0x6B
- renumbered BT9 to BT2, C48 to C13, C49 to C14, C50 to C15, C35 to C19, C39 to C23, C47 to C24, C43 to C25, F6 to F1, F5 to F2, F2 to F4, F1 to F5, L5 to L1
Connections:
- net I2C_SCL is gone; now on net SCL_I2C: U1.13 (P4/SCL)
- net I2C_SDA is gone; now on net SDA_I2C: U1.14 (P3/SDA)
- net CH_BTN: now also SW1.3
- net GAUGE_BTN_A: now also SW1.1
- net GAUGE_BTN_B: now also SW1.2
- net GAUGE_SRP: now also R6.1
- net GND: now also SW1.4
- net at U9.11 (~{INT}): now also TP5.1
- net SDA_I2C: now reaches U9.12 (SDA)
- net SCL_I2C: now reaches U9.13 (SCL)
Other:
- moved on the sheet: BT1A, BT1B, BT2A, BT2B, BT2C, C1, C15, C2, C3, C4, C5, C6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

Commit message: WIP: schematics and layout improvements
Parts:
- removed D16: KPBA-2006SURKCGKC, symbol Device:LED_Dual_AAKK
- removed D6, D7, D8: ORAGE, Mlab_D:LED_1206, symbol LION2CELL01D-rescue:LED-RESCUE-LION2CELL01C
- removed R14, R15, R16: 270R, Resistor_SMD:R_0805_2012Metric, symbol Device:R_Small
- removed R55: R, Resistor_SMD:R_0805_2012Metric, symbol Device:R_Small
- added D16: ORANGE, LED_SMD:LED_1206_3216Metric, symbol Device:LED_Small
- added Q4: BC817-25, Package_TO_SOT_SMD:SOT-23-3, symbol Simulation_SPICE:NPN
- added R1: 1k, Resistor_SMD:R_0805_2012Metric, symbol Device:R_Small
- added R2: 10k, Resistor_SMD:R_0805_2012Metric, symbol Device:R_Small
- D1, D2, D3, D4, D5: footprint Mlab_D:LED_1206 -> LED_SMD:LED_1206_3216Metric
- U2: footprint (none) -> Package_SO:TSSOP-14_4.4x5mm_P0.65mm
Connections:
- net +3.3V: now also R2.2
- net CH_STAT: now also R1.1, R2.1
- net GND: now also Q4.3 (E)
- net at R54.2: now also D16.2 (A)
- net CH_PWR renamed USB_POWER
- net F: no longer names the net of U2.11 (QF)
- net G: no longer names the net of U2.12 (QG)
- net H: no longer names the net of U2.13 (QH)
- new net: D16.1 (K), Q4.1 (C)
- new net: Q4.2 (B), R1.2
Other:
- moved on the sheet: R54

Commit message: wip layout, add datasheets
Parts:
- removed R5: 1k, Resistor_SMD:R_0805_2012Metric, symbol Device:R_Small
- removed SW1: SW_Push_Dual, symbol Switch:SW_Push_Dual
- added Q8: PNP, symbol Simulation_SPICE:PNP
- added R1, R2: 1k, Resistor_SMD:R_0805_2012Metric, symbol Device:R_Small
- added R1: 500R, Resistor_SMD:R_0805_2012Metric, symbol Device:R_Small
- added R1: 250R, Resistor_SMD:R_0805_2012Metric, symbol Device:R_Small
- added SW3: SW_Push, symbol Switch:SW_Push
- C14: value 0u1 -> 100n
Connections:
- net +3V3: now also Q8.3 (E), R2.2
- net CH_BTN: now also R1.1, R2.1, SW3.1
- net GND: now also R1.1, SW3.2
- net GAUGE_BTN_B renamed GAUGE_BTN_IN
- net GAUGE_BTN_IN: now also R1.1, R1.2
- new net: Q8.1 (C), R1.2
- new net: Q8.2 (B), R1.2
Other:
- moved on the sheet: C15, C2, C23, C25, D16, Q4, R1, R2, R37, R38, R4, R54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

Commit message: WIP
Parts:
- removed L1: DE1205-10, Mlab_L:DE1205-10, symbol LION2CELL01D-rescue:INDUCTOR_SMALL
- added L1: 1uH - DFE252012P-1R0M=P2, Inductor_SMD:L_1008_2520Metric, symbol Device:L
- U9: footprint Package_DFN_QFN:Texas_S-PWQFN-N20 -> Mlab_IO:Texas_S-WQFN-HR-18
Connections:
- net +VSW: now also L1.2
- net at C19.1, U9.16 (SW): now also L1.1
Other:
- moved on the sheet: C24

Commit message: WIP, layout improvement
Parts:
- removed R38: R, Resistor_SMD:R_0805_2012Metric, symbol Device:R_Small
- added D13: GREEN, LED_SMD:LED_1206_3216Metric, symbol Device:LED_Small
- added Q4: BC817-25, Package_TO_SOT_SMD:SOT-23-3, symbol Simulation_SPICE:NPN
- added R1: 1k, Resistor_SMD:R_0805_2012Metric, symbol Device:R_Small
- added R15: R, Resistor_SMD:R_0805_2012Metric, symbol Device:R_Small
- added R2: 10k, Resistor_SMD:R_0805_2012Metric, symbol Device:R_Small
- BT1, BT2: value 3xBATT -> BATT
Connections:
- net ch_ilim is gone; now on net GND: R37.2
- net +3.3V: now also R15.1, R2.2
- net GND: now also Q4.3 (E)
- net CH_PG: now reaches TP3.1, U9.3 (~{PG})
- net CH_PG: now also R1.1, R2.1
- net USB_POWER renamed VBUS
- new net: D13.2 (A), R15.2
- new net: Q4.2 (B), R1.2
- new net: D13.1 (K), Q4.1 (C)
Other:
- moved on the sheet: C15, D16, Q4, R1, R2, R54, SW3

Commit message: wip, layout progress
Parts:
- removed R2: 47k, Resistor_SMD:R_0805_2012Metric, symbol Device:R_Small
- added D3, D4, D5: ORAGE, Mlab_D:SMD_LED_RIGHT_KINGBRIGHT_1605, symbol LION2CELL01D-rescue:LED-RESCUE-LION2CELL01C
- added NT1, NT2: NetTie_2, NetTie:NetTie-2_SMD_Pad0.5mm, symbol Device:NetTie_2
- added R11, R12, R13: 270R, Resistor_SMD:R_0805_2012Metric, symbol Device:R_Small
- D1, D13, D16, D2, D3, D4, D5: footprint LED_SMD:LED_1206_3216Metric -> Mlab_D:SMD_LED_RIGHT_KINGBRIGHT_1605
- R2: now not fitted
- R8: footprint Resistor_SMD:R_0805_2012Metric -> Resistor_SMD:R_2512_6332Metric
Connections:
- net +3V3: now also D3.1 (A), D4.1 (A), D5.1 (A)
- net GAUGE_SRP: now also NT2.1; no longer BT1.1- (-), BT1.2- (-), BT2.1- (-), BT2.2- (-), BT2.3- (-), R8.1
- net GND: now also NT1.2; no longer R7.1
- net F: now reaches U2.11 (QF)
- net F: now also R11.2
- net G: now reaches U2.12 (QG)
- net G: now also R12.2
- net H: now reaches U2.13 (QH)
- net H: now also R13.2
- net CHARGE_CTRL: no longer names the net of U1.12 (P5/HDQ)
- new net: D3.2 (K), R11.1
- new net: D5.2 (K), R13.1
- new net: BT1.1- (-), BT1.2- (-), BT2.1- (-), BT2.2- (-), BT2.3- (-), NT2.2, R8.1
- new net: D4.2 (K), R12.1
- new net GAUGE_SRN: NT1.1, R7.1
Other:
- moved on the sheet: BT1A, BT1B, BT2A, BT2B, BT2C, C13, C14, C15, C19, C23, C24, C25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

Commit message: wip, layout improvements
Parts:
- D1, D2: value ORAGE -> RED
- D3, D4, D5: value ORAGE -> GREEN
- SW3: footprint (none) -> Mlab_SW:SKRT
Other:
- note added: "GREEN"
- note added: "ORANGE"
- note added: "RED"
Changed lines of the file:
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@@
+    (stroke (width 0) (type default))
+  )
+  (polyline (pts (xy 266.7 114.3) (xy 266.7 120.65))
     (stroke (width 0) (type default))
   )
@@
     (stroke (width 0) (type default))
   )
+  (polyline (pts (xy 266.7 129.54) (xy 266.7 143.51))
+    (stroke (width 0) (type default))
+  )
   (wire (pts (xy 111.76 165.1) (xy 116.84 165.1))
     (stroke (width 0) (type default))
@@
     (stroke (width 0) (type solid))
   )
+  (polyline (pts (xy 266.7 121.92) (xy 266.7 128.27))
+    (stroke (width 0) (type default))
+  )
   (wire (pts (xy 209.55 123.19) (xy 208.28 123.19))
     (stroke (width 0) (type solid))
@@
     (stroke (width 0) (type default))
   )
+  (text "GREEN" (at 269.24 139.7 90)
+    (effects (font (size 1.27 1.27)) (justify left bottom))
+  )
   (text "FUEL GAUGE" (at 73.66 107.95 0)
     (effects (font (size 2.9972 2.9972)) (justify left bottom))
   )
+  (text "RED" (at 269.24 119.38 90)
+    (effects (font (size 1.27 1.27)) (justify left bottom))
+  )
   (text "Battery Status Indicator" (at 214.63 100.33 0)
     (effects (font (size 2.9972 2.9972)) (justify left bottom))
+  )
+  (text "ORANGE" (at 269.24 128.27 90)
+    (effects (font (size 1.27 1.27)) (justify left bottom))
   )
   (label "CH_BTN" (at 68.58 58.42 0) (fields_autoplaced)
@@
       (effects (font (size 1 1)))
     )
-    (property "Value" "ORAGE" (at 251.46 133.35 0)
+    (property "Value" "GREEN" (at 251.46 133.35 0)
       (effects (font (size 1 1)))
     )
@@
       (effects (font (size 1.27 1.27)))
     )
-    (property "Footprint" "" (at 43.18 80.01 0)
+    (property "Footprint" "Mlab_SW:SKRT" (at 43.18 80.01 0)
       (effects (font (size 1.27 1.27)) hide)
     )
@@
       (effects (font (size 1 1)))
     )
-    (property "Value" "ORAGE" (at 251.46 140.97 0)
+    (property "Value" "GREEN" (at 251.46 140.97 0)
       (effects (font (size 1 1)))
     )
@@
       (effects (font (size 1 1)))
     )
-    (property "Value" "ORAGE" (at 251.46 114.3 0)
+    (property "Value" "RED" (at 251.46 114.3 0)
       (effects (font (size 1 1)))
     )
@@
       (effects (font (size 1 1)))
     )
-    (property "Value" "ORAGE" (at 251.46 137.16 0)
+    (property "Value" "GREEN" (at 251.46 137.16 0)
       (effects (font (size 1 1)))
     )
@@
       (effects (font (size 1 1)))
     )
-    (property "Value" "ORAGE" (at 251.46 129.54 0)
+    (property "Value" "GREEN" (at 251.46 129.54 0)
       (effects (font (size 1 1)))
     )
@@
       (effects (font (size 1 1)))
     )
-    (property "Value" "ORAGE" (at 251.46 118.11 0)
+    (property "Value" "RED" (at 251.46 118.11 0)
       (effects (font (size 1 1)))
     )
@@
     )
     (property "Footprint" "Package_SO:TSSOP-14_4.4x5mm_P0.65mm" (at 228.6 132.08 0)
-      (effects (font (size 1 1)))
+      (effects (font (size 1 1)) hide)
     )
     (property "Datasheet" "" (at 228.6 132.08 0)

Commit message: Wip, layout
Parts:
- removed R2: 1k, Resistor_SMD:R_0805_2012Metric, symbol Device:R_Small
- removed R2 (x2): 10k, Resistor_SMD:R_0805_2012Metric, symbol Device:R_Small
- removed TP3: CH_PG, TestPoint:TestPoint_Pad_D1.5mm, symbol Connector:TestPoint
- removed TP4: CH_STAT, TestPoint:TestPoint_Pad_D1.5mm, symbol Connector:TestPoint
- removed TP5: CH_INT, TestPoint:TestPoint_Pad_D1.5mm, symbol Connector:TestPoint
- C1, C3, C4, C6, C7: value 100nF -> 100n
- C2: value 1uF -> 1u
- D1, D2, D3, D4, D5: symbol LION2CELL01D-rescue:LED-RESCUE-LION2CELL01C -> Device:LED_Small
- Q3: renamed from Q8; value PNP -> BC807-25; footprint (none) -> Package_TO_SOT_SMD:SOT-23-3; symbol Simulation_SPICE:PNP -> Device:Q_PNP_BEC
- Q4: symbol Simulation_SPICE:NPN -> Device:Q_NPN_BEC
- R4: value 10K NTC -> 10k NTC
- renumbered C15 to C11, C19 to C16, C23 to C17, C24 to C18, C25 to C19, C13 to C7, C14 to C8, D16 to D3, D13 to D4, NT2 to NT1, NT1 to NT2, R54 to R21, R15 to R22, R37 to R24, R41 to R27, R42 to R28, SW3 to SW1, U9 to U8
Connections:
- net +3.3V: now also C1.1, C7.1, D1.2 (A), D2.2 (A), D3.2 (A), D3.2 (A), D3.2 (A), D4.2 (A), D4.2 (A), D4.2 (A), D5.2 (A), D5.2 (A), Q3.2 (E), U1.5 (CE), U1.6 (REGIN), U2.14 (VCC), U2.9 (CLR); no longer R21.1, R22.1
- net GND: now also Q4.2 (E), Q4.2 (E); no longer Q4.3 (E), Q4.3 (E)
- net at R13.1: now also D4.1 (K); no longer D5.2 (K)
- net at R22.2: now also Q4.3 (C); no longer D4.2 (A)
- net at R11.1: now also D3.1 (K); no longer D3.2 (K) (x2)
- net at Q4.1 (B): now also R1.2; no longer D3.1 (K)
- net at R13.1: now also D1.1 (K); no longer D5.2 (K)
- net at R1.2: now also Q4.1 (B); no longer Q4.2 (B)
- net at R12.1: now also D5.1 (K); no longer D4.2 (K)
- net at Q3.1 (B): now also R1.2; no longer R1.2
- net at D4.1 (K): now also R22.1; no longer Q4.1 (C)
- net at R9.1: now also D5.1 (K); no longer D1.2 (K)
- net at R10.1: now also D4.1 (K); no longer D2.2 (K)
- net at R12.1: now also D2.1 (K); no longer D4.2 (K)
- net at R21.2: now also Q4.3 (C); no longer D3.2 (A)
- removed net +3V3: C1.1, C7.1, D1.1 (A), D2.1 (A), D3.1 (A), D3.1 (A), D4.1 (A), D4.1 (A), D5.1 (A), D5.1 (A), Q3.3 (E), U1.5 (CE), U1.6 (REGIN), U2.14 (VCC), U2.9 (CLR)
- new net: Q3.3 (C), R1.2
- new net: D3.1 (K), R21.1
Other:
- note added: "Doodhadnout optimální hodnoty odporů k LEDkám"
- note added: "Need to obtain 2.5V, here"
- note added: "Zkontrolovat správnou polaritu LED oproti pouzdru z datasheetu. Symbol, který zde byl použit měl obrácené značení pinů."
- moved on the sheet: D3, D4, R1, R21, R22
