File: hw/sch_pcb/mcu.kicad_sch (KiCad schematic)
At the start: 37 parts, among them J2 SD_Card-FPS009-4200-0, J22 HEADER_2x03, J5 HEADER_1x01, J6 HEADER_1x01, U10 ATMEGA1284P-AU, U11 PCF85263A, U6 AT24CS64-SSHM, Y1 8 MHz, Y2 ABS07-120-32.768KHZ-T

Commit message: wip, update schematics, board outlines
Parts:
- removed J5, J6: HEADER_1x01, Mlab_Pin_Headers:Straight_1x01, symbol MLAB_HEADER:HEADER_1x01
- added J3: SM06B-GHS-TB, Connector_JST:JST_GH_SM06B-GHS-TB_1x06-1MP_P1.25mm_Horizontal, symbol MLAB_CONNECTORS_JST:SM06B-GHS-TB
- added J4: SM04B-GHS-TB, Connector_JST:JST_GH_SM04B-GHS-TB_1x04-1MP_P1.25mm_Horizontal, symbol MLAB_CONNECTORS_JST:SM04B-GHS-TB
- added R33, R34: 100R, Resistor_SMD:R_0603_1608Metric, symbol SPACEDOS02A_PCB01A-rescue:R-device-DATALOGGER01A-rescue-CCP2019V01A-rescue-SPAC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
- added SW2: MCU_RST, symbol Switch:SW_Push
- C25, C36: footprint Capacitor_SMD:C_0603_1608Metric -> Capacitor_SMD:C_0805_2012Metric
- C26, C27, C28, C31, C34, C35, C39, C44, C47, C60: footprint Capacitor_SMD:C_0603_1608Metric -> Capacitor_SMD:C_0805_2012Metric; symbol SPACEDOS01A_PCB01A-rescue:C-device-DATALOGGER01A-rescue-CCP2019V01A-rescue -> Device:C_Small; UST_ID 5c70984812875079b91f8bf2 -> (none)
- C30, C33: footprint Capacitor_SMD:C_0603_1608Metric -> Capacitor_SMD:C_0805_2012Metric; symbol SPACEDOS01A_PCB01A-rescue:C-device-DATALOGGER01A-rescue-CCP2019V01A-rescue -> Device:C_Small; UST_ID 5c70984812875079b91f8be4 -> (none)
- C40: footprint Capacitor_SMD:C_0603_1608Metric -> Capacitor_SMD:C_0805_2012Metric; symbol SPACEDOS01A_PCB01A-rescue:C-device-DATALOGGER01A-rescue-CCP2019V01A-rescue -> Device:C_Small; UST_ID 5c70984812875079b91f8bf5 -> (none)
- C43: footprint Capacitor_SMD:C_0603_1608Metric -> Capacitor_SMD:C_0805_2012Metric; symbol SPACEDOS01A_PCB01A-rescue:C-device-DATALOGGER01A-rescue-CCP2019V01A-rescue -> Device:C_Small; UST_ID 5e3ff6511287502a33bad72b -> (none)
- R17, R18, R23, R24, R25, R45: footprint Resistor_SMD:R_0603_1608Metric -> Resistor_SMD:R_0805_2012Metric
- Y1: footprint Mlab_XTAL:Crystal_HC49-4H_Vertical -> Crystal:Crystal_SMD_3225-4Pin_3.2x2.5mm; symbol Device:Crystal -> Device:Crystal_GND24_Small; UST_ID 5c70984712875079b91f8b0e -> (none)
Connections:
- net PC0 is gone; now on net SCL: U11.7 (SCL), U6.6 (SCL)
- net PC1 is gone; now on net SDA: U11.6 (SDA), U6.5 (SDA)
- net +3.3V: now also C36.1
- net GND: now also C36.2, Y1.2, Y1.4, J3.6, J3.MP, J4.4, J4.MP, SW2.1
- net RST#_P: now also SW2.2
- net at C33.1, U10.8 (XTAL1): now also Y1.3; no longer Y1.2
- new net: J3.3, R34.2
- new net: J3.2, R33.2
- new net 5v_EXT: J3.1, J4.1
- no-connect marks 12 -> 14
Other:
- moved on the sheet: C26, C27, C28, C30, C31, C33, C34, C35, C36, C39, C40, C43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

Commit message: WIP: schematics and layout improvements
Parts:
- removed C22: 10uF, Capacitor_SMD:C_0603_1608Metric, symbol Device:C_Small
- removed C25: 100nF, Capacitor_SMD:C_0805_2012Metric, symbol Device:C_Small
- removed C?: 1nF, Capacitor_SMD:C_0805_2012Metric, symbol Device:C_Small
- removed C?: 1uF, Capacitor_SMD:C_0805_2012Metric, symbol Device:C_Small
- removed J2: SD_Card-FPS009-4200-0, Mlab_CON:FPS009-4200-0, symbol MLAB_CONNECTORS:SD_Card-FPS009-4200-0
- removed L2: 100uH, Inductor_SMD:L_0805_2012Metric_Pad1.15x1.40mm_HandSolder, symbol Device:L
- removed R17, R18, R24, R25: 100R, Resistor_SMD:R_0805_2012Metric, symbol SPACEDOS02A_PCB01A-rescue:R-device-DATALOGGER01A-rescue-CCP2019V01A-rescue-SPAC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
- removed R45: 10R, Resistor_SMD:R_0805_2012Metric, symbol SPACEDOS02A_PCB01A-rescue:R-device-DATALOGGER01A-rescue-CCP2019V01A-rescue-SPAC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
- removed U?: TPS22965-Q1, Package_SON:WSON-8-1EP_2x2mm_P0.5mm_EP0.9x1.6mm_ThermalVias, symbol DATALOGGER01A-rescue:TPS22965-Q1-MLAB_IO
- added C3, C4: C_Small, Capacitor_SMD:C_0805_2012Metric, symbol Device:C_Small
- added C47, C6: 100nF, Capacitor_SMD:C_0805_2012Metric, symbol Device:C_Small
- added C47: 1u, Capacitor_SMD:C_0805_2012Metric, symbol Device:C_Small
- added C5, C7: 100n, Capacitor_SMD:C_0805_2012Metric, symbol Device:C_Small
- added D16 (x3): ORANGE, LED_SMD:LED_1206_3216Metric, symbol Device:LED_Small
- added IC1: MAX14502AETL+, Mlab_IO:QFN40P500X500X80-41N, symbol MLAB_IO:MAX14502AETL+
- added IC2: TMUX1574DYYR, symbol MLAB_IO:TMUX1574DYYR
- added J9: SD_Card-FPS009-4200-0, Mlab_CON:FPS009-4200-0, symbol MLAB_CONNECTORS:SD_Card-FPS009-4200-0
- added NT1: NetTie_2, NetTie:NetTie-2_SMD_Pad0.5mm, symbol Device:NetTie_2
- added Q4 (x3): BC817-25, Package_TO_SOT_SMD:SOT-23-3, symbol Simulation_SPICE:NPN
- added R1 (x3): 1k, Resistor_SMD:R_0805_2012Metric, symbol Device:R_Small
- added R1: 6.19k, Resistor_SMD:R_0805_2012Metric, symbol Device:R_Small
- added R17 (x6): 100R, Resistor_SMD:R_0805_2012Metric, symbol SPACEDOS02A_PCB01A-rescue:R-device-DATALOGGER01A-rescue-CCP2019V01A-rescue-SPAC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
- added R2 (x3): 10k, Resistor_SMD:R_0805_2012Metric, symbol Device:R_Small
- added R54 (x3): R, Resistor_SMD:R_0805_2012Metric, symbol Device:R_Small
- added U3: ISL21080DIH309, Package_TO_SOT_SMD:SOT-23, symbol Reference_Voltage:ISL21070CIH320Z-TK
Connections:
- net RX1 is gone; now on net EXT_RX: U10.11 ((PCINT26/RXD1/INT0)PD2)
- net TX1 is gone; now on net EXT_TX: U10.12 ((PCINT27/TXD1/INT1)PD3)
- net +3.3V: now also C47.1, C6.1, IC1.1 (I2C_SEL), IC1.39 (VCC), IC1.5 (VIO), IC2.16 (VDD), R2.2, R2.2, R2.2, R54.1, R54.1, R54.1
- net AVCC: now also U3.1 (Vin)
- net CS_SD: now also IC1.14 (HDAT1_3)
- net GND: now also C3.2, C4.2, C47.2, C5.2, C6.2, C7.2, IC1.18 (GND_1), IC1.24 (GND_2), IC1.26 (GND_3), IC1.33 (CCRD_PRST), IC1.35 (N.C._1), IC1.36 (N.C._2), IC1.37 (GND_4), IC1.4 (ADD), IC1.41 (GND_5), IC2.8 (GND), J9.12 (SHELL1), J9.3 (VSS), J9.6 (VSS), NT1.1, Q4.3 (E), Q4.3 (E), Q4.3 (E), R1.2
- net MISO: no longer U10.2 ((PCINT14/MISO)PB6)
- net MOSI: no longer U10.1 ((PCINT13/MOSI)PB5)
- net SCK: no longer U10.3 ((PCINT15/SCK)PB7)
- net EXT_I2C_SCL: now reaches J4.2
- net EXT_I2C_SDA: now reaches J4.3
- net EXT_RX: now reaches R34.1
- net SPI_MUX_EN: now reaches U10.21 ((PCINT18/TCK)PC2)
- net SPI_MUX_EN: now also IC2.15 (~{EN})
- net EXT_A1: now reaches U10.35 ((PCINT2/ADC2)PA2)
- net at U10.37 ((PCINT0/ADC0)PA0): now also C47.1, U3.2 (Vout)
- net EXT_B0: now reaches U10.40 ((PCINT8/T0/XCK)PB0)
- net EXT_B1: now reaches U10.41 ((PCINT9/CLKO/T1)PB1)
- net DET_I2C_EN: now reaches U10.42 ((PCINT10/AIN0/INT2)PB2)
- net EXT_TX: now reaches R33.1
- net PC3 renamed SPI_MUX_SEL
- net SPI_MUX_SEL: now also IC2.1 (SEL)
- net PC4: no longer names the net of U10.23 ((PCINT20/TDO)PC4)
- net PC5_D1: no longer names the net of U10.24 ((PCINT21/TDI)PC5)
- net PC6_D2 renamed EXT_C0
- net PC7_D3 renamed EXT_C1
- net RX0 renamed MCU_RX0
- net SCL renamed SCL_MCU
- net SCL_MCU: now also IC1.2 (SCL)
- net SDA renamed SDA_MCU
- net SDA_MCU: now also IC1.3 (SDA)
- net SD_PWR renamed 3v3_SD_CTRL
- net TX0 renamed MCU_TX0
- net Voltage_Reference renamed EXT_A0
- new net: D16.2 (A), R54.2 (x3)
- new net: J9.9 (DAT2), R17.2
- new net: J9.1 (CD/DAT3), R17.2
- new net: J9.2 (CMD), R17.2
- new net: J9.5 (CLK), R17.2
- new net: J9.7 (DAT0), R17.1
- new net: J9.8 (DAT1), R17.1
- new net: D16.1 (K), Q4.1 (C) (x3)
- new net: Q4.2 (B), R1.2 (x3)
- new net #BERR: IC1.6 (~{BERR}/INT)
- new net #BUSSY: IC1.7 (~{BUSY})
- new net #RST: IC1.9 (~{RST})
- new net 3v3_SD: IC1.40 (VSD), J9.4 (VDD)
- new net CCLK1: IC1.32 (CCLK1), R17.1
- new net CCMD1: IC1.34 (CCMD1), R17.1
- new net CDAT1_0: IC1.13 (CDAT1_0), R17.2
- new net CDAT1_1: IC1.12 (CDAT1_1), R17.2
- new net CDAT1_2: IC1.11 (CDAT1_2), R17.1
- new net CDAT1_3: IC1.10 (CDAT1_3), R17.1
- new net CLDO: C5.1, IC1.38 (CLDO)
- new net EXT_MISO: IC2.6 (S2B)
- new net EXT_MOSI: IC2.3 (S1B)
- new net EXT_SCK: IC2.10 (S3B)
- new net GNDA: C47.2, NT1.2, U3.3 (GND)
- new net LED_U1: R1.1, R2.1
- new net LED_U2: R1.1, R2.1
- new net LED_U3: R1.1, R2.1
- new net MISO_MCU: IC2.7 (D2), U10.2 ((PCINT14/MISO)PB6)
- new net MISO_SD: IC1.17 (HDAT1_0), IC2.5 (S2A)
- new net MOSI_MCU: IC2.4 (D1), U10.1 ((PCINT13/MOSI)PB5)
- new net MOSI_SD: IC1.31 (HCMD1), IC2.2 (S1A)
- new net RREF: IC1.27 (RREF), R1.1
- new net SCK_MCU: IC2.9 (D3), U10.3 ((PCINT15/SCK)PB7)
- new net SCK_SD: IC1.29 (HCLK1), IC2.11 (S3A)
- new net USB_CONNECTED: IC1.28 (KVBUS)
- new net USB_D+: IC1.22 (CD+)
- new net USB_D-: IC1.21 (CD-)
- new net USB_FTDI_D+: IC1.20 (HD+)
- new net USB_FTDI_D-: IC1.19 (HD-)
- new net VCC: C4.1
- new net VSD: C3.1
- new net VTM: C7.1, IC1.23 (VTM)
- new net mode: IC1.8 (MODE)
- no-connect marks 14 -> 17
Other:
- note removed: "9,7 mV"
- moved on the sheet: C30, C33, C36, C40, C43, C44, C47, C60, J3, J4, R23, R33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

Commit message: wip layout, add datasheets
Parts:
- removed C28, C47: 100nF, Capacitor_SMD:C_0805_2012Metric, symbol Device:C_Small
- removed J3: SM06B-GHS-TB, Connector_JST:JST_GH_SM06B-GHS-TB_1x06-1MP_P1.25mm_Horizontal, symbol MLAB_CONNECTORS_JST:SM06B-GHS-TB
- removed J4: SM04B-GHS-TB, Connector_JST:JST_GH_SM04B-GHS-TB_1x04-1MP_P1.25mm_Horizontal, symbol MLAB_CONNECTORS_JST:SM04B-GHS-TB
- removed R33, R34: 100R, Resistor_SMD:R_0603_1608Metric, symbol SPACEDOS02A_PCB01A-rescue:R-device-DATALOGGER01A-rescue-CCP2019V01A-rescue-SPAC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
- added R40, R78: R_Small, symbol Device:R_Small
- added SW3 (x2): SW_Push, symbol Switch:SW_Push
Connections:
- net MISO is gone; now on net MISO_MCU: J22.1
- net MOSI is gone; now on net MOSI_MCU: J22.4
- net SCK is gone; now on net SCK_MCU: J22.3
- net SCK_SD is gone; now on net 3v3_SD: IC1.29 (HCLK1), IC2.11 (S3A)
- net +3.3V: now also R40.1, R78.1
- net GND: now also SW3.2, SW3.2
- net LED_U1: now also U10.13 ((PCINT28/XCK1/OC1B)PD4)
- net LED_U2: now also U10.14 ((PCINT294/OC1A)PD5)
- net LED_U3: now also U10.15 ((PCINT30/OC2B/ICP)PD6)
- net SCL_MCU: no longer IC1.2 (SCL), U11.7 (SCL), U6.6 (SCL)
- net SDA_MCU: no longer IC1.3 (SDA), U11.6 (SDA), U6.5 (SDA)
- net BTN_USER_B: now reaches U10.30 ((PCINT7/ADC7)PA7)
- net BTN_USER_B: now also R78.2, SW3.1
- net BTN_USER_A: now reaches U10.31 ((PCINT6/ADC6)PA6)
- net BTN_USER_A: now also R40.2, SW3.1
- new net SCL_I2C: IC1.2 (SCL), U11.7 (SCL), U6.6 (SCL)
- new net SDA_I2C: IC1.3 (SDA), U11.6 (SDA), U6.5 (SDA)
- no-connect marks 17 -> 13
Other:
- note removed: "MISO"
- note removed: "MOSI"
- note removed: "SCK"
- note removed: "VTG"
- moved on the sheet: C26, C27, C31, C34, C35, C39, D16, L1, Q4, R1, R2, R54

Commit message: WIP
Parts:
- added R56, R57: 1k, Resistor_SMD:R_0805_2012Metric, symbol Device:R_Small
- R40, R78: footprint (none) -> Resistor_SMD:R_0805_2012Metric
Connections:
- net 3v3_SD: no longer IC1.29 (HCLK1), IC2.11 (S3A)
- net GND: now also R57.2
- net USB_CONNECTED: no longer names the net of IC1.28 (KVBUS)
- net USB_CONNECTED: now also R56.2, R57.1
- new net SCK_SD: IC1.29 (HCLK1), IC2.11 (S3A)
- new net VBUS: R56.1

Commit message: WIP, layout improvement
Parts:
- removed C47: 100nF, Capacitor_SMD:C_0805_2012Metric, symbol Device:C_Small
- removed NT1: NetTie_2, NetTie:NetTie-2_SMD_Pad0.5mm, symbol Device:NetTie_2
- removed U3: ISL21080DIH309, Package_TO_SOT_SMD:SOT-23, symbol Reference_Voltage:ISL21070CIH320Z-TK
- IC2: footprint (none) -> Mlab_IO:SOT-23-16 THIN
Connections:
- net EXT_A0: now also U10.37 ((PCINT0/ADC0)PA0); no longer U10.36 ((PCINT1/ADC1)PA1)
- net EXT_A1: now also U10.36 ((PCINT1/ADC1)PA1); no longer U10.35 ((PCINT2/ADC2)PA2)
Other:
- moved on the sheet: C3, C4, C5, C6, C7, R1

Commit message: wip, layout progress
Parts:
- D16: footprint LED_SMD:LED_1206_3216Metric -> Mlab_D:SMD_LED_RIGHT_KINGBRIGHT_1605
Connections:
- net SPI_MUX_EN: now also U10.22 ((PCINT19/TMS)PC3); no longer U10.21 ((PCINT18/TCK)PC2)
- net SPI_MUX_SEL: now also U10.21 ((PCINT18/TCK)PC2); no longer U10.22 ((PCINT19/TMS)PC3)
Changed lines of the file:
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@@
     (stroke (width 0) (type default))
   )
-  (text_box "MISO_SD ... pin 31 a 17, asi není dobře.. "
+  (text_box "MISO_SD ... pin 31 a 17, asi není dobře.. Je potřěba zkontrolovat zapojení SPI mezi MCU, "
     (at 130.81 161.29 0) (size 38.1 22.86)
     (stroke (width 0) (type default))
@@
     (effects (font (size 1.524 1.524)) (justify left bottom))
   )
-  (label "SPI_MUX_EN" (at 199.39 83.82 0) (fields_autoplaced)
+  (label "SPI_MUX_EN" (at 199.39 86.36 0) (fields_autoplaced)
     (effects (font (size 1.27 1.27)) (justify left bottom))
   )
@@
     (effects (font (size 1.27 1.27)) (justify left bottom))
   )
-  (label "SPI_MUX_SEL" (at 199.39 86.36 0) (fields_autoplaced)
+  (label "SPI_MUX_SEL" (at 199.39 83.82 0) (fields_autoplaced)
     (effects (font (size 1.27 1.27)) (justify left bottom))
   )
@@
       (effects (font (size 1.27 1.27)) (justify right))
     )
-    (property "Footprint" "LED_SMD:LED_1206_3216Metric" (at 40.64 53.34 90)
+    (property "Footprint" "Mlab_D:SMD_LED_RIGHT_KINGBRIGHT_1605" (at 40.64 53.34 90)
       (effects (font (size 1.27 1.27)) hide)
     )
@@
       (effects (font (size 1.27 1.27)) (justify right))
     )
-    (property "Footprint" "LED_SMD:LED_1206_3216Metric" (at 40.64 82.55 90)
+    (property "Footprint" "Mlab_D:SMD_LED_RIGHT_KINGBRIGHT_1605" (at 40.64 82.55 90)
       (effects (font (size 1.27 1.27)) hide)
     )
@@
       (effects (font (size 1.27 1.27)) (justify right))
     )
-    (property "Footprint" "LED_SMD:LED_1206_3216Metric" (at 77.47 53.34 90)
-      (effects (font (size 1.27 1.27)) hide)
-    )
+    (property "Footprint" "Mlab_D:SMD_LED_RIGHT_KINGBRIGHT_1605" (at 77.47 53.34 90)
+      (effects (font (size 1.27 1.27)) hide)
+    )

Commit message: wip, layout improvements
Parts:
- added R11: 10k, Resistor_SMD:R_0805_2012Metric, symbol Device:R_Small
- SW2, SW3: footprint (none) -> Mlab_SW:KMT031 NGJ LHS C&K
- SW3: footprint (none) -> Mlab_SW:SKRT
Connections:
- net 3v3_SD_CTRL: now also U10.22 ((PCINT19/TMS)PC3); no longer U10.43 ((PCINT11/AIN1/OC0)PB3)
- net GND: now also IC2.15 (~{EN}), R11.1
- net SPI_MUX_SEL: now also R11.2
- net CCLK1 renamed CCLK
- net CCMD1 renamed CCMD
- net CDAT1_0 renamed CDAT0
- net CDAT1_1 renamed CDAT1
- net CDAT1_2 renamed CDAT2
- net CDAT1_3 renamed CDAT3
- net EXT_SCK renamed EXT_SCLK
- net SCK_MCU renamed SCLK_MCU
- net SCK_SD renamed SCLK_SD
- removed net SPI_MUX_EN: IC2.15 (~{EN}), U10.22 ((PCINT19/TMS)PC3)
- no-connect marks 13 -> 15

Commit message: Wip, layout
Parts:
- removed C31, C34, C35, C39: 100nF, Capacitor_SMD:C_0805_2012Metric, symbol Device:C_Small
- removed C4: C_Small, Capacitor_SMD:C_0805_2012Metric, symbol Device:C_Small
- removed L1: 10uH - LQH32CN100K23L, Inductor_SMD:L_1210_3225Metric_Pad1.42x2.65mm_HandSolder, symbol SPACEDOS01A_PCB01A-rescue:L-device-DATALOGGER01A-rescue-CCP2019V01A-rescue
- removed R2 (x3): 10k, Resistor_SMD:R_0805_2012Metric, symbol Device:R_Small
- added BZ1: Buzzer, symbol Device:Buzzer
- added Q4: BC817-25, Package_TO_SOT_SMD:SOT-23-3, symbol Device:Q_NPN_BEC
- added R1: 1k, Resistor_SMD:R_0805_2012Metric, symbol Device:R_Small
- C26, C27, C36, C44, C6, C60: value 100nF -> 100n
- Q4: symbol Simulation_SPICE:NPN -> Device:Q_NPN_BEC
- renumbered R56 to R55, R57 to R56, R40 to R58, R78 to R59, R11 to R60, SW2 to SW4
Connections:
- net AVCC is gone; now on net +3.3V: U10.27 (AVCC)
- net +3.3V: now also D16.2 (A), D16.2 (A), D16.2 (A), BZ1.1 (-); no longer R54.1, R54.1, R54.1
- net GND: now also Q4.2 (E), Q4.2 (E), Q4.2 (E), Q4.2 (E); no longer Q4.3 (E), Q4.3 (E), Q4.3 (E)
- net at R54.2: now also Q4.3 (C); no longer D16.2 (A) (x3)
- net at Q4.1 (B): now also R1.2; no longer D16.1 (K)
- net at R1.2: now also Q4.1 (B); no longer Q4.2 (B) (x2)
- net at D16.1 (K): now also R54.1; no longer Q4.1 (C) (x2)
- net buzzer: now reaches U10.16 ((PCINT31/OC2A)PD7)
- net buzzer: now also R1.1
- new net: Q4.1 (B), R1.2
- new net: BZ1.2 (+), Q4.3 (C)
- new net: D16.1 (K), R54.1
Other:
- moved on the sheet: D16, R54
