File: hw/sch_pcb/mcu.kicad_sch (KiCad schematic)
At the start: 55 parts, among them IC1 MAX14502AETL+, J22 HEADER_2x03, J9 SD_Card-FPS009-4200-0, Q4 BC817-25, SW3 KMT031, SW3 SKRTLAE010, SW4 KMT031, U10 ATMEGA1284P-AU, U11 PCF85263A, U12 TMUX1574DYYR, U6 AT24CS64-SSHM, Y1 8 MHz, Y2 ABS07-120-32.768KHZ-T

Commit message: uprava schematu
Parts:
- removed BZ1: LET9032ES-03L-2.7-16-R, MLAB_BUZZER:MagneticBuzzer_LET9032ES-03L-2.7-16-R, symbol Device:Buzzer
- removed C26, C27, C36, C44, C5, C6, C60, C7: 100n, Capacitor_SMD:C_0805_2012Metric, symbol Device:C_Small
- removed C30, C33: 15p, Capacitor_SMD:C_0805_2012Metric, symbol Device:C_Small
- removed C40: 10u, Capacitor_SMD:C_0805_2012Metric, symbol Device:C_Small
- removed C43: 4u7, Capacitor_SMD:C_0805_2012Metric, symbol Device:C_Small
- removed C47: 1u, Capacitor_SMD:C_0805_2012Metric, symbol Device:C_Small
- removed D16 (x3): ORANGE, Mlab_D:SMD_LED_RIGHT_KINGBRIGHT_1605, symbol Device:LED_Small
- removed IC1: MAX14502AETL+, Mlab_IO:QFN40P500X500X80-41N, symbol MLAB_IO:MAX14502AETL+
- removed J22: HEADER_2x03, Mlab_Pin_Headers:SMD_2x03, symbol MLAB_HEADER:HEADER_2x03
- removed J9: SD_Card-FPS009-4200-0, Mlab_CON:FPS009-4200-0, symbol MLAB_CONNECTORS:SD_Card-FPS009-4200-0
- removed JP7: Jumper_3_Bridged12, Jumper:SolderJumper-3_P1.3mm_Bridged2Bar12_RoundedPad1.0x1.5mm, symbol Jumper:Jumper_3_Bridged12
- removed Q4 (x4): BC817-25, Package_TO_SOT_SMD:SOT-23-3, symbol Device:Q_NPN_BEC
- removed R1 (x4), R54, R55: 1k, Resistor_SMD:R_0805_2012Metric, symbol Device:R_Small
- removed R1: 6.19k, Resistor_SMD:R_0805_2012Metric, symbol Device:R_Small
- removed R17 (x6): 100R, Resistor_SMD:R_0805_2012Metric, symbol SPACEDOS02A_PCB01A-rescue:R-device-DATALOGGER01A-rescue-CCP2019V01A-rescue-SPAC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
- removed R23 (x2), R57, R58, R59: 10k, Resistor_SMD:R_0805_2012Metric, symbol Device:R_Small
- removed R54 (x3): 270R, Resistor_SMD:R_0805_2012Metric, symbol Device:R_Small
- removed SW3, SW4: KMT031, Mlab_SW:KMT031 NGJ LHS C&K, symbol Switch:SW_Push
- removed SW3: SKRTLAE010, Mlab_SW:SKRT, symbol MLAB_SW:SW_Push_shield
- removed U10: ATMEGA1284P-AU, Package_QFP:TQFP-44_10x10mm_P0.8mm, symbol SPACEDOS01A_PCB01A-rescue:ATMEGA1284P-AU-atmel-DATALOGGER01A-rescue-CCP2019V01A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
- removed U11: PCF85263A, Package_SO:TSSOP-10_3x3mm_P0.5mm, symbol MLAB_IO:PCF85263A
- removed U12: TMUX1574DYYR, Mlab_IO:SOT-23-16 THIN, symbol MLAB_IO:TMUX1574DYYR
- removed U6: AT24CS64-SSHM, Package_SO:SOIC-8_3.9x4.9mm_P1.27mm, symbol Memory_EEPROM:AT24CS64-SSHM
- removed Y1: 8 MHz, Crystal:Crystal_SMD_3225-4Pin_3.2x2.5mm, symbol Device:Crystal_GND24_Small
- removed Y2: ABS07-120-32.768KHZ-T, Mlab_XTAL:ABS07, symbol SPACEDOS01A_PCB01A-rescue:Crystal-device-DATALOGGER01A-rescue-CCP2019V01A-rescue
Connections:
- no-connect marks 17 -> 0
