File: hw/sch_pcb/sw_source.kicad_sch (KiCad schematic)
At the start: 31 parts, among them U1 TPS631000DRLR

Commit message: wip, update schematics, board outlines
Parts:
- C1: symbol Device:C -> Device:C_Small; UST_ID 650b58f1462c6d9e7205463b -> (none)
- C2: symbol Device:C -> Device:C_Small; UST_ID 5c70984812875079b91f8bbf -> (none)
- C3: symbol Device:C -> Device:C_Small; UST_ID 5c70984712875079b91f8b53 -> (none)
- R1: symbol Device:R -> Device:R_Small; UST_ID 650b59ec462c6d9e72054677 -> (none)
- R1: footprint Resistor_SMD:R_0603_1608Metric -> Resistor_SMD:R_0805_2012Metric; symbol Device:R -> Device:R_Small; UST_ID 650b59ec462c6d9e72054677 -> (none)
- R2: footprint Resistor_SMD:R_0603_1608Metric -> Resistor_SMD:R_0805_2012Metric; symbol Device:R -> Device:R_Small; UST_ID 650b5a43462c6d9e7205468e -> (none)
- R2: symbol Device:R -> Device:R_Small; UST_ID 650b5a43462c6d9e7205468e -> (none)
- R3: symbol Device:R -> Device:R_Small; UST_ID 650b5abb462c6d9e720546b8 -> (none)
- R4: footprint Resistor_SMD:R_0603_1608Metric -> Resistor_SMD:R_0805_2012Metric
Other:
- moved on the sheet: C1, C2, C3, JP1, R1, R2, R3

Commit message: WIP: schematics and layout improvements
Parts:
- added C22: 10uF, Capacitor_SMD:C_0603_1608Metric, symbol Device:C_Small
- added C25: 100nF, Capacitor_SMD:C_0805_2012Metric, symbol Device:C_Small
- added C8: 10uF, Capacitor_SMD:C_0805_2012Metric, symbol Device:C_Small
- added C?: 1uF, Capacitor_SMD:C_0805_2012Metric, symbol Device:C_Small
- added C?: 1nF, Capacitor_SMD:C_0805_2012Metric, symbol Device:C_Small
- added L1: 1uH, Inductor_SMD:L_1008_2520Metric, symbol Device:L_Small
- added L2: 100uH, Inductor_SMD:L_0805_2012Metric_Pad1.15x1.40mm_HandSolder, symbol Device:L
- added U1: TS5A4594, Package_TO_SOT_SMD:SOT-23-5, symbol MLAB_IO:TS5A4594
- added U?: TPS22965-Q1, Package_SON:WSON-8-1EP_2x2mm_P0.5mm_EP0.9x1.6mm_ThermalVias, symbol DATALOGGER01A-rescue:TPS22965-Q1-MLAB_IO
- JP1: footprint Connector_PinHeader_2.54mm:PinHeader_1x02_P2.54mm_Vertical -> Jumper:SolderJumper-2_P1.3mm_Open_RoundedPad1.0x1.5mm
Connections:
- net +3.3V: now also C?.1, U?.1 (VIN), U?.2 (VIN), U?.4 (VBIAS)
- net GND: now also C22.2, C25.2, C8.2, C?.2, C?.2, U1.3 (GND), U?.5 (GND), U?.9
- new net: L1.2, U1.1 (COM)
- new net: L2.1, U?.7 (VOUT), U?.8 (VOUT)
- new net: C?.1, U?.6 (CT)
- new net 3v3_SD: C22.1, C25.1, C8.1, L1.1, L2.2
- new net 3v3_SD_CTRL: U1.4 (IN), U?.3 (ON)
- new net VCC: U1.2 (NO), U1.5 (VCC)
Other:
- note added: "SD card power switch"

Commit message: wip layout, add datasheets
Parts:
- U1: footprint KiCad:SOTFL50P160X60-8N -> Package_TO_SOT_SMD:SOT-583-8
Connections:
- net VCC is gone; now on net +3.3V: U1.2 (NO), U1.5 (VCC)
Changed lines of the file:
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@@
   (junction (at 267.97 -15.24) (diameter 0) (color 0 0 0 0)
   )
+  (junction (at 134.62 156.21) (diameter 0) (color 0 0 0 0)
+  )
   (junction (at 100.33 147.32) (diameter 0) (color 0 0 0 0)
   )
@@
     (stroke (width 0) (type default))
   )
+  (wire (pts (xy 134.62 156.21) (xy 134.62 154.94))
+    (stroke (width 0) (type default))
+  )
   (wire (pts (xy 124.46 143.51) (xy 124.46 139.7))
     (stroke (width 0) (type default))
@@
     (stroke (width 0) (type default))
   )
-  (wire (pts (xy 134.62 154.94) (xy 134.62 157.48))
-    (stroke (width 0) (type default))
-  )
   (wire (pts (xy 306.07 -15.24) (xy 309.88 -15.24))
     (stroke (width 0) (type solid))
@@
     (stroke (width 0) (type default))
   )
+  (wire (pts (xy 129.54 156.21) (xy 134.62 156.21))
+    (stroke (width 0) (type default))
+  )
   (wire (pts (xy 120.65 34.29) (xy 120.65 30.48))
     (stroke (width 0) (type default))
@@
     (stroke (width 0) (type solid))
   )
+  (wire (pts (xy 134.62 156.21) (xy 134.62 157.48))
+    (stroke (width 0) (type default))
+  )
   (wire (pts (xy 297.18 -6.35) (xy 299.72 -6.35))
     (stroke (width 0) (type solid))
@@
     (effects (font (size 1 1)) (justify right bottom))
   )
-  (label "5v_FB" (at 134.62 157.48 180) (fields_autoplaced)
-    (effects (font (size 1 1)) (justify right bottom))
+  (label "5v_FB" (at 129.54 156.21 0) (fields_autoplaced)
+    (effects (font (size 1 1)) (justify left bottom))
   )
   (label "5v_FB" (at 115.57 175.26 270) (fields_autoplaced)
@@
     )
   )
+  (symbol (lib_id "power:+3.3V") (at 276.86 39.37 0) (unit 1)
+    (in_bom yes) (on_board yes) (dnp no) (fields_autoplaced)
+    (property "Reference" "#PWR?" (at 276.86 43.18 0)
+      (effects (font (size 1 1)) hide)
+    )
+    (property "Value" "+3.3V" (at 276.86 34.29 0)
+      (effects (font (size 1 1)))
+    )
+    (property "Footprint" "" (at 276.86 39.37 0)
+      (effects (font (size 1 1)) hide)
+    )
+    (property "Datasheet" "" (at 276.86 39.37 0)
+      (effects (font (size 1 1)) hide)
+    )
+    (pin "1")
+    (instances
+      (project "Peripherals"
+        (path "/5251a3af-ca7f-447d-b796-a6d47f48d23f"
+          (reference "#PWR?") (unit 1)
+        )
+      )
+      (project "LION5CELL01"
+        (path "/cca3030a-cb35-4155-89c2-3a41e5a0afad"
+          (reference "#PWR058") (unit 1)
+        )
+        (path "/cca3030a-cb35-4155-89c2-3a41e5a0afad/80b69af2-66cc-4579-a230-ef2d06af8a00"
+          (reference "#PWR075") (unit 1)
+        )
+        (path "/cca3030a-cb35-4155-89c2-3a41e5a0afad/c1fc2aff-2b12-4e41-a798-c0c7c2bf1b4c"
+          (reference "#PWR082") (unit 1)
+        )
+      )
+      (project "DATALOGGER02"
+        (path "/d5fa3405-b56f-43e6-a8bd-3ff789d79996/8c16a5bf-8019-4e77-9247-0011396b8bad"
+          (reference "#PWR?") (unit 1)
+        )
+      )
+    )
+  )
   (symbol (lib_id "Device:R_Small") (at 87.63 39.37 90) (unit 1)
     (in_bom yes) (on_board yes) (dnp no) (fields_autoplaced)
@@
       (effects (font (size 1 1)) (justify left))
     )
-    (property "Footprint" "KiCad:SOTFL50P160X60-8N" (at 125.73 58.42 0)
+    (property "Footprint" "Package_TO_SOT_SMD:SOT-583-8" (at 125.73 58.42 0)
       (effects (font (size 1 1)) (justify left) hide)
     )
@@
     )
   )
-  (symbol (lib_id "power:VCC") (at 276.86 39.37 0) (unit 1)
-    (in_bom yes) (on_board yes) (dnp no)
-    (property "Reference" "#PWR024" (at 276.86 43.18 0)
-      (effects (font (size 1.27 1.27)) hide)
-    )
-    (property "Value" "VCC" (at 278.13 35.56 0)
-      (effects (font (size 1.27 1.27)))
-    )
-    (property "Footprint" "" (at 276.86 39.37 0)
-      (effects (font (size 1.27 1.27)) hide)
-    )
-    (property "Datasheet" "" (at 276.86 39.37 0)
-      (effects (font (size 1.27 1.27)) hide)
-    )
-    (pin "1")
-    (instances
-      (project "USBSDREADER01"
-        (path "/2ae32537-a16f-4c5b-a56b-c6dddfb8ddb4"
-          (reference "#PWR024") (unit 1)
-        )
-      )
-      (project "LION5CELL01"
-        (path "/cca3030a-cb35-4155-89c2-3a41e5a0afad/80b69af2-66cc-4579-a230-ef2d06af8a00"
-          (reference "#PWR0146") (unit 1)
-        )
-        (path "/cca3030a-cb35-4155-89c2-3a41e5a0afad/c1fc2aff-2b12-4e41-a798-c0c7c2bf1b4c"
-          (reference "#PWR082") (unit 1)
-        )
-      )
-    )
-  )
   (symbol (lib_id "power:GND") (at 146.05 99.06 0) (unit 1)
     (in_bom yes) (on_board yes) (dnp no)
@@
     )
   )
-  (symbol (lib_id "power:VCC") (at 288.29 29.21 0) (unit 1)
-    (in_bom yes) (on_board yes) (dnp no)
-    (property "Reference" "#PWR025" (at 288.29 33.02 0)
-      (effects (font (size 1.27 1.27)) hide)
-    )
-    (property "Value" "VCC" (at 284.48 27.94 0)
-      (effects (font (size 1.27 1.27)))
-    )
-    (property "Footprint" "" (at 288.29 29.21 0)
-      (effects (font (size 1.27 1.27)) hide)
-    )
-    (property "Datasheet" "" (at 288.29 29.21 0)
-      (effects (font (size 1.27 1.27)) hide)
-    )
-    (pin "1")
-    (instances
-      (project "USBSDREADER01"
-        (path "/2ae32537-a16f-4c5b-a56b-c6dddfb8ddb4"
-          (reference "#PWR025") (unit 1)
-        )
-      )
-      (project "LION5CELL01"
-        (path "/cca3030a-cb35-4155-89c2-3a41e5a0afad/80b69af2-66cc-4579-a230-ef2d06af8a00"
-          (reference "#PWR0149") (unit 1)
-        )
-        (path "/cca3030a-cb35-4155-89c2-3a41e5a0afad/c1fc2aff-2b12-4e41-a798-c0c7c2bf1b4c"
-          (reference "#PWR088") (unit 1)
-        )
-      )
-    )
-  )
   (symbol (lib_id "power:GND") (at 100.33 39.37 0) (unit 1)
     (in_bom yes) (on_board yes) (dnp no) (fields_autoplaced)
@@
   (symbol (lib_id "Device:C_Small") (at 100.33 36.83 0) (unit 1)
     (in_bom yes) (on_board yes) (dnp no)
-    (property "Reference" "C1" (at 102.87 34.29 0)
+    (property "Reference" "C1" (at 102.87 38.1 0)
       (effects (font (size 1 1)) (justify left))
     )
@@
       (effects (font (size 1 1)) (justify left))
     )
-    (property "Footprint" "KiCad:SOTFL50P160X60-8N" (at 125.73 171.45 0)
+    (property "Footprint" "Package_TO_SOT_SMD:SOT-583-8" (at 125.73 171.45 0)
       (effects (font (size 1 1)) (justify left) hide)
     )
@@
     )
   )
+  (symbol (lib_id "power:+3.3V") (at 288.29 29.21 0) (unit 1)
+    (in_bom yes) (on_board yes) (dnp no) (fields_autoplaced)
+    (property "Reference" "#PWR?" (at 288.29 33.02 0)
+      (effects (font (size 1 1)) hide)
+    )
+    (property "Value" "+3.3V" (at 288.29 24.13 0)
+      (effects (font (size 1 1)))
+    )
+    (property "Footprint" "" (at 288.29 29.21 0)
+      (effects (font (size 1 1)) hide)
+    )
+    (property "Datasheet" "" (at 288.29 29.21 0)
+      (effects (font (size 1 1)) hide)
+    )
+    (pin "1")
+    (instances
+      (project "Peripherals"
+        (path "/5251a3af-ca7f-447d-b796-a6d47f48d23f"
+          (reference "#PWR?") (unit 1)
+        )
+      )
+      (project "LION5CELL01"
+        (path "/cca3030a-cb35-4155-89c2-3a41e5a0afad"
+          (reference "#PWR058") (unit 1)
+        )
+        (path "/cca3030a-cb35-4155-89c2-3a41e5a0afad/80b69af2-66cc-4579-a230-ef2d06af8a00"
+          (reference "#PWR075") (unit 1)
+        )
+        (path "/cca3030a-cb35-4155-89c2-3a41e5a0afad/c1fc2aff-2b12-4e41-a798-c0c7c2bf1b4c"
+          (reference "#PWR077") (unit 1)
+        )
+      )
+      (project "DATALOGGER02"
+        (path "/d5fa3405-b56f-43e6-a8bd-3ff789d79996/8c16a5bf-8019-4e77-9247-0011396b8bad"
+          (reference "#PWR?") (unit 1)
+        )
+      )
+    )
+  )
   (symbol (lib_id "Device:R_Small") (at 134.62 96.52 0) (unit 1)
     (in_bom yes) (on_board yes) (dnp no) (fields_autoplaced)
@@
       (effects (font (size 1 1)) (justify left))
     )
-    (property "Footprint" "KiCad:SOTFL50P160X60-8N" (at 125.73 115.57 0)
+    (property "Footprint" "Package_TO_SOT_SMD:SOT-583-8" (at 125.73 115.57 0)
       (effects (font (size 1 1)) (justify left) hide)
     )

Commit message: WIP
Parts:
- removed C8: 10uF, Capacitor_SMD:C_0805_2012Metric, symbol Device:C_Small
- removed L1: 1uH, Inductor_SMD:L_1008_2520Metric, symbol Device:L_Small
- removed U1: TS5A4594, Package_TO_SOT_SMD:SOT-23-5, symbol MLAB_IO:TS5A4594
Other:
- note removed: "SD card power switch"
- moved on the sheet: C22, C25, C?, L2, U?

Commit message: Wip, layout
Parts:
- C22: footprint Capacitor_SMD:C_0603_1608Metric -> Capacitor_SMD:C_0805_2012Metric
- C25: value 100nF -> 100n
- C?: value 1uF -> 1u

Commit message: WIP
Parts:
- C22: UST_ID 5c70984812875079b91f8bf5 -> (none)
- C25: UST_ID 5c70984812875079b91f8bf2 -> (none)
- C?: UST_ID 5c70984712875079b91f8b50 -> (none)
- C?: UST_ID 5c70984712875079b91f8b45 -> (none)
- L1: UST_ID 650b5977462c6d9e72054656 -> (none)
- L2: UST_ID 626fd6fcdc56076e9a222966 -> (none)
- R4, R5: UST_ID 5c70984512875079b91f898c -> (none)
- U1: UST_ID 63de5ae4ae0b2d5aa05e2714 -> (none)
- U?: UST_ID 5c70984712875079b91f8b78 -> (none)
Changed lines of the file:
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@@
       (effects (font (size 1 1)) hide)
     )
-    (property "UST_ID" "5c70984712875079b91f8b50" (at 185.42 39.37 0)
+    (property "UST_ID" "" (at 185.42 39.37 0)
       (effects (font (size 1 1)) hide)
     )
@@
       (effects (font (size 1 1)) hide)
     )
-    (property "UST_ID" "650b5977462c6d9e72054656" (at 119.38 26.67 0)
+    (property "UST_ID" "" (at 119.38 26.67 0)
       (effects (font (size 1 1)) hide)
     )
@@
       (effects (font (size 1 1)) hide)
     )
-    (property "UST_ID" "5c70984512875079b91f898c" (at 87.63 39.37 0)
+    (property "UST_ID" "" (at 87.63 39.37 0)
       (effects (font (size 1 1)) hide)
     )
@@
         )
         (path "/cca3030a-cb35-4155-89c2-3a41e5a0afad/c1fc2aff-2b12-4e41-a798-c0c7c2bf1b4c"
-          (reference "R65") (unit 1)
+          (reference "R64") (unit 1)
         )
       )
@@
       (effects (font (size 1 1)) (justify left) hide)
     )
-    (property "UST_ID" "63de5ae4ae0b2d5aa05e2714" (at 123.19 34.29 0)
+    (property "UST_ID" "" (at 123.19 34.29 0)
       (effects (font (size 1 1)) hide)
     )
@@
       (effects (font (size 1 1)) hide)
     )
-    (property "UST_ID" "5c70984512875079b91f898c" (at 60.96 132.08 0)
+    (property "UST_ID" "" (at 60.96 132.08 0)
       (effects (font (size 1 1)) hide)
     )
@@
         )
         (path "/cca3030a-cb35-4155-89c2-3a41e5a0afad/c1fc2aff-2b12-4e41-a798-c0c7c2bf1b4c"
-          (reference "R62") (unit 1)
+          (reference "R61") (unit 1)
         )
       )
@@
         )
         (path "/cca3030a-cb35-4155-89c2-3a41e5a0afad/c1fc2aff-2b12-4e41-a798-c0c7c2bf1b4c"
-          (reference "R66") (unit 1)
+          (reference "R65") (unit 1)
         )
       )
@@
         )
         (path "/cca3030a-cb35-4155-89c2-3a41e5a0afad/c1fc2aff-2b12-4e41-a798-c0c7c2bf1b4c"
-          (reference "R69") (unit 1)
+          (reference "R68") (unit 1)
         )
       )
@@
       (effects (font (size 1 1)) hide)
     )
-    (property "UST_ID" "5c70984512875079b91f898c" (at 60.96 123.19 0)
+    (property "UST_ID" "" (at 60.96 123.19 0)
       (effects (font (size 1 1)) hide)
     )
@@
         )
         (path "/cca3030a-cb35-4155-89c2-3a41e5a0afad/c1fc2aff-2b12-4e41-a798-c0c7c2bf1b4c"
-          (reference "R61") (unit 1)
+          (reference "R60") (unit 1)
         )
       )
@@
       (effects (font (size 1 1)) (justify left) hide)
     )
-    (property "UST_ID" "63de5ae4ae0b2d5aa05e2714" (at 123.19 147.32 0)
+    (property "UST_ID" "" (at 123.19 147.32 0)
       (effects (font (size 1 1)) hide)
     )
@@
       (effects (font (size 1 1)) hide)
     )
-    (property "UST_ID" "626fd6fcdc56076e9a222966" (at 219.71 34.29 0)
+    (property "UST_ID" "" (at 219.71 34.29 0)
       (effects (font (size 1 1)) hide)
     )
@@
         )
         (path "/cca3030a-cb35-4155-89c2-3a41e5a0afad/c1fc2aff-2b12-4e41-a798-c0c7c2bf1b4c"
-          (reference "R67") (unit 1)
+          (reference "R66") (unit 1)
         )
       )
@@
       (effects (font (size 1 1)) hide)
     )
-    (property "UST_ID" "650b5977462c6d9e72054656" (at 119.38 83.82 0)
+    (property "UST_ID" "" (at 119.38 83.82 0)
       (effects (font (size 1 1)) hide)
     )
@@
       (effects (font (size 1 1)) hide)
     )
-    (property "UST_ID" "5c70984512875079b91f898c" (at 85.09 151.13 0)
+    (property "UST_ID" "" (at 85.09 151.13 0)
       (effects (font (size 1 1)) hide)
     )
@@
         )
         (path "/cca3030a-cb35-4155-89c2-3a41e5a0afad/c1fc2aff-2b12-4e41-a798-c0c7c2bf1b4c"
-          (reference "R63") (unit 1)
+          (reference "R62") (unit 1)
         )
       )
@@
       (effects (font (size 1 1)) hide)
     )
-    (property "UST_ID" "5c70984712875079b91f8b78" (at 205.74 36.83 0)
+    (property "UST_ID" "" (at 205.74 36.83 0)
       (effects (font (size 1 1)) hide)
     )
@@
       (effects (font (size 1 1)) hide)
     )
-    (property "UST_ID" "650b5977462c6d9e72054656" (at 119.38 139.7 0)
+    (property "UST_ID" "" (at 119.38 139.7 0)
       (effects (font (size 1 1)) hide)
     )
@@
         )
         (path "/cca3030a-cb35-4155-89c2-3a41e5a0afad/c1fc2aff-2b12-4e41-a798-c0c7c2bf1b4c"
-          (reference "R70") (unit 1)
+          (reference "R69") (unit 1)
         )
       )
@@
       (effects (font (size 1 1)) hide)
     )
-    (property "UST_ID" "5c70984712875079b91f8b45" (at 217.17 39.37 0)
+    (property "UST_ID" "" (at 217.17 39.37 0)
       (effects (font (size 1 1)) hide)
     )
@@
         )
         (path "/cca3030a-cb35-4155-89c2-3a41e5a0afad/c1fc2aff-2b12-4e41-a798-c0c7c2bf1b4c"
-          (reference "R68") (unit 1)
+          (reference "R67") (unit 1)
         )
       )
@@
       (effects (font (size 1 1)) hide)
     )
-    (property "UST_ID" "5c70984812875079b91f8bf5" (at 227.33 39.37 0)
+    (property "UST_ID" "" (at 227.33 39.37 0)
       (effects (font (size 1 1)) hide)
     )
@@
         )
         (path "/cca3030a-cb35-4155-89c2-3a41e5a0afad/c1fc2aff-2b12-4e41-a798-c0c7c2bf1b4c"
-          (reference "R71") (unit 1)
+          (reference "R70") (unit 1)
         )
       )
@@
       (effects (font (size 1 1)) hide)
     )
-    (property "UST_ID" "5c70984512875079b91f898c" (at 86.36 97.79 0)
+    (property "UST_ID" "" (at 86.36 97.79 0)
       (effects (font (size 1 1)) hide)
     )
@@
         )
         (path "/cca3030a-cb35-4155-89c2-3a41e5a0afad/c1fc2aff-2b12-4e41-a798-c0c7c2bf1b4c"
-          (reference "R64") (unit 1)
+          (reference "R63") (unit 1)
         )
       )
@@
       (effects (font (size 1 1)) hide)
     )
-    (property "UST_ID" "5c70984812875079b91f8bf2" (at 237.49 39.37 0)
+    (property "UST_ID" "" (at 237.49 39.37 0)
       (effects (font (size 1 1)) hide)
     )
@@
       (effects (font (size 1 1)) (justify left) hide)
     )
-    (property "UST_ID" "63de5ae4ae0b2d5aa05e2714" (at 123.19 91.44 0)
-      (effects (font (size 1 1)) hide)
-    )
+    (property "UST_ID" "" (at 123.19 91.44 0)
+      (effects (font (size 1 1)) hide)
+    )

Commit message: wip, split power adapter to BATDATSOCKET01
Parts:
- U1: Height (none) -> 0.5; UST_ID (none) -> 63de5ae4ae0b2d5aa05e2714
Other:
- company: (none) -> MLAB.cz
- title: (none) -> BATDATUNTI01
