File: hw/sch_pcb/connector.kicad_sch (KiCad schematic)
At the start: 1 part, among them J2 46436-9327

Commit message: wip layout, add datasheets
Connections:
- net EXT_B0: now also J2.E5; no longer J2.E6
- net EXT_B1: now also J2.E6; no longer J2.E5
- net EXT_C0: now also J2.E1; no longer J2.E2
- net EXT_C1: now also J2.E2; no longer J2.E1
- net EXT_I2C_SCL: now reaches J2.C1
- net EXT_I2C_SDA: now reaches J2.C2
Changed lines of the file:
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@@
     )
   )
-  (global_label "EXT_C0" (shape input) (at 129.54 110.49 270) (fields_autoplaced)
+  (global_label "EXT_C0" (shape input) (at 127 110.49 270) (fields_autoplaced)
     (effects (font (size 1.27 1.27)) (justify right))
-    (property "Intersheetrefs" "${INTERSHEET_REFS}" (at 129.54 120.2484 90)
+    (property "Intersheetrefs" "${INTERSHEET_REFS}" (at 127 120.2484 90)
       (effects (font (size 1.27 1.27)) (justify right) hide)
     )
@@
     )
   )
+  (global_label "EXT_I2C_SDA" (shape bidirectional) (at 149.86 80.01 0) (fields_autoplaced)
+    (effects (font (size 1 1)) (justify left))
+    (property "Intersheetrefs" "${INTERSHEET_REFS}" (at 162.4663 80.01 0)
+      (effects (font (size 1 1)) (justify left) hide)
+    )
+  )
+  (global_label "EXT_I2C_SCL" (shape input) (at 149.86 77.47 0) (fields_autoplaced)
+    (effects (font (size 1 1)) (justify left))
+    (property "Intersheetrefs" "${INTERSHEET_REFS}" (at 161.5437 77.47 0)
+      (effects (font (size 1 1)) (justify left) hide)
+    )
+  )
   (global_label "3v3_EXT" (shape input) (at 116.84 82.55 180) (fields_autoplaced)
     (effects (font (size 1 1)) (justify right))
@@
     )
   )
-  (global_label "EXT_B1" (shape input) (at 137.16 110.49 270) (fields_autoplaced)
+  (global_label "EXT_B1" (shape input) (at 139.7 110.49 270) (fields_autoplaced)
     (effects (font (size 1.27 1.27)) (justify right))
-    (property "Intersheetrefs" "${INTERSHEET_REFS}" (at 137.16 120.2484 90)
+    (property "Intersheetrefs" "${INTERSHEET_REFS}" (at 139.7 120.2484 90)
       (effects (font (size 1.27 1.27)) (justify right) hide)
     )
@@
     )
   )
-  (global_label "EXT_B0" (shape input) (at 139.7 110.49 270) (fields_autoplaced)
+  (global_label "EXT_B0" (shape input) (at 137.16 110.49 270) (fields_autoplaced)
     (effects (font (size 1.27 1.27)) (justify right))
-    (property "Intersheetrefs" "${INTERSHEET_REFS}" (at 139.7 120.2484 90)
+    (property "Intersheetrefs" "${INTERSHEET_REFS}" (at 137.16 120.2484 90)
       (effects (font (size 1.27 1.27)) (justify right) hide)
     )
   )
-  (global_label "EXT_C1" (shape input) (at 127 110.49 270) (fields_autoplaced)
+  (global_label "EXT_C1" (shape input) (at 129.54 110.49 270) (fields_autoplaced)
     (effects (font (size 1.27 1.27)) (justify right))
-    (property "Intersheetrefs" "${INTERSHEET_REFS}" (at 127 120.2484 90)
+    (property "Intersheetrefs" "${INTERSHEET_REFS}" (at 129.54 120.2484 90)
       (effects (font (size 1.27 1.27)) (justify right) hide)
     )
@@
   )
   (symbol (lib_id "MLAB_CONNECTORS:MOLEX_46436-9327") (at 132.08 74.93 0) (unit 1)
-    (in_bom yes) (on_board yes) (dnp no) (fields_autoplaced)
+    (in_bom yes) (on_board yes) (dnp no)
     (property "Reference" "J2" (at 124.46 77.47 0)
       (effects (font (size 1.27 1.27)) (justify left))
     )
-    (property "Value" "46436-9327" (at 129.54 69.85 90)
+    (property "Value" "46436-9327" (at 137.16 81.28 0)
       (effects (font (size 1.27 1.27)))
     )

Commit message: WIP, layout improvement
Parts:
- removed J2: 46436-9327, Mlab_CON:MOLEX_46436-9327, symbol MLAB_CONNECTORS:MOLEX_46436-9327

Commit message: WIP
Parts:
- added J5: 46436-9327, Mlab_CON:MOLEX_46437-9327, symbol MLAB_CONNECTORS:MOLEX_46436-9327
- added J6: HEADER_2x15, Connector_PinHeader_2.54mm:PinHeader_2x15_P2.54mm_Vertical, symbol MLAB_HEADER:HEADER_2x15
- added JP7: Jumper_3_Bridged12, Jumper:SolderJumper-3_P1.3mm_Bridged12_RoundedPad1.0x1.5mm, symbol Jumper:Jumper_3_Bridged12
Connections:
- new net 3v3: J5.A3, J5.B3, J6.5, J6.6, JP7.1 (A)
- new net 5v: J5.A4, J5.B4, J6.3, J6.4, JP7.3 (B)
- new net A0: J5.D4, J6.10
- new net A1: J5.D5, J6.12
- new net B0: J5.E5, J6.16
- new net B1: J5.E6, J6.14
- new net BATT: J5.P1, J5.P4
- new net C0: J5.E1, J6.20
- new net C1: J5.E2, J6.18
- new net GND: J5.A2, J5.A5, J5.B2, J5.B5, J5.P2, J5.P3, J6.1, J6.2, J6.21, J6.22, J6.29, J6.30
- new net I2C_PWR: J6.25, J6.26, JP7.2 (C)
- new net MISO: J5.D2, J6.17
- new net MOSI: J5.D3, J6.15
- new net RX: J5.E4, J6.11
- new net SCL: J5.C1, J6.23, J6.24
- new net SCLK: J5.D1, J6.19
- new net SDA: J5.C2, J6.27, J6.28
- new net TX: J5.E3, J6.13
- no-connect marks 0 -> 12

Commit message: WIP, add ust ID for existing parts
Parts:
- removed J5: 46436-9327, Mlab_CON:MOLEX_46437-9327, symbol MLAB_CONNECTORS:MOLEX_46436-9327
- removed J6: HEADER_2x15, Connector_PinHeader_2.54mm:PinHeader_2x15_P2.54mm_Vertical, symbol MLAB_HEADER:HEADER_2x15
- removed JP7: Jumper_3_Bridged12, Jumper:SolderJumper-3_P1.3mm_Bridged12_RoundedPad1.0x1.5mm, symbol Jumper:Jumper_3_Bridged12
Connections:
- no-connect marks 12 -> 0
